File: BPS_Test/Hardware/BPS_Test.sch (KiCad schematic (older format))
At the start: 0 parts

Commit message: Major additions to BOM and began Schematics in earnest!
Parts:
- added BT?: BATTERY, symbol BATTERY
- added C? (x2): 10uF, symbol CSMALL
- added C? (x3): .1uF, symbol CSMALL
- added C? (x2): 8pF, symbol CSMALL
- added IC?: ATMEGA644P-A, TQFP44, symbol ATMEGA644P-A
- added U?: SPX29150T-L-5-0/TR, symbol SPX29150T-L-5-0/TR
- added X?: 20 MHz, symbol CRYSTAL
Connections:
- net labels added: +5V, +BATT, GND
- wire segments 0 -> 24
