File: BPS_Test/Hardware/BPS_Test.sch (KiCad schematic (older format))
At the start: 11 parts

Commit message: Fleshed out schematics some more. Updated Project Log and BOM
Parts:
- removed U?: SPX29150T-L-5-0/TR, symbol SPX29150T-L-5-0/TR
- added C? (x3): .1uF, symbol CSMALL
- added L?: 33uH, symbol INDUCTOR
- added P?: ISP, symbol CONN_3X2
- added R? (x2): R, symbol R
- added S?: TL3315NF160Q, symbol TL3315NF160Q
- BT?: value BATTERY -> 6-7.2VDC
Connections:
- net labels added: AIN0, MISO, MOSI, RST, SCK, SMP, SPX29150T-L-5-0/TR, SlaveSelect, VCC, X0, X1, X2, X3, Y0A, Y0B
- wire segments 24 -> 105
Other:
- moved on the sheet: BT?, IC?, X?

Commit message: Updated display matrix to better reflect final project goals
Changed lines of the file:
@@
-EESchema Schematic File Version 2  date 5/5/2012 1:24:45 AM
+EESchema Schematic File Version 2  date 5/5/2012 11:18:12 AM
 LIBS:power
 LIBS:device
@@
 U 1 1 4FA1B881
 P 4550 1950
-F 0 "#U014" H 4850 1550 60  0000 C CNN
+F 0 "#U014" H 4850 1550 60  0001 C CNN
 F 1 "SPX29150T-L-5-0/TR" H 4550 2100 60  0000 C CNN
 	1    4550 1950
