File: BPS_Test/Hardware/BPS_Test.sch (KiCad schematic (older format))
At the start: 19 parts

Commit message: Cleaned up Schematics
Parts:
- added J1: DC, symbol CONN_2
- added J2: USB_2, symbol USB_2
- added R2, R3, R4, R5: 10k, symbol R
- BT1: renamed from BT?; value 6-7.2VDC -> 7.2VDC
- gave numbers to parts that had none: 18
Connections:
- net labels removed: +BATT
- wire segments 120 -> 133
- no-connect marks 0 -> 2
Other:
- note added: "+"
- note added: "-"
