File: BPS_Test/Hardware/BPS_Test_Display.sch (KiCad schematic (older format))
At the start: 22 parts

Commit message: Fleshed out schematics some more. Updated Project Log and BOM
Other:
- moved on the sheet: LED?, R?, U?

Commit message: Updated display matrix to better reflect final project goals
Parts:
- added C? (x2): 10uF, symbol CSMALL
- added C? (x2): .1uF, symbol CSMALL
- added C? (x12): 0.1uF, symbol CSMALL
- added R? (x2): 22k, symbol R
- added U? (x2): AS1107, symbol AS1107
- C? (x6): value CSMALL -> 0.1uF
Connections:
- wire segments 238 -> 324
- no-connect marks 5 -> 25
Other:
- moved on the sheet: R?, U?
