File: BPS_Test/Hardware/BPS_Test_Display.sch (KiCad schematic (older format))
At the start: 42 parts

Commit message: Updated BOM, Project Log, and Schematic PDF, and improved schematic details
Parts:
- added C? (x3): .1uF, symbol CSMALL
- added LED? (x2): RGB_LED, symbol RGB_LED
- C? (x18): value 0.1uF -> .1uF
- gave numbers to parts that had none: 3
Connections:
- wire segments 324 -> 363
- no-connect marks 25 -> 22
Changed lines of the file:
@@
-EESchema Schematic File Version 2  date 5/5/2012 11:24:09 AM
+EESchema Schematic File Version 2  date 5/6/2012 12:55:40 AM
 LIBS:power
 LIBS:device
@@
 EELAYER 25  0
 EELAYER END
-$Descr User 14000 11000
+$Descr User 16000 11000
 encoding utf-8
 Sheet 3 3
 Title "BPS Test Display"
-Date "5 may 2012"
+Date "6 may 2012"
 Rev "1.0"
 Comp "Projects and Stuff LLC"
@@
 Comment4 ""
 $EndDescr
+Wire Wire Line
+	13800 3800 13500 3800
+Wire Wire Line
+	13500 3800 13500 3450
+Wire Wire Line
+	13500 3450 12100 3450
+Connection ~ 12100 3800
+Wire Wire Line
+	12100 3450 12100 3800
+Connection ~ 12000 4100
+Wire Wire Line
+	12000 4100 12000 3550
+Wire Wire Line
+	12000 3550 13600 3550
+Wire Wire Line
+	13600 3550 13600 4100
+Wire Wire Line
+	13600 4100 13800 4100
+Wire Wire Line
+	13800 3100 13550 3100
+Wire Wire Line
+	13550 3100 13550 2650
+Wire Wire Line
+	13550 2650 12050 2650
+Connection ~ 12050 3100
+Wire Wire Line
+	12050 2650 12050 3100
+Wire Wire Line
+	13800 3250 13600 3250
+Connection ~ 15000 2350
+Wire Wire Line
+	15000 2350 2550 2350
+Connection ~ 14900 5350
+Wire Wire Line
+	14900 5400 14900 5350
+Wire Wire Line
+	14800 1150 15000 1150
+Wire Wire Line
+	14800 1150 14800 1300
+Wire Wire Line
+	14800 1500 14800 1550
+Wire Wire Line
+	15000 1150 15000 3800
+Wire Wire Line
+	15100 8600 15100 3250
+Connection ~ 15100 4100
+Connection ~ 15050 3950
+Connection ~ 15000 2950
+Wire Wire Line
+	15100 4100 14950 4100
+Wire Wire Line
+	15100 3250 14950 3250
+Wire Wire Line
+	15000 3800 14950 3800
+Wire Wire Line
+	15000 2950 14950 2950
+Wire Wire Line
+	14950 3100 15050 3100
+Wire Wire Line
+	15050 3950 14950 3950
+Wire Wire Line
+	2550 5700 2700 5700
 Connection ~ 5000 4750
 Wire Wire Line
@@
 Wire Wire Line
 	2700 5700 2700 2650
-Wire Wire Line
-	2700 5700 2550 5700
 Connection ~ 11700 2950
 Wire Wire Line
@@
 	2700 2650 5300 2650
 Wire Wire Line
-	2650 2700 2650 2600
-Wire Wire Line
-	2650 2700 2550 2700
+	2650 2600 2650 2700
 Wire Wire Line
 	6650 5600 6650 5650
@@
 	1050 3300 1150 3300
 Wire Wire Line
-	2550 2350 2600 2350
-Wire Wire Line
 	2550 3300 2600 3300
 Wire Wire Line
@@
 	2550 6300 2600 6300
 Wire Wire Line
-	2550 5350 2600 5350
-Wire Wire Line
 	1050 6300 1150 6300
 Wire Wire Line
@@
 	1050 9300 1150 9300
 Wire Wire Line
-	2550 8350 2600 8350
-Wire Wire Line
 	2550 9300 2600 9300
 Wire Wire Line
@@
 	6650 5400 6650 4850
 Connection ~ 6650 4850
+Wire Wire Line
+	2650 2700 2550 2700
+Wire Wire Line
+	15050 3100 15050 5350
+Wire Wire Line
+	14900 5600 14900 5650
+Wire Wire Line
+	15050 5350 2550 5350
+Wire Wire Line
+	15100 8350 2550 8350
+Connection ~ 15100 8350
+Wire Wire Line
+	15100 8800 15100 8850
+Wire Wire Line
+	12000 3250 12000 2700
+Connection ~ 12000 3250
+Wire Wire Line
+	12000 2700 13600 2700
+Wire Wire Line
+	13600 2700 13600 3250
+Wire Wire Line
+	13800 2950 13500 2950
+Wire Wire Line
+	13500 2950 13500 2600
+Wire Wire Line
+	13500 2600 12100 2600
+Wire Wire Line
+	12100 2600 12100 2950
+Connection ~ 12100 2950
+Wire Wire Line
+	12050 3950 12050 3500
+Connection ~ 12050 3950
+Wire Wire Line
+	12050 3500 13550 3500
+Wire Wire Line
+	13550 3500 13550 3950
+Wire Wire Line
+	13550 3950 13800 3950
+$Comp
+L CSMALL C?
+U 1 1 4FA5DCE7
+P 15100 8700
+F 0 "C?" H 15125 8750 30  0000 L CNN
+F 1 ".1uF" H 15125 8650 30  0000 L CNN
+	1    15100 8700
+	1    0    0    -1
+$EndComp
+$Comp
+L GND #PWR?
+U 1 1 4FA5DCE6
+P 15100 8850
+F 0 "#PWR?" H 15100 8850 30  0001 C CNN
+F 1 "GND" H 15100 8780 30  0001 C CNN
+	1    15100 8850
+	1    0    0    -1
+$EndComp
+$Comp
+L CSMALL C?
+U 1 1 4FA5DCB1
+P 14900 5500
+F 0 "C?" H 14925 5550 30  0000 L CNN
+F 1 ".1uF" H 14925 5450 30  0000 L CNN
+	1    14900 5500
+	1    0    0    -1
+$EndComp
+$Comp
+L GND #PWR?
+U 1 1 4FA5DCB0
+P 14900 5650
+F 0 "#PWR?" H 14900 5650 30  0001 C CNN
+F 1 "GND" H 14900 5580 30  0001 C CNN
+	1    14900 5650
+	1    0    0    -1
+$EndComp
+$Comp
+L GND #PWR?
+U 1 1 4FA5DC8B
+P 14800 1550
+F 0 "#PWR?" H 14800 1550 30  0001 C CNN
+F 1 "GND" H 14800 1480 30  0001 C CNN
+	1    14800 1550
+	1    0    0    -1
+$EndComp
+$Comp
+L CSMALL C?
+U 1 1 4FA5DC8A
+P 14800 1400
+F 0 "C?" H 14825 1450 30  0000 L CNN
+F 1 ".1uF" H 14825 1350 30  0000 L CNN
+	1    14800 1400
+	1    0    0    -1
+$EndComp
+$Comp
+L RGB_LED LED?
+U 1 1 4FA5DC66
+P 14350 3100
+F 0 "LED?" H 14500 2800 60  0000 C CNN
+F 1 "RGB_LED" H 14350 3400 60  0000 C CNN
+	1    14350 3100
+	1    0    0    -1
+$EndComp
+$Comp
+L RGB_LED LED?
+U 1 1 4FA5DC65
+P 14350 3950
+F 0 "LED?" H 14500 3650 60  0000 C CNN
+F 1 "RGB_LED" H 14350 4250 60  0000 C CNN
+	1    14350 3950
+	1    0    0    -1
+$EndComp
 $Comp
 L CSMALL C?
@@
 P 13150 1400
 F 0 "C?" H 13175 1450 30  0000 L CNN
-F 1 "0.1uF" H 13175 1350 30  0000 L CNN
+F 1 ".1uF" H 13175 1350 30  0000 L CNN
 	1    13150 1400
 	1    0    0    -1
@@
 P 11500 1400
 F 0 "C?" H 11525 1450 30  0000 L CNN
-F 1 "0.1uF" H 11525 1350 30  0000 L CNN
+F 1 ".1uF" H 11525 1350 30  0000 L CNN
 	1    11500 1400
 	1    0    0    -1
@@
 P 8200 1400
 F 0 "C?" H 8225 1450 30  0000 L CNN
-F 1 "0.1uF" H 8225 1350 30  0000 L CNN
+F 1 ".1uF" H 8225 1350 30  0000 L CNN
 	1    8200 1400
 	1    0    0    -1
@@
 P 9850 1400
 F 0 "C?" H 9875 1450 30  0000 L CNN
-F 1 "0.1uF" H 9875 1350 30  0000 L CNN
+F 1 ".1uF" H 9875 1350 30  0000 L CNN
 	1    9850 1400
 	1    0    0    -1
@@
 P 6550 1400
 F 0 "C?" H 6575 1450 30  0000 L CNN
-F 1 "0.1uF" H 6575 1350 30  0000 L CNN
+F 1 ".1uF" H 6575 1350 30  0000 L CNN
 	1    6550 1400
 	1    0    0    -1
@@
 P 4900 1400
 F 0 "C?" H 4925 1450 30  0000 L CNN
-F 1 "0.1uF" H 4925 1350 30  0000 L CNN
+F 1 ".1uF" H 4925 1350 30  0000 L CNN
 	1    4900 1400
 	1    0    0    -1
@@
 P 5000 5500
 F 0 "C?" H 5025 5550 30  0000 L CNN
-F 1 "0.1uF" H 5025 5450 30  0000 L CNN
+F 1 ".1uF" H 5025 5450 30  0000 L CNN
 	1    5000 5500
 	1    0    0    -1
@@
 P 13450 8700
 F 0 "C?" H 13475 8750 30  0000 L CNN
-F 1 "0.1uF" H 13475 8650 30  0000 L CNN
+F 1 ".1uF" H 13475 8650 30  0000 L CNN
 	1    13450 8700
 	1    0    0    -1
@@
 P 11800 8700
 F 0 "C?" H 11825 8750 30  0000 L CNN
-F 1 "0.1uF" H 11825 8650 30  0000 L CNN
+F 1 ".1uF" H 11825 8650 30  0000 L CNN
 	1    11800 8700
 	1    0    0    -1
@@
 P 10150 8700
 F 0 "C?" H 10175 8750 30  0000 L CNN
-F 1 "0.1uF" H 10175 8650 30  0000 L CNN
+F 1 ".1uF" H 10175 8650 30  0000 L CNN
 	1    10150 8700
 	1    0    0    -1
@@
 P 8500 8700
 F 0 "C?" H 8525 8750 30  0000 L CNN
-F 1 "0.1uF" H 8525 8650 30  0000 L CNN
+F 1 ".1uF" H 8525 8650 30  0000 L CNN
 	1    8500 8700
 	1    0    0    -1
@@
 P 5200 8700
 F 0 "C?" H 5225 8750 30  0000 L CNN
-F 1 "0.1uF" H 5225 8650 30  0000 L CNN
+F 1 ".1uF" H 5225 8650 30  0000 L CNN
 	1    5200 8700
 	1    0    0    -1
@@
 NoConn ~ 2600 9300
 NoConn ~ 2600 8450
-NoConn ~ 2600 8350
-$Comp
-L AS1107 U?
+$Comp
+L AS1107 UB?
 U 1 1 4FA53118
 P 1850 8450
-F 0 "U?" H 2150 7350 60  0000 C CNN
+F 0 "UB?" H 2150 7350 60  0000 C CNN
 F 1 "AS1107" H 1650 9550 60  0000 C CNN
 	1    1850 8450
@@
 $EndComp
 $Comp
-L AS1107 U?
+L AS1107 UG?
 U 1 1 4FA5310B
 P 1850 5450
-F 0 "U?" H 2150 4350 60  0000 C CNN
+F 0 "UG?" H 2150 4350 60  0000 C CNN
 F 1 "AS1107" H 1650 6550 60  0000 C CNN
 	1    1850 5450
 	1    0    0    -1
 $EndComp
-NoConn ~ 2600 5350
 NoConn ~ 2600 5450
 NoConn ~ 2600 6300
@@
 P 8300 5500
 F 0 "C?" H 8325 5550 30  0000 L CNN
-F 1 "0.1uF" H 8325 5450 30  0000 L CNN
+F 1 ".1uF" H 8325 5450 30  0000 L CNN
 	1    8300 5500
 	1    0    0    -1
@@
 P 11600 5500
 F 0 "C?" H 11625 5550 30  0000 L CNN
-F 1 "0.1uF" H 11625 5450 30  0000 L CNN
+F 1 ".1uF" H 11625 5450 30  0000 L CNN
 	1    11600 5500
 	1    0    0    -1
@@
 P 13250 5500
 F 0 "C?" H 13275 5550 30  0000 L CNN
-F 1 "0.1uF" H 13275 5450 30  0000 L CNN
+F 1 ".1uF" H 13275 5450 30  0000 L CNN
 	1    13250 5500
 	1    0    0    -1
@@
 P 9950 5500
 F 0 "C?" H 9975 5550 30  0000 L CNN
-F 1 "0.1uF" H 9975 5450 30  0000 L CNN
+F 1 ".1uF" H 9975 5450 30  0000 L CNN
 	1    9950 5500
 	1    0    0    -1
@@
 P 6650 5500
 F 0 "C?" H 6675 5550 30  0000 L CNN
-F 1 "0.1uF" H 6675 5450 30  0000 L CNN
+F 1 ".1uF" H 6675 5450 30  0000 L CNN
 	1    6650 5500
 	1    0    0    -1
@@
 P 6850 8700
 F 0 "C?" H 6875 8750 30  0000 L CNN
-F 1 "0.1uF" H 6875 8650 30  0000 L CNN
+F 1 ".1uF" H 6875 8650 30  0000 L CNN
 	1    6850 8700
 	1    0    0    -1
@@
 NoConn ~ 2600 3300
 NoConn ~ 2600 2450
-NoConn ~ 2600 2350
-$Comp
-L AS1107 U?
+$Comp
+L AS1107 UR?
 U 1 1 4FA1E70A
 P 1850 2450
-F 0 "U?" H 2150 1350 60  0000 C CNN
+F 0 "UR?" H 2150 1350 60  0000 C CNN
 F 1 "AS1107" H 1650 3550 60  0000 C CNN
 	1    1850 2450
