File: BPS_Test/Hardware/BPS_Test_Sensors.sch (KiCad schematic (older format))
At the start: 11 parts, among them X0Y0 CAPSENSOR, X1Y0 CAPSENSOR, X2Y0 CAPSENSOR, X3Y0 CAPSENSOR

Commit message: Fleshed out schematics some more. Updated Project Log and BOM
Connections:
- net labels added: GND, VREF
- wire segments 23 -> 24
Other:
- moved on the sheet: RX0, RX1, RX2, RX3, RY0, RYB0
Changed lines of the file:
@@
-EESchema Schematic File Version 2  date 5/2/2012 11:05:33 PM
+EESchema Schematic File Version 2  date 5/5/2012 1:24:45 AM
 LIBS:power
 LIBS:device
@@
 EELAYER 25  0
 EELAYER END
-$Descr A4 11700 8267
+$Descr User 14000 11000
 encoding utf-8
 Sheet 2 3
 Title "BPS Test Sensors"
-Date "3 may 2012"
+Date "5 may 2012"
 Rev "1.0"
 Comp "Projects and Stuff LLC"
@@
 Comment4 ""
 $EndDescr
-Connection ~ 4700 2600
-Wire Wire Line
-	4700 4650 4700 1900
-Wire Wire Line
-	4700 1900 3150 1900
-Wire Wire Line
-	3150 1900 3150 1800
-Connection ~ 4700 4000
-Wire Wire Line
-	4700 3300 3150 3300
-Wire Wire Line
-	3150 3300 3150 3200
-Wire Wire Line
-	2800 3750 3000 3750
-Wire Wire Line
-	2800 2350 3000 2350
-Wire Wire Line
-	3950 5900 4100 5900
-Wire Wire Line
-	4100 5900 4100 5800
-Wire Wire Line
-	2200 3050 2300 3050
-Wire Wire Line
-	2200 1650 2300 1650
-Wire Wire Line
-	4100 5000 4100 5300
-Wire Wire Line
-	4000 4650 4200 4650
-Wire Wire Line
-	4100 4800 4100 4650
-Connection ~ 4100 4650
-Wire Wire Line
-	4000 5150 4100 5150
-Connection ~ 4100 5150
-Wire Wire Line
-	2200 2350 2300 2350
-Wire Wire Line
-	2200 3750 2300 3750
-Wire Wire Line
-	2800 1650 3000 1650
-Wire Wire Line
-	2800 3050 3000 3050
-Wire Wire Line
-	3150 3900 3150 4000
-Wire Wire Line
-	3150 4000 4700 4000
-Wire Wire Line
-	3150 2500 3150 2600
-Wire Wire Line
-	3150 2600 4700 2600
-Connection ~ 4700 3300
+Text GLabel 7300 7350 2    60   Input ~ 0
+GND
+Wire Wire Line
+	7150 7350 7300 7350
+Connection ~ 7900 4400
+Wire Wire Line
+	7900 3700 6350 3700
+Wire Wire Line
+	6350 3700 6350 3600
+Wire Wire Line
+	7900 5100 6350 5100
+Wire Wire Line
+	6350 5100 6350 5000
+Wire Wire Line
+	6000 4150 6200 4150
+Wire Wire Line
+	6000 2750 6200 2750
+Wire Wire Line
+	5400 4850 5500 4850
+Wire Wire Line
+	5400 3450 5500 3450
+Connection ~ 7300 6250
+Wire Wire Line
+	7200 6250 7300 6250
+Connection ~ 7300 5750
+Wire Wire Line
+	7300 5900 7300 5750
+Wire Wire Line
+	7200 5750 7400 5750
+Wire Wire Line
+	7300 6100 7300 6400
+Wire Wire Line
+	5400 2750 5500 2750
+Wire Wire Line
+	5400 4150 5500 4150
+Wire Wire Line
+	7300 6900 7300 7000
+Wire Wire Line
+	7300 7000 7150 7000
+Wire Wire Line
+	6000 3450 6200 3450
+Wire Wire Line
+	6000 4850 6200 4850
+Wire Wire Line
+	6350 4300 6350 4400
+Wire Wire Line
+	6350 4400 7900 4400
+Connection ~ 7900 5100
+Wire Wire Line
+	6350 2900 6350 3000
+Wire Wire Line
+	6350 3000 7900 3000
+Wire Wire Line
+	7900 3000 7900 5750
+Connection ~ 7900 3700
+Text HLabel 7150 7350 0    60   BiDi ~ 0
+VREF
 $Comp
 L CAPSENSOR X3Y0
 U 1 1 4FA1E531
-P 3150 3750
-F 0 "X3Y0" H 3110 3870 60  0000 C CNN
-F 1 "CAPSENSOR" V 3260 3740 40  0000 C CNN
-	1    3150 3750
+P 6350 4850
+F 0 "X3Y0" H 6310 4970 60  0000 C CNN
+F 1 "CAPSENSOR" V 6460 4840 40  0000 C CNN
+	1    6350 4850
 	1    0    0    -1
 $EndComp
@@
 L CAPSENSOR X2Y0
 U 1 1 4FA1E52F
-P 3150 3050
-F 0 "X2Y0" H 3110 3170 60  0000 C CNN
-F 1 "CAPSENSOR" V 3260 3040 40  0000 C CNN
-	1    3150 3050
+P 6350 4150
+F 0 "X2Y0" H 6310 4270 60  0000 C CNN
+F 1 "CAPSENSOR" V 6460 4140 40  0000 C CNN
+	1    6350 4150
 	1    0    0    -1
 $EndComp
@@
 L CAPSENSOR X1Y0
 U 1 1 4FA1E528
-P 3150 2350
-F 0 "X1Y0" H 3110 2470 60  0000 C CNN
-F 1 "CAPSENSOR" V 3260 2340 40  0000 C CNN
-	1    3150 2350
+P 6350 3450
+F 0 "X1Y0" H 6310 3570 60  0000 C CNN
+F 1 "CAPSENSOR" V 6460 3440 40  0000 C CNN
+	1    6350 3450
 	1    0    0    -1
 $EndComp
@@
 L CAPSENSOR X0Y0
 U 1 1 4FA1E50B
-P 3150 1650
-F 0 "X0Y0" H 3110 1770 60  0000 C CNN
-F 1 "CAPSENSOR" V 3260 1640 40  0000 C CNN
-	1    3150 1650
+P 6350 2750
+F 0 "X0Y0" H 6310 2870 60  0000 C CNN
+F 1 "CAPSENSOR" V 6460 2740 40  0000 C CNN
+	1    6350 2750
 	1    0    0    -1
 $EndComp
@@
 L R RYB0
 U 1 1 4FA1E1CF
-P 4100 5550
-F 0 "RYB0" V 4180 5550 50  0000 C CNN
-F 1 "470k" V 4100 5550 50  0000 C CNN
-	1    4100 5550
+P 7300 6650
+F 0 "RYB0" V 7380 6650 50  0000 C CNN
+F 1 "470k" V 7300 6650 50  0000 C CNN
+	1    7300 6650
 	-1   0    0    1
 $EndComp
-Text HLabel 3950 5900 0    60   BiDi ~ 0
+Text HLabel 7150 7000 0    60   BiDi ~ 0
 SMP
 $Comp
 L CSMALL CS0
 U 1 1 4FA1E0FA
-P 4100 4900
-F 0 "CS0" H 4125 4950 30  0000 L CNN
-F 1 "4.7nF" H 4125 4850 30  0000 L CNN
-	1    4100 4900
+P 7300 6000
+F 0 "CS0" H 7325 6050 30  0000 L CNN
+F 1 "4.7nF" H 7325 5950 30  0000 L CNN
+	1    7300 6000
 	1    0    0    -1
 $EndComp
@@
 L R RY0
 U 1 1 4FA1E0DF
-P 4450 4650
-F 0 "RY0" V 4530 4650 50  0000 C CNN
-F 1 "1k" V 4450 4650 50  0000 C CNN
-	1    4450 4650
-	0    -1   -1   0
-$EndComp
-Text HLabel 4000 5150 0    60   BiDi ~ 0
+P 7650 5750
+F 0 "RY0" V 7730 5750 50  0000 C CNN
+F 1 "1k" V 7650 5750 50  0000 C CNN
+	1    7650 5750
+	0    -1   -1   0
+$EndComp
+Text HLabel 7200 6250 0    60   BiDi ~ 0
 Y0B
 $Comp
 L R RX3
 U 1 1 4FA1E026
-P 2550 3750
-F 0 "RX3" V 2630 3750 50  0000 C CNN
-F 1 "1k" V 2550 3750 50  0000 C CNN
-	1    2550 3750
+P 5750 4850
+F 0 "RX3" V 5830 4850 50  0000 C CNN
+F 1 "1k" V 5750 4850 50  0000 C CNN
+	1    5750 4850
 	0    -1   -1   0
 $EndComp
@@
 L R RX2
 U 1 1 4FA1E01D
-P 2550 3050
-F 0 "RX2" V 2630 3050 50  0000 C CNN
-F 1 "1k" V 2550 3050 50  0000 C CNN
-	1    2550 3050
+P 5750 4150
+F 0 "RX2" V 5830 4150 50  0000 C CNN
+F 1 "1k" V 5750 4150 50  0000 C CNN
+	1    5750 4150
 	0    -1   -1   0
 $EndComp
@@
 L R RX1
 U 1 1 4FA1E019
-P 2550 2350
-F 0 "RX1" V 2630 2350 50  0000 C CNN
-F 1 "1k" V 2550 2350 50  0000 C CNN
-	1    2550 2350
+P 5750 3450
+F 0 "RX1" V 5830 3450 50  0000 C CNN
+F 1 "1k" V 5750 3450 50  0000 C CNN
+	1    5750 3450
 	0    -1   -1   0
 $EndComp
@@
 L R RX0
 U 1 1 4FA1E001
-P 2550 1650
-F 0 "RX0" V 2630 1650 50  0000 C CNN
-F 1 "1k" V 2550 1650 50  0000 C CNN
-	1    2550 1650
-	0    -1   -1   0
-$EndComp
-Text HLabel 4000 4650 0    60   BiDi ~ 0
+P 5750 2750
+F 0 "RX0" V 5830 2750 50  0000 C CNN
+F 1 "1k" V 5750 2750 50  0000 C CNN
+	1    5750 2750
+	0    -1   -1   0
+$EndComp
+Text HLabel 7200 5750 0    60   BiDi ~ 0
 Y0A
-Text HLabel 2200 3750 0    60   BiDi ~ 0
+Text HLabel 5400 4850 0    60   BiDi ~ 0
 X3
-Text HLabel 2200 3050 0    60   BiDi ~ 0
+Text HLabel 5400 4150 0    60   BiDi ~ 0
 X2
-Text HLabel 2200 2350 0    60   BiDi ~ 0
+Text HLabel 5400 3450 0    60   BiDi ~ 0
 X1
-Text HLabel 2200 1650 0    60   BiDi ~ 0
+Text HLabel 5400 2750 0    60   BiDi ~ 0
 X0
 $EndSCHEMATC
