File: Pong.0_Test/Hardware/Pong.0_Test_Display.sch (KiCad schematic (older format))
At the start: 47 parts

Commit message: Updated Schematic and Project Log
Parts:
- renumbered R7 to R23, R8 to R24, R9 to R25
Changed lines of the file:
@@
-EESchema Schematic File Version 2  date 5/11/2012 8:16:04 PM
+EESchema Schematic File Version 2  date 6/2/2012 2:18:36 PM
 LIBS:power
 LIBS:device
@@
 Sheet 3 3
 Title "Pong.0 Test Display"
-Date "12 may 2012"
+Date "2 jun 2012"
 Rev "1.0"
 Comp "Projects and Stuff LLC"
@@
 6E 56 52 49 51 4E 59 71 7E 65 C5 4D 0F AF 00 BF F6 21 9D BA 45 88 9C 00 16 00 C0 66 90 E0 00 00
 AC 42 3B 38 00 00 AB 90 E0 00 00 AC 42 82 03 00 B0 EA FF 00 E3 76 B5 A7 81 B6 BC 08 00 00 00 00
-49 45 4E 44 AE 42 60 82 B3 $EndBitmap
+49 45 4E 44 AE 42 60 82 8C $EndBitmap
 EndData
 $EndBitmap
@@
 $EndComp
 $Comp
-L GND #PWR019
+L GND #PWR61
 U 1 1 4FA5DCE6
 P 15100 8850
-F 0 "#PWR019" H 15100 8850 30  0001 C CNN
+F 0 "#PWR61" H 15100 8850 30  0001 C CNN
 F 1 "GND" H 15100 8780 30  0001 C CNN
 	1    15100 8850
@@
 $EndComp
 $Comp
-L GND #PWR020
+L GND #PWR60
 U 1 1 4FA5DCB0
 P 14900 5650
-F 0 "#PWR020" H 14900 5650 30  0001 C CNN
+F 0 "#PWR60" H 14900 5650 30  0001 C CNN
 F 1 "GND" H 14900 5580 30  0001 C CNN
 	1    14900 5650
@@
 $EndComp
 $Comp
-L GND #PWR021
+L GND #PWR59
 U 1 1 4FA5DC8B
 P 14800 1550
-F 0 "#PWR021" H 14800 1550 30  0001 C CNN
+F 0 "#PWR59" H 14800 1550 30  0001 C CNN
 F 1 "GND" H 14800 1480 30  0001 C CNN
 	1    14800 1550
@@
 $EndComp
 $Comp
-L GND #PWR022
+L GND #PWR56
 U 1 1 4FA53D20
 P 13150 1550
-F 0 "#PWR022" H 13150 1550 30  0001 C CNN
+F 0 "#PWR56" H 13150 1550 30  0001 C CNN
 F 1 "GND" H 13150 1480 30  0001 C CNN
 	1    13150 1550
@@
 $EndComp
 $Comp
-L GND #PWR023
+L GND #PWR53
 U 1 1 4FA53D1F
 P 11500 1550
-F 0 "#PWR023" H 11500 1550 30  0001 C CNN
+F 0 "#PWR53" H 11500 1550 30  0001 C CNN
 F 1 "GND" H 11500 1480 30  0001 C CNN
 	1    11500 1550
@@
 $EndComp
 $Comp
-L GND #PWR024
+L GND #PWR47
 U 1 1 4FA53D0F
 P 8200 1550
-F 0 "#PWR024" H 8200 1550 30  0001 C CNN
+F 0 "#PWR47" H 8200 1550 30  0001 C CNN
 F 1 "GND" H 8200 1480 30  0001 C CNN
 	1    8200 1550
@@
 $EndComp
 $Comp
-L GND #PWR025
+L GND #PWR50
 U 1 1 4FA53D0E
 P 9850 1550
-F 0 "#PWR025" H 9850 1550 30  0001 C CNN
+F 0 "#PWR50" H 9850 1550 30  0001 C CNN
 F 1 "GND" H 9850 1480 30  0001 C CNN
 	1    9850 1550
@@
 $EndComp
 $Comp
-L GND #PWR026
+L GND #PWR44
 U 1 1 4FA53CFE
 P 6550 1550
-F 0 "#PWR026" H 6550 1550 30  0001 C CNN
+F 0 "#PWR44" H 6550 1550 30  0001 C CNN
 F 1 "GND" H 6550 1480 30  0001 C CNN
 	1    6550 1550
@@
 $EndComp
 $Comp
-L GND #PWR027
+L GND #PWR41
 U 1 1 4FA53CED
 P 4900 1550
-F 0 "#PWR027" H 4900 1550 30  0001 C CNN
+F 0 "#PWR41" H 4900 1550 30  0001 C CNN
 F 1 "GND" H 4900 1480 30  0001 C CNN
 	1    4900 1550
@@
 $EndComp
 $Comp
-L GND #PWR028
+L GND #PWR42
 U 1 1 4FA53CDE
 P 5000 5650
-F 0 "#PWR028" H 5000 5650 30  0001 C CNN
+F 0 "#PWR42" H 5000 5650 30  0001 C CNN
 F 1 "GND" H 5000 5580 30  0001 C CNN
 	1    5000 5650
@@
 $EndComp
 $Comp
-L GND #PWR029
+L GND #PWR58
 U 1 1 4FA53465
 P 13450 8850
-F 0 "#PWR029" H 13450 8850 30  0001 C CNN
+F 0 "#PWR58" H 13450 8850 30  0001 C CNN
 F 1 "GND" H 13450 8780 30  0001 C CNN
 	1    13450 8850
@@
 $EndComp
 $Comp
-L GND #PWR030
+L GND #PWR55
 U 1 1 4FA53453
 P 11800 8850
-F 0 "#PWR030" H 11800 8850 30  0001 C CNN
+F 0 "#PWR55" H 11800 8850 30  0001 C CNN
 F 1 "GND" H 11800 8780 30  0001 C CNN
 	1    11800 8850
@@
 $EndComp
 $Comp
-L GND #PWR031
+L GND #PWR52
 U 1 1 4FA5344B
 P 10150 8850
-F 0 "#PWR031" H 10150 8850 30  0001 C CNN
+F 0 "#PWR52" H 10150 8850 30  0001 C CNN
 F 1 "GND" H 10150 8780 30  0001 C CNN
 	1    10150 8850
@@
 $EndComp
 $Comp
-L GND #PWR032
+L GND #PWR49
 U 1 1 4FA53441
 P 8500 8850
-F 0 "#PWR032" H 8500 8850 30  0001 C CNN
+F 0 "#PWR49" H 8500 8850 30  0001 C CNN
 F 1 "GND" H 8500 8780 30  0001 C CNN
 	1    8500 8850
@@
 $EndComp
 $Comp
-L GND #PWR033
+L GND #PWR43
 U 1 1 4FA53436
 P 5200 8850
-F 0 "#PWR033" H 5200 8850 30  0001 C CNN
+F 0 "#PWR43" H 5200 8850 30  0001 C CNN
 F 1 "GND" H 5200 8780 30  0001 C CNN
 	1    5200 8850
@@
 NoConn ~ 2600 2900
 $Comp
-L GND #PWR034
+L GND #PWR40
 U 1 1 4FA5311D
 P 1500 7200
-F 0 "#PWR034" H 1500 7200 30  0001 C CNN
+F 0 "#PWR40" H 1500 7200 30  0001 C CNN
 F 1 "GND" H 1500 7130 30  0001 C CNN
 	1    1500 7200
@@
 $EndComp
 $Comp
-L GND #PWR035
+L GND #PWR37
 U 1 1 4FA5311C
 P 1250 7200
-F 0 "#PWR035" H 1250 7200 30  0001 C CNN
+F 0 "#PWR37" H 1250 7200 30  0001 C CNN
 F 1 "GND" H 1250 7130 30  0001 C CNN
 	1    1250 7200
@@
 NoConn ~ 2600 7500
 $Comp
-L R R9
+L R R25
 U 1 1 4FA53119
 P 950 7650
-F 0 "R9" V 1030 7650 50  0000 C CNN
+F 0 "R25" V 1030 7650 50  0000 C CNN
 F 1 "22k" V 950 7650 50  0000 C CNN
 	1    950  7650
@@
 GND
 $Comp
-L R R8
+L R R24
 U 1 1 4FA5310A
 P 950 4650
-F 0 "R8" V 1030 4650 50  0000 C CNN
+F 0 "R24" V 1030 4650 50  0000 C CNN
 F 1 "22k" V 950 4650 50  0000 C CNN
 	1    950  4650
@@
 $EndComp
 $Comp
-L GND #PWR036
+L GND #PWR36
 U 1 1 4FA53107
 P 1250 4200
-F 0 "#PWR036" H 1250 4200 30  0001 C CNN
+F 0 "#PWR36" H 1250 4200 30  0001 C CNN
 F 1 "GND" H 1250 4130 30  0001 C CNN
 	1    1250 4200
@@
 $EndComp
 $Comp
-L GND #PWR037
+L GND #PWR39
 U 1 1 4FA53106
 P 1500 4200
-F 0 "#PWR037" H 1500 4200 30  0001 C CNN
+F 0 "#PWR39" H 1500 4200 30  0001 C CNN
 F 1 "GND" H 1500 4130 30  0001 C CNN
 	1    1500 4200
@@
 $EndComp
 $Comp
-L GND #PWR038
+L GND #PWR57
 U 1 1 4FA1F5DE
 P 13250 5650
-F 0 "#PWR038" H 13250 5650 30  0001 C CNN
+F 0 "#PWR57" H 13250 5650 30  0001 C CNN
 F 1 "GND" H 13250 5580 30  0001 C CNN
 	1    13250 5650
@@
 $EndComp
 $Comp
-L GND #PWR039
+L GND #PWR54
 U 1 1 4FA1F5DC
 P 11600 5650
-F 0 "#PWR039" H 11600 5650 30  0001 C CNN
+F 0 "#PWR54" H 11600 5650 30  0001 C CNN
 F 1 "GND" H 11600 5580 30  0001 C CNN
 	1    11600 5650
@@
 $EndComp
 $Comp
-L GND #PWR040
+L GND #PWR48
 U 1 1 4FA1F5D7
 P 8300 5650
-F 0 "#PWR040" H 8300 5650 30  0001 C CNN
+F 0 "#PWR48" H 8300 5650 30  0001 C CNN
 F 1 "GND" H 8300 5580 30  0001 C CNN
 	1    8300 5650
@@
 $EndComp
 $Comp
-L GND #PWR041
+L GND #PWR51
 U 1 1 4FA1F5D5
 P 9950 5650
-F 0 "#PWR041" H 9950 5650 30  0001 C CNN
+F 0 "#PWR51" H 9950 5650 30  0001 C CNN
 F 1 "GND" H 9950 5580 30  0001 C CNN
 	1    9950 5650
@@
 $EndComp
 $Comp
-L GND #PWR042
+L GND #PWR45
 U 1 1 4FA1F5D3
 P 6650 5650
-F 0 "#PWR042" H 6650 5650 30  0001 C CNN
+F 0 "#PWR45" H 6650 5650 30  0001 C CNN
 F 1 "GND" H 6650 5580 30  0001 C CNN
 	1    6650 5650
@@
 $EndComp
 $Comp
-L GND #PWR043
+L GND #PWR46
 U 1 1 4FA1F5CD
 P 6850 8850
-F 0 "#PWR043" H 6850 8850 30  0001 C CNN
+F 0 "#PWR46" H 6850 8850 30  0001 C CNN
 F 1 "GND" H 6850 8780 30  0001 C CNN
 	1    6850 8850
@@
 $EndComp
 $Comp
-L GND #PWR044
+L GND #PWR38
 U 1 1 4FA1F458
 P 1500 1200
-F 0 "#PWR044" H 1500 1200 30  0001 C CNN
+F 0 "#PWR38" H 1500 1200 30  0001 C CNN
 F 1 "GND" H 1500 1130 30  0001 C CNN
 	1    1500 1200
@@
 $EndComp
 $Comp
-L GND #PWR045
+L GND #PWR35
 U 1 1 4FA1F455
 P 1250 1200
-F 0 "#PWR045" H 1250 1200 30  0001 C CNN
+F 0 "#PWR35" H 1250 1200 30  0001 C CNN
 F 1 "GND" H 1250 1130 30  0001 C CNN
 	1    1250 1200
@@
 VIN
 $Comp
-L R R7
+L R R23
 U 1 1 4FA1E852
 P 950 1650
-F 0 "R7" V 1030 1650 50  0000 C CNN
+F 0 "R23" V 1030 1650 50  0000 C CNN
 F 1 "22k" V 950 1650 50  0000 C CNN
 	1    950  1650
