File: Pong.0_Test/Hardware/Pong.0_Test_Display.sch (KiCad schematic (older format))
At the start: 47 parts

Commit message: Cleaned up schematics and corrected crystal load capacitor calculation error (should be 36pF vice 9pF)
Parts:
- C26: renamed from C12; value .1uF -> 0.1uF
- C27: renamed from C13; value .1uF -> 0.1uF
- C28: renamed from C14; value .1uF -> 0.1uF
- C32: renamed from C18; value .1uF -> 0.1uF
- C33: renamed from C19; value .1uF -> 0.1uF
- C34: renamed from C20; value .1uF -> 0.1uF
- C35: renamed from C21; value .1uF -> 0.1uF
- C36: renamed from C22; value .1uF -> 0.1uF
- C37: renamed from C23; value .1uF -> 0.1uF
- C38: renamed from C24; value .1uF -> 0.1uF
- C39: renamed from C25; value .1uF -> 0.1uF
- C40: renamed from C26; value .1uF -> 0.1uF
- C41: renamed from C27; value .1uF -> 0.1uF
- C42: renamed from C28; value .1uF -> 0.1uF
- C43: renamed from C29; value .1uF -> 0.1uF
- C44: renamed from C30; value .1uF -> 0.1uF
- C45: renamed from C31; value .1uF -> 0.1uF
- C46: renamed from C32; value .1uF -> 0.1uF
- C47: renamed from C33; value .1uF -> 0.1uF
- C48: renamed from C34; value .1uF -> 0.1uF
- C49: renamed from C35; value .1uF -> 0.1uF
- C50: renamed from C36; value .1uF -> 0.1uF
- C51: renamed from C37; value .1uF -> 0.1uF
- C52: renamed from C38; value .1uF -> 0.1uF
- renumbered C15 to C29, C16 to C30, C17 to C31, R23 to R44, R24 to R45, R25 to R46
Connections:
- wire segments 363 -> 369
Other:
- note added: "Place 0.1uF Caps closest to\nthe chips for better decoupling."
- moved on the sheet: R44, R45, R46
