File: Pong.0_Test/Hardware/Pong.0_Test.sch (KiCad schematic (older format))
At the start: 42 parts, among them IC1 ATMEGA644P-A, J1 DC, J2 USBMICRO-B, P1 ISP, SW1 SPST, X1 20 MHz

Commit message: Updated Slider and Project Log
Connections:
- wire segments 158 -> 161
Other:
- note added: "ISP Header"
- note added: "Power Block"

Commit message: Cleaned up schematics and added footprint column to BOM. Yet to be populated
Parts:
- BT1: value 7.2VDC -> 7.4VDC
Other:
- note added: "Layout Notes:\n1) Place the .1uF caps as close to the input power pins as possible\n2) UU00 through UU19 can be negated by using the pullup resistors on the associated IO pins of the AVR"

Commit message: Updated Schematics with LED indicators and cleanup and updated Project Log
Parts:
- added P3: CONN_10X2, symbol CONN_10X2
Connections:
- wire segments 161 -> 180
Other:
- note added: "Layout Notes:\n1) Place the .1uF caps as close to the input power pins as possible\n2) UU00 through UU19 are unused in this test device, but can be accessed at header P3"
- note removed: "Layout Notes:\n1) Place the .1uF caps as close to the input power pins as possible\n2) UU00 through UU19 can be negated by using the pullup resistors on the associated IO pins of the AVR"

Commit message: Cleaned up schematics and corrected crystal load capacitor calculation error (should be 36pF vice 9pF)
Parts:
- added C10: 33uF, symbol CSMALL
- C1: value .1uF -> 0.1uF
- C11: renamed from C4; value 8pF -> 36pF
- C12: renamed from C5; value 8pF -> 36pF
- C2: value .1uF -> 10uF
- C3: renamed from C6; value .1uF -> 0.1uF
- C4: renamed from C3; value 10uF -> 0.1uF
- C5: renamed from C8; value .1uF -> 0.1uF
- C6: renamed from C7; value .1uF -> 0.1uF
- C7: renamed from C11; value .1uF -> 0.1uF
- C8: renamed from C9; value 10uF -> 0.1uF
- C9: renamed from C10; value .1uF -> 10uF
- renumbered P3 to P2, R3 to R2, R4 to R3, R5 to R4, R6 to R5, R7 to R6, R8 to R7, R9 to R8, R2 to R9
Connections:
- net labels added: XTAL1_1, XTAL1_2
- net labels removed: +5V
- wire segments 180 -> 184
Other:
- note added: "Crystal and Load Caps"
- note added: "Layout Notes:\n1) Place the 0.1uF caps as close to the input power pins as possible\n2) UU00 through UU19 are unused in this test device, but can be accessed at header P3"
- note removed: "Layout Notes:\n1) Place the .1uF caps as close to the input power pins as possible\n2) UU00 through UU19 are unused in this test device, but can be accessed at header P3"
- moved on the sheet: J1, P1, R9, X1

Commit message: Added 2 buttons and continued organizing PCB.
Parts:
- added C53, C54, C55, C56: 0.1uF, symbol CSMALL
- added S2, S3: TL3315NF160Q, symbol TL3315NF160Q
- R21, R22: value 10K -> 10k
Connections:
- wire segments 184 -> 208
Other:
- moved on the sheet: R9
