File: Pong.0_Test/Hardware/Pong.0_Test_Sensors.sch (KiCad schematic (older format))
At the start: 11 parts, among them X0Y0 CAPSENSOR, X1Y0 CAPSENSOR, X2Y0 CAPSENSOR, X3Y0 CAPSENSOR

Commit message: Cleaned up schematics and corrected crystal load capacitor calculation error (should be 36pF vice 9pF)
Parts:
- renumbered CS0 to CS1, RX0 to RX1, RX1 to RX2, RX2 to RX3, RX3 to RX4, RY0 to RY1, RYB0 to RYB1, X0Y0 to X0Y1, X1Y0 to X1Y1, X2Y0 to X2Y1, X3Y0 to X3Y1
Changed lines of the file:
@@
-EESchema Schematic File Version 2  date 9/11/2012 10:09:55 PM
+EESchema Schematic File Version 2  date 1/1/2013 2:06:25 AM
 LIBS:power
 LIBS:device
@@
 Sheet 2 4
 Title "Pong.0 Test Board"
-Date "12 sep 2012"
+Date "1 jan 2013"
 Rev "1.0"
 Comp "Projects and Stuff LLC"
@@
 6E 56 52 49 51 4E 59 71 7E 65 C5 4D 0F AF 00 BF F6 21 9D BA 45 88 9C 00 16 00 C0 66 90 E0 00 00
 AC 42 3B 38 00 00 AB 90 E0 00 00 AC 42 82 03 00 B0 EA FF 00 E3 76 B5 A7 81 B6 BC 08 00 00 00 00
-49 45 4E 44 AE 42 60 82 75 $EndBitmap
+49 45 4E 44 AE 42 60 82 3E $EndBitmap
 EndData
 $EndBitmap
@@
 VREF
 $Comp
-L CAPSENSOR X3Y0
+L CAPSENSOR X3Y1
 U 1 1 4FA1E531
 P 6350 4850
-F 0 "X3Y0" H 6310 4970 60  0000 C CNN
+F 0 "X3Y1" H 6310 4970 60  0000 C CNN
 F 1 "CAPSENSOR" V 6460 4840 40  0000 C CNN
 	1    6350 4850
@@
 $EndComp
 $Comp
-L CAPSENSOR X2Y0
+L CAPSENSOR X2Y1
 U 1 1 4FA1E52F
 P 6350 4150
-F 0 "X2Y0" H 6310 4270 60  0000 C CNN
+F 0 "X2Y1" H 6310 4270 60  0000 C CNN
 F 1 "CAPSENSOR" V 6460 4140 40  0000 C CNN
 	1    6350 4150
@@
 $EndComp
 $Comp
-L CAPSENSOR X1Y0
+L CAPSENSOR X1Y1
 U 1 1 4FA1E528
 P 6350 3450
-F 0 "X1Y0" H 6310 3570 60  0000 C CNN
+F 0 "X1Y1" H 6310 3570 60  0000 C CNN
 F 1 "CAPSENSOR" V 6460 3440 40  0000 C CNN
 	1    6350 3450
@@
 $EndComp
 $Comp
-L CAPSENSOR X0Y0
+L CAPSENSOR X0Y1
 U 1 1 4FA1E50B
 P 6350 2750
-F 0 "X0Y0" H 6310 2870 60  0000 C CNN
+F 0 "X0Y1" H 6310 2870 60  0000 C CNN
 F 1 "CAPSENSOR" V 6460 2740 40  0000 C CNN
 	1    6350 2750
@@
 $EndComp
 $Comp
-L R RYB0
+L R RYB1
 U 1 1 4FA1E1CF
 P 7300 6650
-F 0 "RYB0" V 7380 6650 50  0000 C CNN
+F 0 "RYB1" V 7380 6650 50  0000 C CNN
 F 1 "470k" V 7300 6650 50  0000 C CNN
 	1    7300 6650
@@
 SMP
 $Comp
-L CSMALL CS0
+L CSMALL CS1
 U 1 1 4FA1E0FA
 P 7300 6000
-F 0 "CS0" H 7325 6050 30  0000 L CNN
+F 0 "CS1" H 7325 6050 30  0000 L CNN
 F 1 "4.7nF" H 7325 5950 30  0000 L CNN
 	1    7300 6000
@@
 $EndComp
 $Comp
-L R RY0
+L R RY1
 U 1 1 4FA1E0DF
 P 7650 5750
-F 0 "RY0" V 7730 5750 50  0000 C CNN
+F 0 "RY1" V 7730 5750 50  0000 C CNN
 F 1 "1k" V 7650 5750 50  0000 C CNN
 	1    7650 5750
@@
 Y0B
 $Comp
-L R RX3
+L R RX4
 U 1 1 4FA1E026
 P 5750 4850
-F 0 "RX3" V 5830 4850 50  0000 C CNN
+F 0 "RX4" V 5830 4850 50  0000 C CNN
 F 1 "1k" V 5750 4850 50  0000 C CNN
 	1    5750 4850
@@
 $EndComp
 $Comp
-L R RX2
+L R RX3
 U 1 1 4FA1E01D
 P 5750 4150
-F 0 "RX2" V 5830 4150 50  0000 C CNN
+F 0 "RX3" V 5830 4150 50  0000 C CNN
 F 1 "1k" V 5750 4150 50  0000 C CNN
 	1    5750 4150
@@
 $EndComp
 $Comp
-L R RX1
+L R RX2
 U 1 1 4FA1E019
 P 5750 3450
-F 0 "RX1" V 5830 3450 50  0000 C CNN
+F 0 "RX2" V 5830 3450 50  0000 C CNN
 F 1 "1k" V 5750 3450 50  0000 C CNN
 	1    5750 3450
@@
 $EndComp
 $Comp
-L R RX0
+L R RX1
 U 1 1 4FA1E001
 P 5750 2750
-F 0 "RX0" V 5830 2750 50  0000 C CNN
+F 0 "RX1" V 5830 2750 50  0000 C CNN
 F 1 "1k" V 5750 2750 50  0000 C CNN
 	1    5750 2750
