File: Pong.0_Test/Hardware/Pong.0_Test_Slider.sch (KiCad schematic (older format))
At the start: 27 parts, among them IC2 ATMEGA168PA-A, P2 ISP_2

Commit message: Updated Schematics with LED indicators and cleanup and updated Project Log
Parts:
- added C44, C45, C46, C47, C48, C49: CSMALL, symbol CSMALL
- added D-S1, D-S2, D-S3, D-S4, D-S5, D-S6: LED, symbol LED
- added R39, R40, R41, R42, R43, R44: 330, symbol R
Connections:
- wire segments 90 -> 127
Other:
- moved on the sheet: IC2, L2, P2

Commit message: Cleaned up schematics and corrected crystal load capacitor calculation error (should be 36pF vice 9pF)
Parts:
- added C24, C25: 36pF, symbol CSMALL
- added R23, R24: 10K, symbol R
- added X2: 20MHz, symbol CRYSTAL
- C13: renamed from C39; value .1uF -> 0.1uF
- C15: renamed from C41; value .1uF -> 0.1uF
- C16: renamed from C42; value .1uF -> 0.1uF
- C17: renamed from C44; value CSMALL -> 0.1uF
- C18: renamed from C45; value CSMALL -> 0.1uF
- C19: renamed from C46; value CSMALL -> 0.1uF
- C20: renamed from C47; value CSMALL -> 0.1uF
- C21: renamed from C48; value CSMALL -> 0.1uF
- C22: renamed from C49; value CSMALL -> 0.1uF
- renumbered C40 to C14, C43 to C23, P2 to P3, R39 to R25, R40 to R26, R41 to R27, R42 to R28, R43 to R29, R44 to R30, R26 to R31, R27 to R32, R28 to R33, R29 to R34, R30 to R35, R31 to R36, R32 to R37, R33 to R38, R34 to R39, R35 to R40, R36 to R41, R37 to R42, R38 to R43
Connections:
- net labels added: XTAL2_1
- net labels removed: XTAL1_2
- wire segments 127 -> 141
Other:
- note added: "Crystal and Load Caps"
- note added: "Place 0.1uF Caps closest to\nthe chips for better decoupling."
- note added: "These LEDs will be used to display which\nvalue is selected via the slider (1 through 6)"
- moved on the sheet: P3
