File: Hardware/Controller.sch (KiCad schematic (older format))
At the start: 12 parts

Commit message: Continued populating the schematics.
Parts:
- added C?: CSMALL, ~, symbol CSMALL
- added R? (x2): 10k, ~, symbol R
- added R? (x2): R, ~, symbol R
- added U?: R1EX24064AXXS0A, symbol R1EX24064AXXS0A
Connections:
- wire segments 75 -> 95
Other:
- note added: "64 KBit EEPROM\n8000 x 8-bit words\n32-byte page write"
- note added: "Device 8-bit address:\n1 - 0 - 1 - 0 - A0 - A1 - A2 - R/W"
- note added: "EXTERNAL EEPROM MEMORY"
- note added: "LOGIC HEADERS"
- note added: "Only one of these resisotrs should actually be populated.\nPull high for write-protect. Pull low for normal read/write."
- note added: "PDI INTERFACE"
- moved on the sheet: IC?, L?, P?

Commit message: Added new Winbond Flash Memory chip
Parts:
- removed C?: CSMALL, ~, symbol CSMALL
- removed R? (x2): 10k, ~, symbol R
- removed R? (x2): R, ~, symbol R
- removed U?: R1EX24064AXXS0A, symbol R1EX24064AXXS0A
- added C?: 0.1uF, ~, symbol CSMALL
- added U?: W25X20A, symbol W25X20A
Connections:
- wire segments 95 -> 86
Other:
- note added: "EXTERNAL FLASH MEMORY"
- note removed: "64 KBit EEPROM\n8000 x 8-bit words\n32-byte page write"
- note removed: "Device 8-bit address:\n1 - 0 - 1 - 0 - A0 - A1 - A2 - R/W"
- note removed: "EXTERNAL EEPROM MEMORY"
- note removed: "Only one of these resisotrs should actually be populated.\nPull high for write-protect. Pull low for normal read/write."
Changed lines of the file:
@@
 6E 56 52 49 51 4E 59 71 7E 65 C5 4D 0F AF 00 BF F6 21 9D BA 45 88 9C 00 16 00 C0 66 90 E0 00 00
 AC 42 3B 38 00 00 AB 90 E0 00 00 AC 42 82 03 00 B0 EA FF 00 E3 76 B5 A7 81 B6 BC 08 00 00 00 00
-49 45 4E 44 AE 42 60 82 3E $EndBitmap
+49 45 4E 44 AE 42 60 82 6B $EndBitmap
 EndData
 $EndBitmap
@@
 Wire Wire Line
 	11950 2800 12000 2800
-$Comp
-L R1EX24064AXXS0A U?
-U 1 1 5235EC9A
-P 9500 4500
-F 0 "U?" H 9650 4050 60  0000 C CNN
-F 1 "R1EX24064AXXS0A" H 9500 4950 60  0000 C CNN
-F 2 "" H 9500 4500 60  0000 C CNN
-F 3 "" H 9500 4500 60  0000 C CNN
-	1    9500 4500
-	1    0    0    -1
-$EndComp
-Text Notes 9100 5150 0    60   ~ 0
-64 KBit EEPROM\n8000 x 8-bit words\n32-byte page write
-$Comp
-L R R?
-U 1 1 5235ECA9
-P 10100 3900
-F 0 "R?" V 10180 3900 40  0000 C CNN
-F 1 "10k" V 10107 3901 40  0000 C CNN
-F 2 "~" V 10030 3900 30  0000 C CNN
-F 3 "~" H 10100 3900 30  0000 C CNN
-	1    10100 3900
-	1    0    0    -1
-$EndComp
-$Comp
-L R R?
-U 1 1 5235ECBC
-P 10400 4200
-F 0 "R?" V 10480 4200 40  0000 C CNN
-F 1 "10k" V 10407 4201 40  0000 C CNN
-F 2 "~" V 10330 4200 30  0000 C CNN
-F 3 "~" H 10400 4200 30  0000 C CNN
-	1    10400 4200
-	0    -1   -1   0
-$EndComp
-Wire Wire Line
-	10050 4200 10150 4200
-Wire Wire Line
-	10100 4150 10100 4200
-Connection ~ 10100 4200
-Text Notes 10200 4000 0    60   ~ 0
-Only one of these resisotrs should actually be populated.\nPull high for write-protect. Pull low for normal read/write.
-$Comp
-L GND #PWR?
-U 1 1 5235ED79
-P 10700 4250
-F 0 "#PWR?" H 10700 4250 30  0001 C CNN
-F 1 "GND" H 10700 4180 30  0001 C CNN
-F 2 "" H 10700 4250 60  0000 C CNN
-F 3 "" H 10700 4250 60  0000 C CNN
-	1    10700 4250
-	1    0    0    -1
-$EndComp
-Wire Wire Line
-	10650 4200 10700 4200
-Wire Wire Line
-	10700 4200 10700 4250
-Wire Wire Line
-	10100 3650 10100 3600
-Text Label 10100 3600 0    60   ~ 0
-CTRL_3_3V
-$Comp
-L CSMALL C?
-U 1 1 5235F398
-P 8900 4350
-F 0 "C?" H 8925 4400 30  0000 L CNN
-F 1 "CSMALL" H 8925 4300 30  0000 L CNN
-F 2 "~" H 8900 4350 60  0000 C CNN
-F 3 "~" H 8900 4350 60  0000 C CNN
-	1    8900 4350
-	1    0    0    -1
-$EndComp
-$Comp
-L GND #PWR?
-U 1 1 5235F3A7
-P 8900 4550
-F 0 "#PWR?" H 8900 4550 30  0001 C CNN
-F 1 "GND" H 8900 4480 30  0001 C CNN
-F 2 "" H 8900 4550 60  0000 C CNN
-F 3 "" H 8900 4550 60  0000 C CNN
-	1    8900 4550
-	1    0    0    -1
-$EndComp
-Text Label 8900 3900 0    60   ~ 0
-CTRL_3_3V
-Wire Wire Line
-	8900 3900 8900 4250
-Wire Wire Line
-	8900 4200 8950 4200
-Connection ~ 8900 4200
-Wire Wire Line
-	8900 4450 8900 4550
-Wire Wire Line
-	8900 4500 8950 4500
-Connection ~ 8900 4500
-$Comp
-L R R?
-U 1 1 5235F6F2
-P 8650 4400
-F 0 "R?" V 8730 4400 40  0000 C CNN
-F 1 "R" V 8657 4401 40  0000 C CNN
-F 2 "~" V 8580 4400 30  0000 C CNN
-F 3 "~" H 8650 4400 30  0000 C CNN
-	1    8650 4400
-	1    0    0    -1
-$EndComp
-$Comp
-L R R?
-U 1 1 5235F6FD
-P 8450 4400
-F 0 "R?" V 8530 4400 40  0000 C CNN
-F 1 "R" V 8457 4401 40  0000 C CNN
-F 2 "~" V 8380 4400 30  0000 C CNN
-F 3 "~" H 8450 4400 30  0000 C CNN
-	1    8450 4400
-	1    0    0    -1
-$EndComp
-Wire Wire Line
-	8350 4700 8950 4700
-Wire Wire Line
-	8650 4700 8650 4650
-Wire Wire Line
-	8350 4800 8950 4800
-Wire Wire Line
-	8450 4800 8450 4650
-Connection ~ 8650 4700
-Connection ~ 8450 4800
-Wire Wire Line
-	8900 4100 8450 4100
-Wire Wire Line
-	8450 4100 8450 4150
-Connection ~ 8900 4100
-Wire Wire Line
-	8650 4150 8650 4100
-Connection ~ 8650 4100
-$Comp
-L GND #PWR?
-U 1 1 5235FD02
-P 10100 4850
-F 0 "#PWR?" H 10100 4850 30  0001 C CNN
-F 1 "GND" H 10100 4780 30  0001 C CNN
-F 2 "" H 10100 4850 60  0000 C CNN
-F 3 "" H 10100 4850 60  0000 C CNN
-	1    10100 4850
-	1    0    0    -1
-$EndComp
-Wire Wire Line
-	10050 4600 10100 4600
-Wire Wire Line
-	10100 4600 10100 4850
-Wire Wire Line
-	10050 4700 10100 4700
-Connection ~ 10100 4700
-Wire Wire Line
-	10050 4800 10100 4800
-Connection ~ 10100 4800
-Text Notes 10150 4700 0    60   ~ 0
-Device 8-bit address:\n1 - 0 - 1 - 0 - A0 - A1 - A2 - R/W
-Text Label 8350 4800 2    60   ~ 0
-CTRL_SCL
-Text Label 8350 4700 2    60   ~ 0
-CTRL_SDA
 Text Notes 7900 3450 0    60   ~ 12
-EXTERNAL EEPROM MEMORY
+EXTERNAL FLASH MEMORY
 Wire Notes Line
 	7850 1700 7850 5400
@@
 Text Notes 10300 1800 0    60   ~ 12
 PDI INTERFACE
+$Comp
+L W25X20A U?
+U 1 1 523B50DB
+P 10400 4500
+F 0 "U?" H 10600 4000 60  0000 C CNN
+F 1 "W25X20A" H 10300 5200 60  0000 C CNN
+F 2 "" H 10550 4300 60  0000 C CNN
+F 3 "" H 10550 4300 60  0000 C CNN
+	1    10400 4500
+	1    0    0    -1
+$EndComp
+$Comp
+L GND #PWR?
+U 1 1 523B52F0
+P 9750 4900
+F 0 "#PWR?" H 9750 4900 30  0001 C CNN
+F 1 "GND" H 9750 4830 30  0001 C CNN
+F 2 "" H 9750 4900 60  0000 C CNN
+F 3 "" H 9750 4900 60  0000 C CNN
+	1    9750 4900
+	1    0    0    -1
+$EndComp
+Wire Wire Line
+	9800 4850 9750 4850
+Wire Wire Line
+	9750 4850 9750 4900
+$Comp
+L CSMALL C?
+U 1 1 523B535A
+P 9750 4100
+F 0 "C?" H 9775 4150 30  0000 L CNN
+F 1 "0.1uF" H 9775 4050 30  0000 L CNN
+F 2 "~" H 9750 4100 60  0000 C CNN
+F 3 "~" H 9750 4100 60  0000 C CNN
+	1    9750 4100
+	1    0    0    -1
+$EndComp
+$Comp
+L GND #PWR?
+U 1 1 523B56AC
+P 9750 4250
+F 0 "#PWR?" H 9750 4250 30  0001 C CNN
+F 1 "GND" H 9750 4180 30  0001 C CNN
+F 2 "" H 9750 4250 60  0000 C CNN
+F 3 "" H 9750 4250 60  0000 C CNN
+	1    9750 4250
+	1    0    0    -1
+$EndComp
+Wire Wire Line
+	9750 4200 9750 4250
+Wire Wire Line
+	9700 3950 9800 3950
+Wire Wire Line
+	9750 3950 9750 4000
+Connection ~ 9750 3950
+Wire Wire Line
+	9800 4350 9700 4350
+Wire Wire Line
+	9800 4450 9700 4450
+Wire Wire Line
+	9800 4550 9700 4550
+Wire Wire Line
+	9800 4650 9700 4650
+Wire Wire Line
+	11000 4350 11050 4350
+Wire Wire Line
+	11000 3950 11050 3950
 $EndSCHEMATC

Commit message: Corrected Flash chip version and modified pins.
Parts:
- removed U?: W25X20A, symbol W25X20A
- added U?: W25X20CL, ~, symbol W25X20CL
- added U? (x2): 10k, ~, symbol R_SMALL
Connections:
- net labels added: CTRL_~HOLD, CTRL_~WP
- wire segments 86 -> 90
Changed lines of the file:
@@
 6E 56 52 49 51 4E 59 71 7E 65 C5 4D 0F AF 00 BF F6 21 9D BA 45 88 9C 00 16 00 C0 66 90 E0 00 00
 AC 42 3B 38 00 00 AB 90 E0 00 00 AC 42 82 03 00 B0 EA FF 00 E3 76 B5 A7 81 B6 BC 08 00 00 00 00
-49 45 4E 44 AE 42 60 82 6B $EndBitmap
+49 45 4E 44 AE 42 60 82 F8 $EndBitmap
 EndData
 $EndBitmap
@@
 PDI INTERFACE
 $Comp
-L W25X20A U?
-U 1 1 523B50DB
-P 10400 4500
-F 0 "U?" H 10600 4000 60  0000 C CNN
-F 1 "W25X20A" H 10300 5200 60  0000 C CNN
-F 2 "" H 10550 4300 60  0000 C CNN
-F 3 "" H 10550 4300 60  0000 C CNN
-	1    10400 4500
-	1    0    0    -1
-$EndComp
-$Comp
 L GND #PWR?
 U 1 1 523B52F0
@@
 Wire Wire Line
 	9800 4650 9700 4650
-Wire Wire Line
-	11000 4350 11050 4350
-Wire Wire Line
-	11000 3950 11050 3950
+$Comp
+L W25X20CL U?
+U 1 1 523B4EE3
+P 10400 4500
+F 0 "U?" H 10600 4000 60  0000 C CNN
+F 1 "W25X20CL" H 10350 5200 60  0000 C CNN
+F 2 "~" H 10550 4300 60  0000 C CNN
+F 3 "~" H 10550 4300 60  0000 C CNN
+	1    10400 4500
+	1    0    0    -1
+$EndComp
+$Comp
+L R_SMALL U?
+U 1 1 523B50F5
+P 11050 3750
+F 0 "U?" H 11090 3700 28  0000 C CNN
+F 1 "10k" H 11050 3750 22  0000 C CNN
+F 2 "~" H 11050 3750 60  0000 C CNN
+F 3 "~" H 11050 3750 60  0000 C CNN
+	1    11050 3750
+	0    -1   -1   0
+$EndComp
+$Comp
+L R_SMALL U?
+U 1 1 523B5104
+P 11800 4150
+F 0 "U?" H 11840 4100 28  0000 C CNN
+F 1 "10k" H 11800 4150 22  0000 C CNN
+F 2 "~" H 11800 4150 60  0000 C CNN
+F 3 "~" H 11800 4150 60  0000 C CNN
+	1    11800 4150
+	0    -1   -1   0
+$EndComp
+Wire Wire Line
+	11050 3950 11050 3900
+Wire Wire Line
+	11800 4350 11800 4300
+Connection ~ 11800 4350
+Connection ~ 11050 3950
+Text HLabel 11100 3950 2    60   Input ~ 0
+CTRL_~WP
+Wire Wire Line
+	11000 4350 11850 4350
+Wire Wire Line
+	11000 3950 11100 3950
+Text HLabel 11850 4350 2    60   Input ~ 0
+CTRL_~HOLD
+Text HLabel 9700 3950 0    60   Input ~ 0
+CTRL_3_3V
+Wire Wire Line
+	11050 3600 11050 3550
+Wire Wire Line
+	11800 4000 11800 3950
+Text HLabel 11050 3550 2    60   Input ~ 0
+CTRL_3_3V
+Text HLabel 11800 3950 2    60   Input ~ 0
+CTRL_3_3V
 $EndSCHEMATC
