File: Hardware/Controller.sch (KiCad schematic (older format))
At the start: 16 parts

Commit message: Updated from ATXMEGA64A4U to ATXMEGA64A3U
Parts:
- removed IC?: ATXMEGA64A4U-A, TQFP44, symbol ATXMEGA64A4U-A
- added C? (x2): 0.1uF, ~, symbol CSMALL
- added IC?: ATXMEGA64A3U-A, TQFP64, symbol ATXMEGA64A3U-A
- added P?: LOGIC_PORT_B, symbol CONN_9
Connections:
- net labels added: CTRL_MISO_1, CTRL_MISO_2, CTRL_MOSI_1, CTRL_MOSI_2, CTRL_RXD0, CTRL_SCK_1, CTRL_SCK_2, CTRL_SCL_1, CTRL_SCL_2, CTRL_SDA_1, CTRL_SDA_2, CTRL_TXD0, CTRL_XCK0, CTRL_~SS~_1, CTRL_~SS~_2, D+, D-, TCK, TDI, TDO, TMS
- net labels removed: CTRL_SCL, CTRL_SDA
- wire segments 100 -> 140
Other:
- moved on the sheet: L?, P?

Commit message: Added devices and corrected pins and labels
Parts:
- added C? (x4): 0.1uF, ~, symbol CSMALL
- added D?: LED, ~, symbol LED
- added P?: ISP, symbol CONN_3X2
- added P?: CONN_5X2, symbol CONN_5X2
- added R? (x5): 10k, ~, symbol R_SMALL
- added R?: R_SMALL, ~, symbol R_SMALL
- added SW? (x4): TEST, ~, symbol SW_PUSH
- added SW?: RESET, ~, symbol SW_PUSH
- gave numbers to parts that had none: 1
Connections:
- net labels added: CTRL_D+, CTRL_D-, CTRL_SMP, CTRL_X0, CTRL_X1, CTRL_X2, CTRL_X3, CTRL_X4, CTRL_X5, CTRL_X6, CTRL_X7, CTRL_Y0A, CTRL_Y0B, CTRL_Y1A, CTRL_Y1B, CTRL_Y2A, CTRL_Y2B, CTRL_Y3A, CTRL_Y3B, PDI_CLK, PDI_DATA, RXD, STATUS_LED, SW_TEST1, SW_TEST2, SW_TEST3, SW_TEST4, TXD, XCK, ~HOLD, ~WP
- net labels removed: CTRL_MISO, CTRL_MOSI, CTRL_RXD0, CTRL_SCK, CTRL_TXD0, CTRL_XCK0, CTRL_~HOLD, CTRL_~SS, CTRL_~WP, D+, D-, X0, X1, X2, X3, X4, X5, X6, X7, Y0A, Y0B, Y1A, Y1B, Y2A, Y2B, Y3A, Y3B
- wire segments 140 -> 198
- no-connect marks 0 -> 4
Other:
- note added: "BUTTONS"
- note added: "Ferrite Bead\nPer AVR1012\nSection 2.1"
- note added: "ISP Header for programming\nthe Flash Memory directly"
- note added: "JTAG INTERFACE"
- note added: "PDI_CLK and\n~RESET~ share\nthe same line"
- note added: "RESET CIRCUITRY"
- note added: "STATUS LED"
- moved on the sheet: P?, R?, U?

Commit message: Updated pin names
Parts:
- removed C? (x2): 0.1uF, ~, symbol CSMALL
- removed R? (x2): 10k, ~, symbol R_SMALL
- removed SW? (x2): TEST, ~, symbol SW_PUSH
Connections:
- net labels added: CTRL_AREF, CTRL_GDO0, CTRL_GDO2
- net labels removed: SW_TEST3, SW_TEST4
- wire segments 198 -> 185
Other:
- note added: "(Used for CC2500 GDO0)"
- moved on the sheet: D?, IC?, L?, P?, R?, SW?, U?

Commit message: Finalized pin placement/layout
Parts:
- removed C?: 10uF, ~, symbol CSMALL
- removed C?: 0.1uF, ~, symbol CSMALL
- removed R?: 10k, ~, symbol R_SMALL
- removed SW?: TEST, ~, symbol SW_PUSH
- added C?: 10uF, ~, symbol CPOLSMALL
Connections:
- net labels added: CTRL_INT, CTRL_IRQ, CTRL_RSTN, CTRL_~SS~2_2
- net labels removed: SW_TEST2
- wire segments 185 -> 174
Changed lines of the file:
@@
 Sheet 7 7
 Title "Pong.0"
-Date "25 sep 2013"
+Date "26 sep 2013"
 Rev "0.3"
 Comp "Projects and Stuff LLC"
@@
 F 3 "" H 5700 2400 60  0000 C CNN
 	1    5700 2400
-	1    0    0    -1
-$EndComp
-$Comp
-L CSMALL C?
-U 1 1 522DE6D0
-P 3050 2450
-F 0 "C?" H 3075 2500 30  0000 L CNN
-F 1 "10uF" H 3075 2400 30  0000 L CNN
-F 2 "~" H 3050 2450 60  0000 C CNN
-F 3 "~" H 3050 2450 60  0000 C CNN
-	1    3050 2450
 	1    0    0    -1
 $EndComp
@@
 6E 56 52 49 51 4E 59 71 7E 65 C5 4D 0F AF 00 BF F6 21 9D BA 45 88 9C 00 16 00 C0 66 90 E0 00 00
 AC 42 3B 38 00 00 AB 90 E0 00 00 AC 42 82 03 00 B0 EA FF 00 E3 76 B5 A7 81 B6 BC 08 00 00 00 00
-49 45 4E 44 AE 42 60 82 E3 $EndBitmap
+49 45 4E 44 AE 42 60 82 79 $EndBitmap
 EndData
 $EndBitmap
@@
 	1    0    0    -1
 $EndComp
-$Comp
-L CSMALL C?
-U 1 1 5242E604
-P 10100 7650
-F 0 "C?" H 10125 7700 30  0000 L CNN
-F 1 "0.1uF" H 10125 7600 30  0000 L CNN
-F 2 "~" H 10100 7650 60  0000 C CNN
-F 3 "~" H 10100 7650 60  0000 C CNN
-	1    10100 7650
-	1    0    0    -1
-$EndComp
-$Comp
-L SW_PUSH SW?
-U 1 1 5242E60A
-P 9900 7750
-F 0 "SW?" H 10050 7860 50  0000 C CNN
-F 1 "TEST" H 9900 7670 50  0000 C CNN
-F 2 "~" H 9900 7750 60  0000 C CNN
-F 3 "~" H 9900 7750 60  0000 C CNN
-	1    9900 7750
-	0    -1   -1   0
-$EndComp
-$Comp
-L R_SMALL R?
-U 1 1 5242E610
-P 10000 7150
-F 0 "R?" H 10040 7100 28  0000 C CNN
-F 1 "10k" H 10000 7150 22  0000 C CNN
-F 2 "~" H 10000 7150 60  0000 C CNN
-F 3 "~" H 10000 7150 60  0000 C CNN
-	1    10000 7150
-	0    -1   -1   0
-$EndComp
-$Comp
-L GND #PWR088
-U 1 1 5242E620
-P 10000 8150
-F 0 "#PWR088" H 10000 8150 30  0001 C CNN
-F 1 "GND" H 10000 8080 30  0001 C CNN
-F 2 "" H 10000 8150 60  0000 C CNN
-F 3 "" H 10000 8150 60  0000 C CNN
-	1    10000 8150
-	1    0    0    -1
-$EndComp
-Text Label 9800 7350 2    60   ~ 0
-SW_TEST2
-Text HLabel 10000 6950 0    60   Input ~ 0
-CTRL_3_3V
 Text Notes 7900 6700 0    60   ~ 12
 BUTTONS
@@
 Text Label 6900 4300 2    60   ~ 0
 TDI
-Text Label 6900 4850 2    60   ~ 0
+Text Label 2600 5500 0    60   ~ 0
 SW_TEST1
-Text Label 6900 4950 2    60   ~ 0
-SW_TEST2
 Text Label 8000 3650 0    60   ~ 0
 TMS
@@
 	5750 4300 6900 4300
 Wire Wire Line
-	5750 4850 6900 4850
-Wire Wire Line
-	5750 4950 6900 4950
+	2600 5500 3750 5500
 Wire Wire Line
 	5750 4650 5800 4650
@@
 	5750 5800 6900 5800
 Wire Wire Line
-	3700 5500 3750 5500
-Wire Wire Line
-	3700 5600 3750 5600
+	5750 4850 5800 4850
+Wire Wire Line
+	5750 4950 5800 4950
 Wire Wire Line
 	3700 5700 3750 5700
@@
 Wire Notes Line
 	14500 1600 14500 8300
-Wire Wire Line
-	9900 7450 9900 7400
-Wire Wire Line
-	9900 7400 10100 7400
-Wire Wire Line
-	10000 7300 10000 7400
-Wire Wire Line
-	10100 7400 10100 7550
-Connection ~ 10000 7400
-Wire Wire Line
-	9900 8050 9900 8100
-Wire Wire Line
-	9900 8100 10100 8100
-Wire Wire Line
-	10100 8100 10100 7750
-Wire Wire Line
-	10000 8100 10000 8150
-Connection ~ 10000 8100
-Wire Wire Line
-	10000 7350 9800 7350
-Connection ~ 10000 7350
-Wire Wire Line
-	10000 7000 10000 6950
 Wire Notes Line
 	14500 8300 7850 8300
@@
 Wire Wire Line
 	5750 4500 6900 4500
+Text HLabel 3700 4950 0    60   Input ~ 0
+CTRL_~SS~2_2
+Text HLabel 5800 4850 2    60   Input ~ 0
+CTRL_INT
+Text HLabel 5800 4950 2    60   Input ~ 0
+CTRL_IRQ
+$Comp
+L CPOLSMALL C?
+U 1 1 524465B9
+P 3050 2500
+F 0 "C?" H 3100 2600 28  0000 C CNN
+F 1 "10uF" H 3075 2475 28  0000 L CNN
+F 2 "~" H 3050 2500 60  0000 C CNN
+F 3 "~" H 3050 2500 60  0000 C CNN
+	1    3050 2500
+	1    0    0    -1
+$EndComp
+Text HLabel 3750 5600 0    60   Input ~ 0
+CTRL_RSTN
 $EndSCHEMATC

Commit message: Annotated Schematics
Parts:
- gave numbers to parts that had none: 28

Commit message: Made corrections based on ERC results
Connections:
- no-connect marks 4 -> 6
Changed lines of the file:
@@
 $EndComp
 $Comp
-L GND #PWR72
+L GND #PWR066
 U 1 1 522DE695
 P 3800 2600
-F 0 "#PWR72" H 3800 2600 30  0001 C CNN
+F 0 "#PWR066" H 3800 2600 30  0001 C CNN
 F 1 "GND" H 3800 2530 30  0001 C CNN
 F 2 "" H 3800 2600 60  0000 C CNN
@@
 $EndComp
 $Comp
-L GND #PWR73
+L GND #PWR067
 U 1 1 522DE69B
 P 4000 2600
-F 0 "#PWR73" H 4000 2600 30  0001 C CNN
+F 0 "#PWR067" H 4000 2600 30  0001 C CNN
 F 1 "GND" H 4000 2530 30  0001 C CNN
 F 2 "" H 4000 2600 60  0000 C CNN
@@
 $EndComp
 $Comp
-L GND #PWR74
+L GND #PWR068
 U 1 1 522DE6A1
 P 4200 2600
-F 0 "#PWR74" H 4200 2600 30  0001 C CNN
+F 0 "#PWR068" H 4200 2600 30  0001 C CNN
 F 1 "GND" H 4200 2530 30  0001 C CNN
 F 2 "" H 4200 2600 60  0000 C CNN
@@
 $EndComp
 $Comp
-L GND #PWR81
+L GND #PWR069
 U 1 1 522DE6A7
 P 5700 2400
-F 0 "#PWR81" H 5700 2400 30  0001 C CNN
+F 0 "#PWR069" H 5700 2400 30  0001 C CNN
 F 1 "GND" H 5700 2330 30  0001 C CNN
 F 2 "" H 5700 2400 60  0000 C CNN
@@
 $EndComp
 $Comp
-L GND #PWR69
+L GND #PWR070
 U 1 1 522DE6D6
 P 3050 2600
-F 0 "#PWR69" H 3050 2600 30  0001 C CNN
+F 0 "#PWR070" H 3050 2600 30  0001 C CNN
 F 1 "GND" H 3050 2530 30  0001 C CNN
 F 2 "" H 3050 2600 60  0000 C CNN
@@
 $EndComp
 $Comp
-L GND #PWR82
+L GND #PWR071
 U 1 1 522DE6F2
 P 5900 2400
-F 0 "#PWR82" H 5900 2400 30  0001 C CNN
+F 0 "#PWR071" H 5900 2400 30  0001 C CNN
 F 1 "GND" H 5900 2330 30  0001 C CNN
 F 2 "" H 5900 2400 60  0000 C CNN
@@
 6E 56 52 49 51 4E 59 71 7E 65 C5 4D 0F AF 00 BF F6 21 9D BA 45 88 9C 00 16 00 C0 66 90 E0 00 00
 AC 42 3B 38 00 00 AB 90 E0 00 00 AC 42 82 03 00 B0 EA FF 00 E3 76 B5 A7 81 B6 BC 08 00 00 00 00
-49 45 4E 44 AE 42 60 82 AF $EndBitmap
+49 45 4E 44 AE 42 60 82 B4 $EndBitmap
 EndData
 $EndBitmap
@@
 $EndComp
 $Comp
-L GND #PWR83
+L GND #PWR072
 U 1 1 522E22DB
 P 8700 4400
-F 0 "#PWR83" H 8700 4400 30  0001 C CNN
+F 0 "#PWR072" H 8700 4400 30  0001 C CNN
 F 1 "GND" H 8700 4330 30  0001 C CNN
 F 2 "" H 8700 4400 60  0000 C CNN
@@
 $EndComp
 $Comp
-L GND #PWR86
+L GND #PWR073
 U 1 1 522E2335
 P 10200 4400
-F 0 "#PWR86" H 10200 4400 30  0001 C CNN
+F 0 "#PWR073" H 10200 4400 30  0001 C CNN
 F 1 "GND" H 10200 4330 30  0001 C CNN
 F 2 "" H 10200 4400 60  0000 C CNN
@@
 PDI INTERFACE
 $Comp
-L GND #PWR88
+L GND #PWR074
 U 1 1 523B52F0
 P 11450 6150
-F 0 "#PWR88" H 11450 6150 30  0001 C CNN
+F 0 "#PWR074" H 11450 6150 30  0001 C CNN
 F 1 "GND" H 11450 6080 30  0001 C CNN
 F 2 "" H 11450 6150 60  0000 C CNN
@@
 $EndComp
 $Comp
-L GND #PWR87
+L GND #PWR075
 U 1 1 523B56AC
 P 11450 5500
-F 0 "#PWR87" H 11450 5500 30  0001 C CNN
+F 0 "#PWR075" H 11450 5500 30  0001 C CNN
 F 1 "GND" H 11450 5430 30  0001 C CNN
 F 2 "" H 11450 5500 60  0000 C CNN
@@
 $EndComp
 $Comp
-L GND #PWR70
+L GND #PWR076
 U 1 1 5241DCB1
 P 3400 2600
-F 0 "#PWR70" H 3400 2600 30  0001 C CNN
+F 0 "#PWR076" H 3400 2600 30  0001 C CNN
 F 1 "GND" H 3400 2530 30  0001 C CNN
 F 2 "" H 3400 2600 60  0000 C CNN
@@
 $EndComp
 $Comp
-L GND #PWR71
+L GND #PWR077
 U 1 1 5241DCB7
 P 3600 2600
-F 0 "#PWR71" H 3600 2600 30  0001 C CNN
+F 0 "#PWR077" H 3600 2600 30  0001 C CNN
 F 1 "GND" H 3600 2530 30  0001 C CNN
 F 2 "" H 3600 2600 60  0000 C CNN
@@
 CTRL_SCK_1
 $Comp
-L GND #PWR75
+L GND #PWR078
 U 1 1 5241F98A
 P 4500 6150
-F 0 "#PWR75" H 4500 6150 30  0001 C CNN
+F 0 "#PWR078" H 4500 6150 30  0001 C CNN
 F 1 "GND" H 4500 6080 30  0001 C CNN
 F 2 "" H 4500 6150 60  0000 C CNN
@@
 $EndComp
 $Comp
-L GND #PWR76
+L GND #PWR079
 U 1 1 5241F999
 P 4600 6150
-F 0 "#PWR76" H 4600 6150 30  0001 C CNN
+F 0 "#PWR079" H 4600 6150 30  0001 C CNN
 F 1 "GND" H 4600 6080 30  0001 C CNN
 F 2 "" H 4600 6150 60  0000 C CNN
@@
 $EndComp
 $Comp
-L GND #PWR77
+L GND #PWR080
 U 1 1 5241F9A8
 P 4700 6150
-F 0 "#PWR77" H 4700 6150 30  0001 C CNN
+F 0 "#PWR080" H 4700 6150 30  0001 C CNN
 F 1 "GND" H 4700 6080 30  0001 C CNN
 F 2 "" H 4700 6150 60  0000 C CNN
@@
 $EndComp
 $Comp
-L GND #PWR78
+L GND #PWR081
 U 1 1 5241F9B7
 P 4800 6150
-F 0 "#PWR78" H 4800 6150 30  0001 C CNN
+F 0 "#PWR081" H 4800 6150 30  0001 C CNN
 F 1 "GND" H 4800 6080 30  0001 C CNN
 F 2 "" H 4800 6150 60  0000 C CNN
@@
 $EndComp
 $Comp
-L GND #PWR79
+L GND #PWR082
 U 1 1 5241F9C6
 P 4900 6150
-F 0 "#PWR79" H 4900 6150 30  0001 C CNN
+F 0 "#PWR082" H 4900 6150 30  0001 C CNN
 F 1 "GND" H 4900 6080 30  0001 C CNN
 F 2 "" H 4900 6150 60  0000 C CNN
@@
 $EndComp
 $Comp
-L GND #PWR80
+L GND #PWR083
 U 1 1 5241F9D5
 P 5000 6150
-F 0 "#PWR80" H 5000 6150 30  0001 C CNN
+F 0 "#PWR083" H 5000 6150 30  0001 C CNN
 F 1 "GND" H 5000 6080 30  0001 C CNN
 F 2 "" H 5000 6150 60  0000 C CNN
@@
 $EndComp
 $Comp
-L GND #PWR89
+L GND #PWR084
 U 1 1 5241FC10
 P 11750 4400
-F 0 "#PWR89" H 11750 4400 30  0001 C CNN
+F 0 "#PWR084" H 11750 4400 30  0001 C CNN
 F 1 "GND" H 11750 4330 30  0001 C CNN
 F 2 "" H 11750 4400 60  0000 C CNN
@@
 $EndComp
 $Comp
-L GND #PWR84
+L GND #PWR085
 U 1 1 5242CAEA
 P 8950 8150
-F 0 "#PWR84" H 8950 8150 30  0001 C CNN
+F 0 "#PWR085" H 8950 8150 30  0001 C CNN
 F 1 "GND" H 8950 8080 30  0001 C CNN
 F 2 "" H 8950 8150 60  0000 C CNN
@@
 $EndComp
 $Comp
-L GND #PWR93
+L GND #PWR086
 U 1 1 5242D310
 P 13900 8150
-F 0 "#PWR93" H 13900 8150 30  0001 C CNN
+F 0 "#PWR086" H 13900 8150 30  0001 C CNN
 F 1 "GND" H 13900 8080 30  0001 C CNN
 F 2 "" H 13900 8150 60  0000 C CNN
@@
 PDI_CLK
 $Comp
-L GND #PWR92
+L GND #PWR087
 U 1 1 5242D8EE
 P 13900 4000
-F 0 "#PWR92" H 13900 4000 30  0001 C CNN
+F 0 "#PWR087" H 13900 4000 30  0001 C CNN
 F 1 "GND" H 13900 3930 30  0001 C CNN
 F 2 "" H 13900 4000 60  0000 C CNN
@@
 TMS
 $Comp
-L GND #PWR91
+L GND #PWR088
 U 1 1 5243F5C0
 P 13700 2500
-F 0 "#PWR91" H 13700 2500 30  0001 C CNN
+F 0 "#PWR088" H 13700 2500 30  0001 C CNN
 F 1 "GND" H 13700 2430 30  0001 C CNN
 F 2 "" H 13700 2500 60  0000 C CNN
@@
 $EndComp
 $Comp
-L GND #PWR90
+L GND #PWR089
 U 1 1 5245EF15
 P 12000 7950
-F 0 "#PWR90" H 12000 7950 30  0001 C CNN
+F 0 "#PWR089" H 12000 7950 30  0001 C CNN
 F 1 "GND" H 12000 7880 30  0001 C CNN
 F 2 "" H 12000 7950 60  0000 C CNN
@@
 CTRL_3_3V
 $Comp
-L GND #PWR85
+L GND #PWR090
 U 1 1 52437304
 P 9750 5550
-F 0 "#PWR85" H 9750 5550 30  0001 C CNN
+F 0 "#PWR090" H 9750 5550 30  0001 C CNN
 F 1 "GND" H 9750 5480 30  0001 C CNN
 F 2 "" H 9750 5550 60  0000 C CNN
@@
 Text HLabel 10200 4050 0    60   Input ~ 0
 CTRL_GDO2
-Wire Wire Line
-	5750 2950 5800 2950
 Wire Wire Line
 	5750 3050 5800 3050
@@
 Text HLabel 3750 5600 0    60   Input ~ 0
 CTRL_RSTN
+NoConn ~ 10200 4150
+NoConn ~ 10200 4250
+Wire Wire Line
+	5750 2950 5800 2950
 $EndSCHEMATC
