File: Hardware/Controller.sch (KiCad schematic (older format))
At the start: 28 parts, among them IC1 ATXMEGA64A3U-A, P1 LOGIC_PORT_A, P2 ISP, P3 LOGIC_PORT_B, P4 LOGIC_PORT_B, P5 CONN_5X2, P6 PDI, SW1 TEST, SW2 RESET, U8 W25X20CL

Commit message: Added sensors and LEDs to PCB, and began dimensioning board
Parts:
- P5: value CONN_5X2 -> JTAG
- renumbered IC1 to U9
Changed lines of the file:
@@
 Sheet 7 7
 Title "Pong.0"
-Date "26 sep 2013"
+Date "16 nov 2013"
 Rev "0.3"
 Comp "Projects and Stuff LLC"
@@
 6E 56 52 49 51 4E 59 71 7E 65 C5 4D 0F AF 00 BF F6 21 9D BA 45 88 9C 00 16 00 C0 66 90 E0 00 00
 AC 42 3B 38 00 00 AB 90 E0 00 00 AC 42 82 03 00 B0 EA FF 00 E3 76 B5 A7 81 B6 BC 08 00 00 00 00
-49 45 4E 44 AE 42 60 82 35 $EndBitmap
+49 45 4E 44 AE 42 60 82 48 $EndBitmap
 EndData
 $EndBitmap
@@
 CTRL_D+
 $Comp
-L ATXMEGA64A3U-A IC1
+L ATXMEGA64A3U-A U9
 U 1 1 5241DAA8
 P 4750 4350
-F 0 "IC1" H 3950 5900 50  0000 L BNN
+F 0 "U9" H 3950 5900 50  0000 L BNN
 F 1 "ATXMEGA64A3U-A" H 5100 2700 50  0000 L BNN
 F 2 "TQFP64" H 4100 2750 50  0001 C CNN
@@
 P 12850 2250
 F 0 "P5" H 12850 2550 60  0000 C CNN
-F 1 "CONN_5X2" V 12850 2250 50  0000 C CNN
+F 1 "JTAG" V 12850 2250 50  0000 C CNN
 F 2 "" H 12850 2250 60  0000 C CNN
 F 3 "" H 12850 2250 60  0000 C CNN
