File: Hardware/LED_Display.sch (KiCad schematic (older format))
At the start: 4 parts

Commit message: Updated BOM and Schematic with significant components
Parts:
- removed U? (x3): AS1117, symbol AS1117
- removed U?: PCA9306, symbol PCA9306
- added C?: 0.1uF, ~, symbol CSMALL
- added R? (x6): 560, ~, symbol R
- added R?: 200k, ~, symbol R
- added U? (x3): AS1116, symbol AS1116
- added U?: NVT2006, symbol NVT2006
Connections:
- net labels added: 3_3V, 5V, GND
- wire segments 4 -> 25
Other:
- note added: "SPI Level\nTranslator"
- note removed: "I2C Level\nTranslator"

Commit message: Updated LED Display Sheet
Parts:
- added C? (x2): 0.1uF, ~, symbol CSMALL
- added C? (x2): 10uF, ~, symbol CSMALL
- added D? (x64): RGB_LED_V2, ~, symbol RGB_LED_V2
- added R? (x2): 560, ~, symbol R
- added R? (x2): R, ~, symbol R
Connections:
- net labels added: DISP_5V, DISP_MISO, DISP_MOSI, DISP_SCK, DISP_~SS
- wire segments 25 -> 82
- no-connect marks 0 -> 3
Other:
- moved on the sheet: R?, U?

Commit message: Continued populating the schematics.
Parts:
- removed C? (x3): 0.1uF, ~, symbol CSMALL
- removed C? (x2): 10uF, ~, symbol CSMALL
- removed D? (x57): RGB_LED_V2, ~, symbol RGB_LED_V2
- removed R? (x8): 560, ~, symbol R
- removed R?: 200k, ~, symbol R
- removed R? (x2): R, ~, symbol R
- removed U? (x3): AS1116, symbol AS1116
- removed U?: NVT2006, symbol NVT2006
- added C1, C2: 1uF, ~, symbol CSMALL
- added C3: 2.2uF, ~, symbol CSMALL
- added D1, D10, D11, D13, D14, D17, D18, D19, D2, D20, D21, D22, D23, D24, D25, D26, D28, D29, D3, D30, D31, D32, D33, D34, D35, D36, D37, D38, D39, D4, D40, D41, D42, D43, D44, D45, D5, D6, D7, D8, D9: RGB_LED_V2, ~, symbol RGB_LED_V2
- added U1: R_SMALL, symbol R_SMALL
- added U?: AS1119, symbol AS1119
- gave numbers to parts that had none: 7
Connections:
- net labels added: -VDD-, CS0, CS1, CS10, CS11, CS12, CS13, CS14, CS15, CS16, CS17, CS2, CS3, CS4, CS5, CS6, CS7, CS8, CS9, RSTN
- net labels removed: 3_3V, 5V, DISP_5V, DISP_MISO, DISP_MOSI, DISP_SCK, DISP_~SS
- wire segments 82 -> 345
- no-connect marks 3 -> 0
Other:
- note removed: "SPI Level\nTranslator"
- moved on the sheet: D12, D15, D16, D27, D46, D47, D48

Commit message: Corrected LED_Display pins
Parts:
- added C? (x3): 0.1uF, ~, symbol CSMALL
- added C? (x3): 10uF, ~, symbol CSMALL
- U1: value R_SMALL -> 5k
Connections:
- net labels added: 3_3V, DISP_3_3V, DISP_RSTN, DISP_SCL, DISP_SDA
- net labels removed: -VDD-, RSTN
- wire segments 345 -> 363
Other:
- moved on the sheet: U1
Changed lines of the file:
@@
 $Descr B 17000 11000
 encoding utf-8
-Sheet 2 8
+Sheet 8 8
 Title "Pong.0"
 Date "19 sep 2013"
@@
 6E 56 52 49 51 4E 59 71 7E 65 C5 4D 0F AF 00 BF F6 21 9D BA 45 88 9C 00 16 00 C0 66 90 E0 00 00
 AC 42 3B 38 00 00 AB 90 E0 00 00 AC 42 82 03 00 B0 EA FF 00 E3 76 B5 A7 81 B6 BC 08 00 00 00 00
-49 45 4E 44 AE 42 60 82 20 $EndBitmap
+49 45 4E 44 AE 42 60 82 3E $EndBitmap
 EndData
 $EndBitmap
@@
 L R_SMALL U1
 U 1 1 523B45D6
-P 2050 4800
-F 0 "U1" H 2090 4750 28  0000 C CNN
-F 1 "R_SMALL" H 2050 4800 22  0000 C CNN
-F 2 "" H 2050 4800 60  0000 C CNN
-F 3 "" H 2050 4800 60  0000 C CNN
-	1    2050 4800
-	1    0    0    -1
-$EndComp
-Text Label 1800 4800 2    60   ~ 0
-RSTN
-Text Label 1850 4750 0    60   ~ 0
--VDD-
+P 2000 4800
+F 0 "U1" H 2040 4750 28  0000 C CNN
+F 1 "5k" H 2000 4800 22  0000 C CNN
+F 2 "" H 2000 4800 60  0000 C CNN
+F 3 "" H 2000 4800 60  0000 C CNN
+	1    2000 4800
+	1    0    0    -1
+$EndComp
 Wire Wire Line
 	2800 6300 2800 6350
@@
 	2200 5100 2250 5100
 Wire Wire Line
-	2200 4800 2250 4800
-Wire Wire Line
-	1800 4800 1900 4800
-Wire Wire Line
-	1850 4800 1850 4750
-Connection ~ 1850 4800
+	2150 4800 2250 4800
 Wire Wire Line
 	7100 2800 7100 2850
@@
 Wire Wire Line
 	13600 7500 13600 7450
+Wire Wire Line
+	2250 4400 2200 4400
+Wire Wire Line
+	2250 4500 2200 4500
+Text HLabel 2200 4400 0    60   Input ~ 0
+DISP_SDA
+Text HLabel 2200 4500 0    60   Input ~ 0
+DISP_SCL
+Text HLabel 2200 4700 0    60   Input ~ 0
+DISP_RSTN
+$Comp
+L CSMALL C?
+U 1 1 523B4869
+P 2200 4150
+F 0 "C?" H 2225 4200 30  0000 L CNN
+F 1 "0.1uF" H 2225 4100 30  0000 L CNN
+F 2 "~" H 2200 4150 60  0000 C CNN
+F 3 "~" H 2200 4150 60  0000 C CNN
+	1    2200 4150
+	1    0    0    -1
+$EndComp
+$Comp
+L CSMALL C?
+U 1 1 523B487C
+P 2000 4150
+F 0 "C?" H 2025 4200 30  0000 L CNN
+F 1 "10uF" H 2025 4100 30  0000 L CNN
+F 2 "~" H 2000 4150 60  0000 C CNN
+F 3 "~" H 2000 4150 60  0000 C CNN
+	1    2000 4150
+	1    0    0    -1
+$EndComp
+$Comp
+L CSMALL C?
+U 1 1 523B488C
+P 1700 4050
+F 0 "C?" H 1725 4100 30  0000 L CNN
+F 1 "0.1uF" H 1725 4000 30  0000 L CNN
+F 2 "~" H 1700 4050 60  0000 C CNN
+F 3 "~" H 1700 4050 60  0000 C CNN
+	1    1700 4050
+	1    0    0    -1
+$EndComp
+$Comp
+L CSMALL C?
+U 1 1 523B4892
+P 1500 4050
+F 0 "C?" H 1525 4100 30  0000 L CNN
+F 1 "10uF" H 1525 4000 30  0000 L CNN
+F 2 "~" H 1500 4050 60  0000 C CNN
+F 3 "~" H 1500 4050 60  0000 C CNN
+	1    1500 4050
+	1    0    0    -1
+$EndComp
+$Comp
+L CSMALL C?
+U 1 1 523B4898
+P 1200 3950
+F 0 "C?" H 1225 4000 30  0000 L CNN
+F 1 "0.1uF" H 1225 3900 30  0000 L CNN
+F 2 "~" H 1200 3950 60  0000 C CNN
+F 3 "~" H 1200 3950 60  0000 C CNN
+	1    1200 3950
+	1    0    0    -1
+$EndComp
+$Comp
+L CSMALL C?
+U 1 1 523B489E
+P 1000 3950
+F 0 "C?" H 1025 4000 30  0000 L CNN
+F 1 "10uF" H 1025 3900 30  0000 L CNN
+F 2 "~" H 1000 3950 60  0000 C CNN
+F 3 "~" H 1000 3950 60  0000 C CNN
+	1    1000 3950
+	1    0    0    -1
+$EndComp
+Wire Wire Line
+	2250 4000 2000 4000
+Wire Wire Line
+	2000 4000 2000 4050
+Wire Wire Line
+	2200 4050 2200 4000
+Connection ~ 2200 4000
+Wire Wire Line
+	1500 3900 2250 3900
+Wire Wire Line
+	1700 3900 1700 3950
+Wire Wire Line
+	1500 3900 1500 3950
+Connection ~ 1700 3900
+Wire Wire Line
+	1000 3850 1000 3800
+Wire Wire Line
+	1000 3800 2250 3800
+Wire Wire Line
+	1200 3800 1200 3850
+Connection ~ 1200 3800
+$Comp
+L GND #PWR?
+U 1 1 523B53EE
+P 1000 4100
+F 0 "#PWR?" H 1000 4100 30  0001 C CNN
+F 1 "GND" H 1000 4030 30  0001 C CNN
+F 2 "" H 1000 4100 60  0000 C CNN
+F 3 "" H 1000 4100 60  0000 C CNN
+	1    1000 4100
+	1    0    0    -1
+$EndComp
+$Comp
+L GND #PWR?
+U 1 1 523B53FB
+P 1200 4100
+F 0 "#PWR?" H 1200 4100 30  0001 C CNN
+F 1 "GND" H 1200 4030 30  0001 C CNN
+F 2 "" H 1200 4100 60  0000 C CNN
+F 3 "" H 1200 4100 60  0000 C CNN
+	1    1200 4100
+	1    0    0    -1
+$EndComp
+$Comp
+L GND #PWR?
+U 1 1 523B5401
+P 1500 4200
+F 0 "#PWR?" H 1500 4200 30  0001 C CNN
+F 1 "GND" H 1500 4130 30  0001 C CNN
+F 2 "" H 1500 4200 60  0000 C CNN
+F 3 "" H 1500 4200 60  0000 C CNN
+	1    1500 4200
+	1    0    0    -1
+$EndComp
+$Comp
+L GND #PWR?
+U 1 1 523B5407
+P 1700 4200
+F 0 "#PWR?" H 1700 4200 30  0001 C CNN
+F 1 "GND" H 1700 4130 30  0001 C CNN
+F 2 "" H 1700 4200 60  0000 C CNN
+F 3 "" H 1700 4200 60  0000 C CNN
+	1    1700 4200
+	1    0    0    -1
+$EndComp
+$Comp
+L GND #PWR?
+U 1 1 523B540D
+P 2000 4300
+F 0 "#PWR?" H 2000 4300 30  0001 C CNN
+F 1 "GND" H 2000 4230 30  0001 C CNN
+F 2 "" H 2000 4300 60  0000 C CNN
+F 3 "" H 2000 4300 60  0000 C CNN
+	1    2000 4300
+	1    0    0    -1
+$EndComp
+$Comp
+L GND #PWR?
+U 1 1 523B5413
+P 2200 4300
+F 0 "#PWR?" H 2200 4300 30  0001 C CNN
+F 1 "GND" H 2200 4230 30  0001 C CNN
+F 2 "" H 2200 4300 60  0000 C CNN
+F 3 "" H 2200 4300 60  0000 C CNN
+	1    2200 4300
+	1    0    0    -1
+$EndComp
+Wire Wire Line
+	2200 4250 2200 4300
+Wire Wire Line
+	2000 4250 2000 4300
+Wire Wire Line
+	1700 4200 1700 4150
+Wire Wire Line
+	1500 4150 1500 4200
+Wire Wire Line
+	1200 4100 1200 4050
+Wire Wire Line
+	1000 4050 1000 4100
+Text HLabel 1450 3250 0    60   Input ~ 0
+DISP_3_3V
+Wire Wire Line
+	1450 3250 1500 3250
+Text Label 1500 3250 0    60   ~ 0
+3_3V
+Text Label 1000 3800 0    60   ~ 0
+3_3V
+Text Label 1500 3900 0    60   ~ 0
+3_3V
+Text Label 2000 4000 0    60   ~ 0
+3_3V
+Text Label 1150 3950 0    60   ~ 0
+3_3V
+Text Label 1800 4800 2    60   ~ 0
+3_3V
+Wire Wire Line
+	2200 4800 2200 4700
+Wire Wire Line
+	1800 4800 1850 4800
+Connection ~ 2200 4800
 $EndSCHEMATC

Commit message: Corrected Flash chip version and modified pins.
Parts:
- U1: value 5k -> 10k
Changed lines of the file:
@@
 6E 56 52 49 51 4E 59 71 7E 65 C5 4D 0F AF 00 BF F6 21 9D BA 45 88 9C 00 16 00 C0 66 90 E0 00 00
 AC 42 3B 38 00 00 AB 90 E0 00 00 AC 42 82 03 00 B0 EA FF 00 E3 76 B5 A7 81 B6 BC 08 00 00 00 00
-49 45 4E 44 AE 42 60 82 6B $EndBitmap
+49 45 4E 44 AE 42 60 82 F8 $EndBitmap
 EndData
 $EndBitmap
@@
 P 2000 4800
 F 0 "U1" H 2040 4750 28  0000 C CNN
-F 1 "5k" H 2000 4800 22  0000 C CNN
+F 1 "10k" H 2000 4800 22  0000 C CNN
 F 2 "" H 2000 4800 60  0000 C CNN
 F 3 "" H 2000 4800 60  0000 C CNN
