File: Hardware/LED_Display.sch (KiCad schematic (older format))
At the start: 59 parts, among them U1 10k

Commit message: Minor Cosmetic Changes
Parts:
- renumbered C1 to C?, C2 to C?, C3 to C?, U1 to R?
Changed lines of the file:
@@
 Sheet 5 7
 Title "Pong.0"
-Date "24 sep 2013"
+Date "25 sep 2013"
 Rev "0.3"
 Comp "Projects and Stuff LLC"
@@
 6E 56 52 49 51 4E 59 71 7E 65 C5 4D 0F AF 00 BF F6 21 9D BA 45 88 9C 00 16 00 C0 66 90 E0 00 00
 AC 42 3B 38 00 00 AB 90 E0 00 00 AC 42 82 03 00 B0 EA FF 00 E3 76 B5 A7 81 B6 BC 08 00 00 00 00
-49 45 4E 44 AE 42 60 82 81 $EndBitmap
+49 45 4E 44 AE 42 60 82 D0 $EndBitmap
 EndData
 $EndBitmap
@@
 $EndComp
 $Comp
-L CSMALL C1
+L CSMALL C?
 U 1 1 523B3911
 P 3050 6350
-F 0 "C1" H 3075 6400 30  0000 L CNN
+F 0 "C?" H 3075 6400 30  0000 L CNN
 F 1 "1uF" H 3075 6300 30  0000 L CNN
 F 2 "~" H 3050 6350 60  0000 C CNN
@@
 $EndComp
 $Comp
-L CSMALL C2
+L CSMALL C?
 U 1 1 523B391E
 P 3450 6350
-F 0 "C2" H 3475 6400 30  0000 L CNN
+F 0 "C?" H 3475 6400 30  0000 L CNN
 F 1 "1uF" H 3475 6300 30  0000 L CNN
 F 2 "~" H 3450 6350 60  0000 C CNN
@@
 $EndComp
 $Comp
-L CSMALL C3
+L CSMALL C?
 U 1 1 523B4142
 P 4150 6350
-F 0 "C3" H 4175 6400 30  0000 L CNN
+F 0 "C?" H 4175 6400 30  0000 L CNN
 F 1 "2.2uF" H 4175 6300 30  0000 L CNN
 F 2 "~" H 4150 6350 60  0000 C CNN
@@
 $EndComp
 $Comp
-L R_SMALL U1
+L R_SMALL R?
 U 1 1 523B45D6
 P 2100 4800
-F 0 "U1" H 2140 4750 28  0000 C CNN
+F 0 "R?" H 2140 4750 28  0000 C CNN
 F 1 "10k" H 2100 4800 22  0000 C CNN
 F 2 "" H 2100 4800 60  0000 C CNN

Commit message: Minor misc changes
Parts:
- removed C? (x3): 10uF, ~, symbol CSMALL
- added C? (x18): 1nF, ~, symbol CSMALL
- added C? (x3): 0.1uF, ~, symbol CSMALL
- added C? (x3): 10uF, symbol CPOLSMALL
Connections:
- net labels added: DISP_IRQ, DISP_SYNC
- wire segments 368 -> 409

Commit message: Fine-tuned some pins and labels
Parts:
- added R? (x3): 10k, ~, symbol R_SMALL
Connections:
- net labels removed: DISP_SYNC
- wire segments 409 -> 412
Other:
- moved on the sheet: C?, R?, U?

Commit message: Annotated Schematics
Parts:
- gave numbers to parts that had none: 35

Commit message: Made corrections based on ERC results
Parts:
- removed C28, C35, C42: 0.1uF, ~, symbol CSMALL
Connections:
- wire segments 412 -> 409
Changed lines of the file:
@@
 6E 56 52 49 51 4E 59 71 7E 65 C5 4D 0F AF 00 BF F6 21 9D BA 45 88 9C 00 16 00 C0 66 90 E0 00 00
 AC 42 3B 38 00 00 AB 90 E0 00 00 AC 42 82 03 00 B0 EA FF 00 E3 76 B5 A7 81 B6 BC 08 00 00 00 00
-49 45 4E 44 AE 42 60 82 AF $EndBitmap
+49 45 4E 44 AE 42 60 82 B4 $EndBitmap
 EndData
 $EndBitmap
@@
 $EndComp
 $Comp
-L GND #PWR31
+L GND #PWR022
 U 1 1 523B3940
 P 4600 6400
-F 0 "#PWR31" H 4600 6400 30  0001 C CNN
+F 0 "#PWR022" H 4600 6400 30  0001 C CNN
 F 1 "GND" H 4600 6330 30  0001 C CNN
 F 2 "" H 4600 6400 60  0000 C CNN
@@
 $EndComp
 $Comp
-L GND #PWR32
+L GND #PWR023
 U 1 1 523B394D
 P 4700 6400
-F 0 "#PWR32" H 4700 6400 30  0001 C CNN
+F 0 "#PWR023" H 4700 6400 30  0001 C CNN
 F 1 "GND" H 4700 6330 30  0001 C CNN
 F 2 "" H 4700 6400 60  0000 C CNN
@@
 $EndComp
 $Comp
-L GND #PWR33
+L GND #PWR024
 U 1 1 523B3953
 P 4800 6400
-F 0 "#PWR33" H 4800 6400 30  0001 C CNN
+F 0 "#PWR024" H 4800 6400 30  0001 C CNN
 F 1 "GND" H 4800 6330 30  0001 C CNN
 F 2 "" H 4800 6400 60  0000 C CNN
@@
 $EndComp
 $Comp
-L GND #PWR30
+L GND #PWR025
 U 1 1 523B3B6E
 P 3100 5350
-F 0 "#PWR30" H 3100 5350 30  0001 C CNN
+F 0 "#PWR025" H 3100 5350 30  0001 C CNN
 F 1 "GND" H 3100 5280 30  0001 C CNN
 F 2 "" H 3100 5350 60  0000 C CNN
@@
 $EndComp
 $Comp
-L GND #PWR29
+L GND #PWR026
 U 1 1 523B3B74
 P 3100 5150
-F 0 "#PWR29" H 3100 5150 30  0001 C CNN
+F 0 "#PWR026" H 3100 5150 30  0001 C CNN
 F 1 "GND" H 3100 5080 30  0001 C CNN
 F 2 "" H 3100 5150 60  0000 C CNN
@@
 $EndComp
 $Comp
-L GND #PWR22
+L GND #PWR027
 U 1 1 523B53EE
 P 1850 4100
-F 0 "#PWR22" H 1850 4100 30  0001 C CNN
+F 0 "#PWR027" H 1850 4100 30  0001 C CNN
 F 1 "GND" H 1850 4030 30  0001 C CNN
 F 2 "" H 1850 4100 60  0000 C CNN
@@
 $EndComp
 $Comp
-L GND #PWR23
+L GND #PWR028
 U 1 1 523B53FB
 P 2050 4100
-F 0 "#PWR23" H 2050 4100 30  0001 C CNN
+F 0 "#PWR028" H 2050 4100 30  0001 C CNN
 F 1 "GND" H 2050 4030 30  0001 C CNN
 F 2 "" H 2050 4100 60  0000 C CNN
@@
 $EndComp
 $Comp
-L GND #PWR24
+L GND #PWR029
 U 1 1 523B5401
 P 2350 4200
-F 0 "#PWR24" H 2350 4200 30  0001 C CNN
+F 0 "#PWR029" H 2350 4200 30  0001 C CNN
 F 1 "GND" H 2350 4130 30  0001 C CNN
 F 2 "" H 2350 4200 60  0000 C CNN
@@
 $EndComp
 $Comp
-L GND #PWR25
+L GND #PWR030
 U 1 1 523B5407
 P 2550 4200
-F 0 "#PWR25" H 2550 4200 30  0001 C CNN
+F 0 "#PWR030" H 2550 4200 30  0001 C CNN
 F 1 "GND" H 2550 4130 30  0001 C CNN
 F 2 "" H 2550 4200 60  0000 C CNN
@@
 $EndComp
 $Comp
-L GND #PWR27
+L GND #PWR031
 U 1 1 523B540D
 P 2850 4300
-F 0 "#PWR27" H 2850 4300 30  0001 C CNN
+F 0 "#PWR031" H 2850 4300 30  0001 C CNN
 F 1 "GND" H 2850 4230 30  0001 C CNN
 F 2 "" H 2850 4300 60  0000 C CNN
@@
 $EndComp
 $Comp
-L GND #PWR28
+L GND #PWR032
 U 1 1 523B5413
 P 3050 4300
-F 0 "#PWR28" H 3050 4300 30  0001 C CNN
+F 0 "#PWR032" H 3050 4300 30  0001 C CNN
 F 1 "GND" H 3050 4230 30  0001 C CNN
 F 2 "" H 3050 4300 60  0000 C CNN
@@
 $EndComp
 $Comp
-L GND #PWR34
+L GND #PWR033
 U 1 1 5243051B
 P 14000 3350
-F 0 "#PWR34" H 14000 3350 30  0001 C CNN
+F 0 "#PWR033" H 14000 3350 30  0001 C CNN
 F 1 "GND" H 14000 3280 30  0001 C CNN
 F 2 "" H 14000 3350 60  0000 C CNN
@@
 $EndComp
 $Comp
-L GND #PWR41
+L GND #PWR034
 U 1 1 52430528
 P 14200 3250
-F 0 "#PWR41" H 14200 3250 30  0001 C CNN
+F 0 "#PWR034" H 14200 3250 30  0001 C CNN
 F 1 "GND" H 14200 3180 30  0001 C CNN
 F 2 "" H 14200 3250 60  0000 C CNN
@@
 $EndComp
 $Comp
-L GND #PWR48
+L GND #PWR035
 U 1 1 5243052E
 P 14400 3150
-F 0 "#PWR48" H 14400 3150 30  0001 C CNN
+F 0 "#PWR035" H 14400 3150 30  0001 C CNN
 F 1 "GND" H 14400 3080 30  0001 C CNN
 F 2 "" H 14400 3150 60  0000 C CNN
@@
 $EndComp
 $Comp
-L GND #PWR35
+L GND #PWR036
 U 1 1 52431549
 P 14000 4400
-F 0 "#PWR35" H 14000 4400 30  0001 C CNN
+F 0 "#PWR036" H 14000 4400 30  0001 C CNN
 F 1 "GND" H 14000 4330 30  0001 C CNN
 F 2 "" H 14000 4400 60  0000 C CNN
@@
 $EndComp
 $Comp
-L GND #PWR42
+L GND #PWR037
 U 1 1 5243154F
 P 14200 4300
-F 0 "#PWR42" H 14200 4300 30  0001 C CNN
+F 0 "#PWR037" H 14200 4300 30  0001 C CNN
 F 1 "GND" H 14200 4230 30  0001 C CNN
 F 2 "" H 14200 4300 60  0000 C CNN
@@
 $EndComp
 $Comp
-L GND #PWR49
+L GND #PWR038
 U 1 1 52431555
 P 14400 4200
-F 0 "#PWR49" H 14400 4200 30  0001 C CNN
+F 0 "#PWR038" H 14400 4200 30  0001 C CNN
 F 1 "GND" H 14400 4130 30  0001 C CNN
 F 2 "" H 14400 4200 60  0000 C CNN
@@
 $EndComp
 $Comp
-L GND #PWR36
+L GND #PWR039
 U 1 1 52431570
 P 14000 5450
-F 0 "#PWR36" H 14000 5450 30  0001 C CNN
+F 0 "#PWR039" H 14000 5450 30  0001 C CNN
 F 1 "GND" H 14000 5380 30  0001 C CNN
 F 2 "" H 14000 5450 60  0000 C CNN
@@
 $EndComp
 $Comp
-L GND #PWR43
+L GND #PWR040
 U 1 1 52431576
 P 14200 5350
-F 0 "#PWR43" H 14200 5350 30  0001 C CNN
+F 0 "#PWR040" H 14200 5350 30  0001 C CNN
 F 1 "GND" H 14200 5280 30  0001 C CNN
 F 2 "" H 14200 5350 60  0000 C CNN
@@
 $EndComp
 $Comp
-L GND #PWR50
+L GND #PWR041
 U 1 1 5243157C
 P 14400 5250
-F 0 "#PWR50" H 14400 5250 30  0001 C CNN
+F 0 "#PWR041" H 14400 5250 30  0001 C CNN
 F 1 "GND" H 14400 5180 30  0001 C CNN
 F 2 "" H 14400 5250 60  0000 C CNN
@@
 $EndComp
 $Comp
-L GND #PWR37
+L GND #PWR042
 U 1 1 52431597
 P 14000 6500
-F 0 "#PWR37" H 14000 6500 30  0001 C CNN
+F 0 "#PWR042" H 14000 6500 30  0001 C CNN
 F 1 "GND" H 14000 6430 30  0001 C CNN
 F 2 "" H 14000 6500 60  0000 C CNN
@@
 $EndComp
 $Comp
-L GND #PWR44
+L GND #PWR043
 U 1 1 5243159D
 P 14200 6400
-F 0 "#PWR44" H 14200 6400 30  0001 C CNN
+F 0 "#PWR043" H 14200 6400 30  0001 C CNN
 F 1 "GND" H 14200 6330 30  0001 C CNN
 F 2 "" H 14200 6400 60  0000 C CNN
@@
 $EndComp
 $Comp
-L GND #PWR51
+L GND #PWR044
 U 1 1 524315A3
 P 14400 6300
-F 0 "#PWR51" H 14400 6300 30  0001 C CNN
+F 0 "#PWR044" H 14400 6300 30  0001 C CNN
 F 1 "GND" H 14400 6230 30  0001 C CNN
 F 2 "" H 14400 6300 60  0000 C CNN
@@
 $EndComp
 $Comp
-L GND #PWR38
+L GND #PWR045
 U 1 1 524315BE
 P 14000 7500
-F 0 "#PWR38" H 14000 7500 30  0001 C CNN
+F 0 "#PWR045" H 14000 7500 30  0001 C CNN
 F 1 "GND" H 14000 7430 30  0001 C CNN
 F 2 "" H 14000 7500 60  0000 C CNN
@@
 $EndComp
 $Comp
-L GND #PWR45
+L GND #PWR046
 U 1 1 524315C4
 P 14200 7400
-F 0 "#PWR45" H 14200 7400 30  0001 C CNN
+F 0 "#PWR046" H 14200 7400 30  0001 C CNN
 F 1 "GND" H 14200 7330 30  0001 C CNN
 F 2 "" H 14200 7400 60  0000 C CNN
@@
 $EndComp
 $Comp
-L GND #PWR52
+L GND #PWR047
 U 1 1 524315CA
 P 14400 7300
-F 0 "#PWR52" H 14400 7300 30  0001 C CNN
+F 0 "#PWR047" H 14400 7300 30  0001 C CNN
 F 1 "GND" H 14400 7230 30  0001 C CNN
 F 2 "" H 14400 7300 60  0000 C CNN
@@
 $EndComp
 $Comp
-L GND #PWR39
+L GND #PWR048
 U 1 1 524315E5
 P 14000 8550
-F 0 "#PWR39" H 14000 8550 30  0001 C CNN
+F 0 "#PWR048" H 14000 8550 30  0001 C CNN
 F 1 "GND" H 14000 8480 30  0001 C CNN
 F 2 "" H 14000 8550 60  0000 C CNN
@@
 $EndComp
 $Comp
-L GND #PWR46
+L GND #PWR049
 U 1 1 524315EB
 P 14200 8450
-F 0 "#PWR46" H 14200 8450 30  0001 C CNN
+F 0 "#PWR049" H 14200 8450 30  0001 C CNN
 F 1 "GND" H 14200 8380 30  0001 C CNN
 F 2 "" H 14200 8450 60  0000 C CNN
@@
 $EndComp
 $Comp
-L GND #PWR53
+L GND #PWR050
 U 1 1 524315F1
 P 14400 8350
-F 0 "#PWR53" H 14400 8350 30  0001 C CNN
+F 0 "#PWR050" H 14400 8350 30  0001 C CNN
 F 1 "GND" H 14400 8280 30  0001 C CNN
 F 2 "" H 14400 8350 60  0000 C CNN
 F 3 "" H 14400 8350 60  0000 C CNN
 	1    14400 8350
-	1    0    0    -1
-$EndComp
-$Comp
-L CSMALL C42
-U 1 1 52431621
-P 14400 10300
-F 0 "C42" H 14425 10350 30  0000 L CNN
-F 1 "0.1uF" H 14425 10250 30  0000 L CNN
-F 2 "~" H 14400 10300 60  0000 C CNN
-F 3 "~" H 14400 10300 60  0000 C CNN
-	1    14400 10300
-	1    0    0    -1
-$EndComp
-$Comp
-L CSMALL C35
-U 1 1 52431627
-P 14200 10400
-F 0 "C35" H 14225 10450 30  0000 L CNN
-F 1 "0.1uF" H 14225 10350 30  0000 L CNN
-F 2 "~" H 14200 10400 60  0000 C CNN
-F 3 "~" H 14200 10400 60  0000 C CNN
-	1    14200 10400
-	1    0    0    -1
-$EndComp
-$Comp
-L CSMALL C28
-U 1 1 5243162D
-P 14000 10500
-F 0 "C28" H 14025 10550 30  0000 L CNN
-F 1 "0.1uF" H 14025 10450 30  0000 L CNN
-F 2 "~" H 14000 10500 60  0000 C CNN
-F 3 "~" H 14000 10500 60  0000 C CNN
-	1    14000 10500
-	1    0    0    -1
-$EndComp
-$Comp
-L GND #PWR40
-U 1 1 52431633
-P 14000 10650
-F 0 "#PWR40" H 14000 10650 30  0001 C CNN
-F 1 "GND" H 14000 10580 30  0001 C CNN
-F 2 "" H 14000 10650 60  0000 C CNN
-F 3 "" H 14000 10650 60  0000 C CNN
-	1    14000 10650
-	1    0    0    -1
-$EndComp
-$Comp
-L GND #PWR47
-U 1 1 52431639
-P 14200 10550
-F 0 "#PWR47" H 14200 10550 30  0001 C CNN
-F 1 "GND" H 14200 10480 30  0001 C CNN
-F 2 "" H 14200 10550 60  0000 C CNN
-F 3 "" H 14200 10550 60  0000 C CNN
-	1    14200 10550
-	1    0    0    -1
-$EndComp
-$Comp
-L GND #PWR54
-U 1 1 5243163F
-P 14400 10450
-F 0 "#PWR54" H 14400 10450 30  0001 C CNN
-F 1 "GND" H 14400 10380 30  0001 C CNN
-F 2 "" H 14400 10450 60  0000 C CNN
-F 3 "" H 14400 10450 60  0000 C CNN
-	1    14400 10450
 	1    0    0    -1
 $EndComp
@@
 $EndComp
 $Comp
-L GND #PWR26
+L GND #PWR051
 U 1 1 52445CA0
 P 2750 5550
-F 0 "#PWR26" H 2750 5550 30  0001 C CNN
+F 0 "#PWR051" H 2750 5550 30  0001 C CNN
 F 1 "GND" H 2750 5480 30  0001 C CNN
 F 2 "" H 2750 5550 60  0000 C CNN
@@
 	14000 8500 14000 8550
 Wire Wire Line
-	14400 10400 14400 10450
-Wire Wire Line
-	14200 10500 14200 10550
-Wire Wire Line
-	14000 10600 14000 10650
-Wire Wire Line
 	14000 3050 14000 3100
