File: Hardware/LED_Display_B.sch (KiCad schematic (older format))
At the start: 53 parts, among them U1 R_SMALL

Commit message: Continued populating the schematics.
Parts:
- removed C1, C2: 1uF, ~, symbol CSMALL
- removed C3: 2.2uF, ~, symbol CSMALL
- removed D1, D10, D11, D12, D13, D14, D15, D16, D17, D18, D19, D2, D20, D21, D22, D23, D24, D25, D26, D27, D28, D29, D3, D30, D31, D32, D33, D34, D35, D36, D37, D38, D39, D4, D40, D41, D42, D43, D44, D45, D46, D47, D48, D5, D6, D7, D8, D9: RGB_LED_V2, ~, symbol RGB_LED_V2
- removed U1: R_SMALL, symbol R_SMALL
- removed U?: AS1119, symbol AS1119
- added C? (x3): 0.1uF, ~, symbol CSMALL
- added C? (x2): 10uF, ~, symbol CSMALL
- added D? (x64): RGB_LED_V2, ~, symbol RGB_LED_V2
- added R? (x8): 560, ~, symbol R
- added R?: 200k, ~, symbol R
- added R? (x2): R, ~, symbol R
- added U? (x3): AS1116, symbol AS1116
- added U?: NVT2006, symbol NVT2006
Connections:
- net labels added: 3_3V, 5V, DISP_B_5V, DISP_B_MISO, DISP_B_MOSI, DISP_B_SCK, DISP_B_~SS
- net labels removed: -VDD-, CS0, CS1, CS10, CS11, CS12, CS13, CS14, CS15, CS16, CS17, CS2, CS3, CS4, CS5, CS6, CS7, CS8, CS9, RSTN
- wire segments 345 -> 82
- no-connect marks 0 -> 3
Other:
- note added: "SPI Level\nTranslator"
