File: Hardware/LED_Display_B.sch (KiCad schematic (older format))
At the start: 76 parts

Commit message: Non-critical changes
Parts:
- removed D? (x40): RGB_LED_V2, ~, symbol RGB_LED_V2
Connections:
- wire segments 48 -> 49
Other:
- moved on the sheet: D?, R?, U?

Commit message: Completed schematic page
Parts:
- removed D? (x8): RGB_LED_V2, ~, symbol RGB_LED_V2
- added C?: 0.1uF, ~, symbol CSMALL
- added C?: 10uF, symbol CPOLSMALL
- added R?: 10k, ~, symbol R_SMALL
Connections:
- net labels added: DIG0, DIG1, DIG2, DIG3, DIG4, DIG5, SEGA, SEGB, SEGC, SEGD, SEGE, SEGF, SEGG, SEGH
- wire segments 49 -> 173
Other:
- moved on the sheet: D?

Commit message: Annotated Schematics
Parts:
- gave numbers to parts that had none: 31
Changed lines of the file:
@@
 SPI Level\nTranslator
 $Comp
-L AS1116 U?
+L AS1116 U6
 U 1 1 522A01E5
 P 6300 2700
-F 0 "U?" H 6600 1850 60  0000 C CNN
+F 0 "U6" H 6600 1850 60  0000 C CNN
 F 1 "AS1116" H 6100 3750 60  0000 C CNN
 F 2 "" H 6300 2700 60  0000 C CNN
@@
 $EndComp
 $Comp
-L NVT2006 U?
+L NVT2006 U5
 U 1 1 522A0581
 P 3350 3850
-F 0 "U?" H 3500 3500 60  0000 C CNN
+F 0 "U5" H 3500 3500 60  0000 C CNN
 F 1 "NVT2006" H 3200 5000 60  0000 C CNN
 F 2 "" H 3350 3850 60  0000 C CNN
@@
 $EndComp
 $Comp
-L R R?
+L R R16
 U 1 1 522A0590
 P 2600 3250
-F 0 "R?" V 2680 3250 40  0000 C CNN
+F 0 "R16" V 2680 3250 40  0000 C CNN
 F 1 "560" V 2607 3251 40  0000 C CNN
 F 2 "~" V 2530 3250 30  0000 C CNN
@@
 $EndComp
 $Comp
-L R R?
+L R R18
 U 1 1 522A05B3
 P 4300 3250
-F 0 "R?" V 4380 3250 40  0000 C CNN
+F 0 "R18" V 4380 3250 40  0000 C CNN
 F 1 "560" V 4307 3251 40  0000 C CNN
 F 2 "~" V 4230 3250 30  0000 C CNN
@@
 $EndComp
 $Comp
-L R R?
+L R R15
 U 1 1 522A066A
 P 2400 3250
-F 0 "R?" V 2480 3250 40  0000 C CNN
+F 0 "R15" V 2480 3250 40  0000 C CNN
 F 1 "560" V 2407 3251 40  0000 C CNN
 F 2 "~" V 2330 3250 30  0000 C CNN
@@
 $EndComp
 $Comp
-L R R?
+L R R14
 U 1 1 522A0670
 P 2200 3250
-F 0 "R?" V 2280 3250 40  0000 C CNN
+F 0 "R14" V 2280 3250 40  0000 C CNN
 F 1 "560" V 2207 3251 40  0000 C CNN
 F 2 "~" V 2130 3250 30  0000 C CNN
@@
 $EndComp
 $Comp
-L R R?
+L R R19
 U 1 1 522A0676
 P 4500 3250
-F 0 "R?" V 4580 3250 40  0000 C CNN
+F 0 "R19" V 4580 3250 40  0000 C CNN
 F 1 "560" V 4507 3251 40  0000 C CNN
 F 2 "~" V 4430 3250 30  0000 C CNN
@@
 $EndComp
 $Comp
-L R R?
+L R R20
 U 1 1 522A067C
 P 4700 3250
-F 0 "R?" V 4780 3250 40  0000 C CNN
+F 0 "R20" V 4780 3250 40  0000 C CNN
 F 1 "560" V 4707 3251 40  0000 C CNN
 F 2 "~" V 4630 3250 30  0000 C CNN
@@
 $EndComp
 $Comp
-L CSMALL C?
+L CSMALL C43
 U 1 1 522A06D5
 P 4000 3100
-F 0 "C?" H 4025 3150 30  0000 L CNN
+F 0 "C43" H 4025 3150 30  0000 L CNN
 F 1 "0.1uF" H 4025 3050 30  0000 L CNN
 F 2 "~" H 4000 3100 60  0000 C CNN
@@
 $EndComp
 $Comp
-L GND #PWR054
+L GND #PWR57
 U 1 1 522A06FF
 P 4000 3250
-F 0 "#PWR054" H 4000 3250 30  0001 C CNN
+F 0 "#PWR57" H 4000 3250 30  0001 C CNN
 F 1 "GND" H 4000 3180 30  0001 C CNN
 F 2 "" H 4000 3250 60  0000 C CNN
@@
 $EndComp
 $Comp
-L R R?
+L R R17
 U 1 1 522A0726
 P 4000 2550
-F 0 "R?" V 4080 2550 40  0000 C CNN
+F 0 "R17" V 4080 2550 40  0000 C CNN
 F 1 "200k" V 4007 2551 40  0000 C CNN
 F 2 "~" V 3930 2550 30  0000 C CNN
@@
 6E 56 52 49 51 4E 59 71 7E 65 C5 4D 0F AF 00 BF F6 21 9D BA 45 88 9C 00 16 00 C0 66 90 E0 00 00
 AC 42 3B 38 00 00 AB 90 E0 00 00 AC 42 82 03 00 B0 EA FF 00 E3 76 B5 A7 81 B6 BC 08 00 00 00 00
-49 45 4E 44 AE 42 60 82 79 $EndBitmap
+49 45 4E 44 AE 42 60 82 AF $EndBitmap
 EndData
 $EndBitmap
@@
 DISP_B_SCK
 $Comp
-L R R?
+L R R13
 U 1 1 5232229C
 P 2000 3250
-F 0 "R?" V 2080 3250 40  0000 C CNN
+F 0 "R13" V 2080 3250 40  0000 C CNN
 F 1 "560" V 2007 3251 40  0000 C CNN
 F 2 "~" V 1930 3250 30  0000 C CNN
@@
 DISP_B_~SS
 $Comp
-L R R?
+L R R21
 U 1 1 52322462
 P 4900 3250
-F 0 "R?" V 4980 3250 40  0000 C CNN
+F 0 "R21" V 4980 3250 40  0000 C CNN
 F 1 "560" V 4907 3251 40  0000 C CNN
 F 2 "~" V 4830 3250 30  0000 C CNN
@@
 $EndComp
 $Comp
-L GND #PWR055
+L GND #PWR58
 U 1 1 5232255B
 P 4000 4100
-F 0 "#PWR055" H 4000 4100 30  0001 C CNN
+F 0 "#PWR58" H 4000 4100 30  0001 C CNN
 F 1 "GND" H 4000 4030 30  0001 C CNN
 F 2 "" H 4000 4100 60  0000 C CNN
@@
 $EndComp
 $Comp
-L GND #PWR056
+L GND #PWR55
 U 1 1 523225D0
 P 2650 4100
-F 0 "#PWR056" H 2650 4100 30  0001 C CNN
+F 0 "#PWR55" H 2650 4100 30  0001 C CNN
 F 1 "GND" H 2650 4030 30  0001 C CNN
 F 2 "" H 2650 4100 60  0000 C CNN
@@
 NoConn ~ 5650 3300
 $Comp
-L GND #PWR057
+L GND #PWR61
 U 1 1 52322D99
 P 5600 3450
-F 0 "#PWR057" H 5600 3450 30  0001 C CNN
+F 0 "#PWR61" H 5600 3450 30  0001 C CNN
 F 1 "GND" H 5600 3380 30  0001 C CNN
 F 2 "" H 5600 3450 60  0000 C CNN
@@
 $EndComp
 $Comp
-L RGB_LED_V2 D?
+L RGB_LED_V2 D49
 U 1 1 52324597
 P 8250 2150
-F 0 "D?" H 8425 1925 60  0000 C CNN
+F 0 "D49" H 8425 1925 60  0000 C CNN
 F 1 "RGB_LED_V2" V 8050 2150 60  0001 C CNN
 F 2 "~" V 8250 2130 60  0000 C CNN
@@
 $EndComp
 $Comp
-L RGB_LED_V2 D?
+L RGB_LED_V2 D50
 U 1 1 5232459D
 P 9150 2150
-F 0 "D?" H 9325 1925 60  0000 C CNN
+F 0 "D50" H 9325 1925 60  0000 C CNN
 F 1 "RGB_LED_V2" V 8950 2150 60  0001 C CNN
 F 2 "~" V 9150 2130 60  0000 C CNN
@@
 $EndComp
 $Comp
-L RGB_LED_V2 D?
+L RGB_LED_V2 D51
 U 1 1 523245A3
 P 10050 2150
-F 0 "D?" H 10225 1925 60  0000 C CNN
+F 0 "D51" H 10225 1925 60  0000 C CNN
 F 1 "RGB_LED_V2" V 9850 2150 60  0001 C CNN
 F 2 "~" V 10050 2130 60  0000 C CNN
@@
 $EndComp
 $Comp
-L RGB_LED_V2 D?
+L RGB_LED_V2 D52
 U 1 1 523245A9
 P 10950 2150
-F 0 "D?" H 11125 1925 60  0000 C CNN
+F 0 "D52" H 11125 1925 60  0000 C CNN
 F 1 "RGB_LED_V2" V 10750 2150 60  0001 C CNN
 F 2 "~" V 10950 2130 60  0000 C CNN
@@
 $EndComp
 $Comp
-L RGB_LED_V2 D?
+L RGB_LED_V2 D53
 U 1 1 523245AF
 P 11850 2150
-F 0 "D?" H 12025 1925 60  0000 C CNN
+F 0 "D53" H 12025 1925 60  0000 C CNN
 F 1 "RGB_LED_V2" V 11650 2150 60  0001 C CNN
 F 2 "~" V 11850 2130 60  0000 C CNN
@@
 $EndComp
 $Comp
-L RGB_LED_V2 D?
+L RGB_LED_V2 D54
 U 1 1 523245B5
 P 12750 2150
-F 0 "D?" H 12925 1925 60  0000 C CNN
+F 0 "D54" H 12925 1925 60  0000 C CNN
 F 1 "RGB_LED_V2" V 12550 2150 60  0001 C CNN
 F 2 "~" V 12750 2130 60  0000 C CNN
@@
 $EndComp
 $Comp
-L RGB_LED_V2 D?
+L RGB_LED_V2 D55
 U 1 1 523245BB
 P 13650 2150
-F 0 "D?" H 13825 1925 60  0000 C CNN
+F 0 "D55" H 13825 1925 60  0000 C CNN
 F 1 "RGB_LED_V2" V 13450 2150 60  0001 C CNN
 F 2 "~" V 13650 2130 60  0000 C CNN
@@
 $EndComp
 $Comp
-L RGB_LED_V2 D?
+L RGB_LED_V2 D56
 U 1 1 523245C1
 P 14550 2150
-F 0 "D?" H 14725 1925 60  0000 C CNN
+F 0 "D56" H 14725 1925 60  0000 C CNN
 F 1 "RGB_LED_V2" V 14350 2150 60  0001 C CNN
 F 2 "~" V 14550 2130 60  0000 C CNN
@@
 $EndComp
 $Comp
-L RGB_LED_V2 D?
+L RGB_LED_V2 D57
 U 1 1 523245C7
 P 8250 3200
-F 0 "D?" H 8425 2975 60  0000 C CNN
+F 0 "D57" H 8425 2975 60  0000 C CNN
 F 1 "RGB_LED_V2" V 8050 3200 60  0001 C CNN
 F 2 "~" V 8250 3180 60  0000 C CNN
@@
 $EndComp
 $Comp
-L RGB_LED_V2 D?
+L RGB_LED_V2 D58
 U 1 1 523245CD
 P 9150 3200
-F 0 "D?" H 9325 2975 60  0000 C CNN
+F 0 "D58" H 9325 2975 60  0000 C CNN
 F 1 "RGB_LED_V2" V 8950 3200 60  0001 C CNN
 F 2 "~" V 9150 3180 60  0000 C CNN
@@
 $EndComp
 $Comp
-L RGB_LED_V2 D?
+L RGB_LED_V2 D59
 U 1 1 523245D3
 P 10050 3200
-F 0 "D?" H 10225 2975 60  0000 C CNN
+F 0 "D59" H 10225 2975 60  0000 C CNN
 F 1 "RGB_LED_V2" V 9850 3200 60  0001 C CNN
 F 2 "~" V 10050 3180 60  0000 C CNN
@@
 $EndComp
 $Comp
-L RGB_LED_V2 D?
+L RGB_LED_V2 D60
 U 1 1 523B548D
 P 10950 3200
-F 0 "D?" H 11125 2975 60  0000 C CNN
+F 0 "D60" H 11125 2975 60  0000 C CNN
 F 1 "RGB_LED_V2" V 10750 3200 60  0001 C CNN
 F 2 "~" V 10950 3180 60  0000 C CNN
@@
 $EndComp
 $Comp
-L RGB_LED_V2 D?
+L RGB_LED_V2 D61
 U 1 1 523245DF
 P 11850 3200
-F 0 "D?" H 12025 2975 60  0000 C CNN
+F 0 "D61" H 12025 2975 60  0000 C CNN
 F 1 "RGB_LED_V2" V 11650 3200 60  0001 C CNN
 F 2 "~" V 11850 3180 60  0000 C CNN
@@
 $EndComp
 $Comp
-L RGB_LED_V2 D?
+L RGB_LED_V2 D62
 U 1 1 523245E5
 P 12750 3200
-F 0 "D?" H 12925 2975 60  0000 C CNN
+F 0 "D62" H 12925 2975 60  0000 C CNN
 F 1 "RGB_LED_V2" V 12550 3200 60  0001 C CNN
 F 2 "~" V 12750 3180 60  0000 C CNN
@@
 $EndComp
 $Comp
-L RGB_LED_V2 D?
+L RGB_LED_V2 D63
 U 1 1 523B5490
 P 13650 3200
-F 0 "D?" H 13825 2975 60  0000 C CNN
+F 0 "D63" H 13825 2975 60  0000 C CNN
 F 1 "RGB_LED_V2" V 13450 3200 60  0001 C CNN
 F 2 "~" V 13650 3180 60  0000 C CNN
@@
 $EndComp
 $Comp
-L RGB_LED_V2 D?
+L RGB_LED_V2 D64
 U 1 1 523B5491
 P 14550 3200
-F 0 "D?" H 14725 2975 60  0000 C CNN
+F 0 "D64" H 14725 2975 60  0000 C CNN
 F 1 "RGB_LED_V2" V 14350 3200 60  0001 C CNN
 F 2 "~" V 14550 3180 60  0000 C CNN
@@
 DISP_B_3_3V
 $Comp
-L GND #PWR058
+L GND #PWR56
 U 1 1 52406923
 P 3350 4500
-F 0 "#PWR058" H 3350 4500 30  0001 C CNN
+F 0 "#PWR56" H 3350 4500 30  0001 C CNN
 F 1 "GND" H 3350 4430 30  0001 C CNN
 F 2 "" H 3350 4500 60  0000 C CNN
@@
 DISP_B_5V
 $Comp
-L GND #PWR?
+L GND #PWR59
 U 1 1 5243B889
 P 4850 2100
-F 0 "#PWR?" H 4850 2100 30  0001 C CNN
+F 0 "#PWR59" H 4850 2100 30  0001 C CNN
 F 1 "GND" H 4850 2030 30  0001 C CNN
 F 2 "" H 4850 2100 60  0000 C CNN
@@
 $EndComp
 $Comp
-L R_SMALL R?
+L R_SMALL R22
 U 1 1 5243B898
 P 5450 2100
-F 0 "R?" H 5490 2050 28  0000 C CNN
+F 0 "R22" H 5490 2050 28  0000 C CNN
 F 1 "10k" H 5450 2100 22  0000 C CNN
 F 2 "~" H 5450 2100 60  0000 C CNN
@@
 $EndComp
 $Comp
-L CSMALL C?
+L CSMALL C45
 U 1 1 5243BD03
 P 5050 1950
-F 0 "C?" H 5075 2000 30  0000 L CNN
+F 0 "C45" H 5075 2000 30  0000 L CNN
 F 1 "0.1uF" H 5075 1900 30  0000 L CNN
 F 2 "~" H 5050 1950 60  0000 C CNN
@@
 $EndComp
 $Comp
-L GND #PWR?
+L GND #PWR60
 U 1 1 5243BD09
 P 5050 2100
-F 0 "#PWR?" H 5050 2100 30  0001 C CNN
+F 0 "#PWR60" H 5050 2100 30  0001 C CNN
 F 1 "GND" H 5050 2030 30  0001 C CNN
 F 2 "" H 5050 2100 60  0000 C CNN
@@
 $EndComp
 $Comp
-L CPOLSMALL C?
+L CPOLSMALL C44
 U 1 1 5243C100
 P 4850 2000
-F 0 "C?" H 4900 2100 28  0000 C CNN
+F 0 "C44" H 4900 2100 28  0000 C CNN
 F 1 "10uF" H 4875 1975 28  0000 L CNN
 F 2 "" H 4850 2000 60  0000 C CNN

Commit message: Made corrections based on ERC results
Connections:
- no-connect marks 1 -> 3
Other:
- note added: "Waiting to hear\nback from AMS\non these two pins"
- moved on the sheet: D57, D58, D59, D60, D61, D62, D63, D64
