File: Hardware/RF.sch (KiCad schematic (older format))
At the start: 6 parts

Commit message: Updated Schematic with Battery Manager and updated some uC pins
Parts:
- added C?: 1uF, ~, symbol CSMALL
- added C?: 0.1uF, ~, symbol CSMALL
Connections:
- wire segments 23 -> 28
Changed lines of the file:
@@
 LIBS:valves
 LIBS:Pong.0
+LIBS:bq24163
+LIBS:usb-micro-b
+LIBS:IP4234CZ6
 LIBS:Pong.0-cache
 EELAYER 27 0
@@
 $Descr B 17000 11000
 encoding utf-8
-Sheet 3 3
+Sheet 3 4
 Title "Pong.0"
-Date "6 sep 2013"
+Date "8 sep 2013"
 Rev "0.2"
 Comp "Projects and Stuff LLC"
@@
 	1    0    0    -1
 $EndComp
+$Comp
+L CSMALL C?
+U 1 1 522CB32E
+P 5300 2550
+F 0 "C?" H 5325 2600 30  0000 L CNN
+F 1 "1uF" H 5325 2500 30  0000 L CNN
+F 2 "~" H 5300 2550 60  0000 C CNN
+F 3 "~" H 5300 2550 60  0000 C CNN
+	1    5300 2550
+	1    0    0    -1
+$EndComp
+$Comp
+L CSMALL C?
+U 1 1 522CB33B
+P 5000 2550
+F 0 "C?" H 5025 2600 30  0000 L CNN
+F 1 "0.1uF" H 5025 2500 30  0000 L CNN
+F 2 "~" H 5000 2550 60  0000 C CNN
+F 3 "~" H 5000 2550 60  0000 C CNN
+	1    5000 2550
+	1    0    0    -1
+$EndComp
+$Comp
+L GND #PWR?
+U 1 1 522CB343
+P 5000 2700
+F 0 "#PWR?" H 5000 2700 30  0001 C CNN
+F 1 "GND" H 5000 2630 30  0001 C CNN
+F 2 "" H 5000 2700 60  0000 C CNN
+F 3 "" H 5000 2700 60  0000 C CNN
+	1    5000 2700
+	1    0    0    -1
+$EndComp
+$Comp
+L GND #PWR?
+U 1 1 522CB350
+P 5300 2700
+F 0 "#PWR?" H 5300 2700 30  0001 C CNN
+F 1 "GND" H 5300 2630 30  0001 C CNN
+F 2 "" H 5300 2700 60  0000 C CNN
+F 3 "" H 5300 2700 60  0000 C CNN
+	1    5300 2700
+	1    0    0    -1
+$EndComp
+Wire Wire Line
+	5000 2650 5000 2700
+Wire Wire Line
+	5300 2650 5300 2700
+Wire Wire Line
+	5000 2450 5000 2400
+Wire Wire Line
+	5000 2400 5550 2400
+Wire Wire Line
+	5300 2400 5300 2450
+Connection ~ 5550 2400
+Connection ~ 5300 2400
 $EndSCHEMATC

Commit message: Continued populating the schematics.
Connections:
- net labels added: RF_3_3V, RF_MISO, RF_MOSI, RF_SCK, RF_~SS
- net labels removed: 3_3V
- wire segments 28 -> 34
Changed lines of the file:
@@
 $Descr B 17000 11000
 encoding utf-8
-Sheet 3 7
+Sheet 3 8
 Title "Pong.0"
-Date "12 sep 2013"
-Rev "0.2"
+Date "19 sep 2013"
+Rev "0.3"
 Comp "Projects and Stuff LLC"
 Comment1 ""
@@
 Connection ~ 5550 2800
 Connection ~ 5550 2300
-Text Label 5550 2250 2    60   ~ 0
-3_3V
 $Comp
 L CSMALL C?
@@
 6E 56 52 49 51 4E 59 71 7E 65 C5 4D 0F AF 00 BF F6 21 9D BA 45 88 9C 00 16 00 C0 66 90 E0 00 00
 AC 42 3B 38 00 00 AB 90 E0 00 00 AC 42 82 03 00 B0 EA FF 00 E3 76 B5 A7 81 B6 BC 08 00 00 00 00
-49 45 4E 44 AE 42 60 82 DC $EndBitmap
+49 45 4E 44 AE 42 60 82 20 $EndBitmap
 EndData
 $EndBitmap
@@
 EndData
 $EndBitmap
+Text HLabel 5550 2250 0    60   Input ~ 0
+RF_3_3V
+Wire Wire Line
+	5600 3300 5550 3300
+Wire Wire Line
+	5600 3400 5550 3400
+Text HLabel 5550 3300 0    60   Input ~ 0
+RF_SCK
+Text HLabel 5550 3400 0    60   Input ~ 0
+RF_MOSI
+Text HLabel 5550 3500 0    60   Input ~ 0
+RF_MISO
+Wire Wire Line
+	5550 3500 5600 3500
+Wire Wire Line
+	5600 3800 5550 3800
+Wire Wire Line
+	5600 3700 5550 3700
+Wire Wire Line
+	5600 3600 5550 3600
+Text HLabel 5550 3800 0    60   Input ~ 0
+RF_~SS
 $EndSCHEMATC
