File: Hardware/RF.sch (KiCad schematic (older format))
At the start: 8 parts

Commit message: Cleaned up RF Schematic Page
Connections:
- net labels added: GDO0_ATEST, GDO2
Changed lines of the file:
@@
 $Descr B 17000 11000
 encoding utf-8
-Sheet 2 7
+Sheet 7 7
 Title "Pong.0"
 Date "20 sep 2013"
@@
 L CSMALL C?
 U 1 1 522A191A
-P 6000 4950
-F 0 "C?" H 6025 5000 30  0000 L CNN
-F 1 "15pF" H 6025 4900 30  0000 L CNN
-F 2 "~" H 6000 4950 60  0000 C CNN
-F 3 "~" H 6000 4950 60  0000 C CNN
-	1    6000 4950
+P 6000 4750
+F 0 "C?" H 6025 4800 30  0000 L CNN
+F 1 "15pF" H 6025 4700 30  0000 L CNN
+F 2 "~" H 6000 4750 60  0000 C CNN
+F 3 "~" H 6000 4750 60  0000 C CNN
+	1    6000 4750
 	1    0    0    -1
 $EndComp
@@
 L CSMALL C?
 U 1 1 522A1927
-P 6700 4950
-F 0 "C?" H 6725 5000 30  0000 L CNN
-F 1 "15pF" H 6725 4900 30  0000 L CNN
-F 2 "~" H 6700 4950 60  0000 C CNN
-F 3 "~" H 6700 4950 60  0000 C CNN
-	1    6700 4950
-	1    0    0    -1
-$EndComp
-Wire Wire Line
-	6000 4550 6000 4850
+P 6700 4750
+F 0 "C?" H 6725 4800 30  0000 L CNN
+F 1 "15pF" H 6725 4700 30  0000 L CNN
+F 2 "~" H 6700 4750 60  0000 C CNN
+F 3 "~" H 6700 4750 60  0000 C CNN
+	1    6700 4750
+	1    0    0    -1
+$EndComp
 Wire Wire Line
 	6050 4600 6000 4600
 Connection ~ 6000 4600
 Wire Wire Line
-	6700 4550 6700 4850
-Wire Wire Line
 	6650 4600 6700 4600
 Connection ~ 6700 4600
@@
 L GND #PWR?
 U 1 1 522A193B
-P 6700 5100
-F 0 "#PWR?" H 6700 5100 30  0001 C CNN
-F 1 "GND" H 6700 5030 30  0001 C CNN
-F 2 "" H 6700 5100 60  0000 C CNN
-F 3 "" H 6700 5100 60  0000 C CNN
-	1    6700 5100
+P 6700 4900
+F 0 "#PWR?" H 6700 4900 30  0001 C CNN
+F 1 "GND" H 6700 4830 30  0001 C CNN
+F 2 "" H 6700 4900 60  0000 C CNN
+F 3 "" H 6700 4900 60  0000 C CNN
+	1    6700 4900
 	1    0    0    -1
 $EndComp
@@
 L GND #PWR?
 U 1 1 522A1948
-P 6000 5100
-F 0 "#PWR?" H 6000 5100 30  0001 C CNN
-F 1 "GND" H 6000 5030 30  0001 C CNN
-F 2 "" H 6000 5100 60  0000 C CNN
-F 3 "" H 6000 5100 60  0000 C CNN
-	1    6000 5100
-	1    0    0    -1
-$EndComp
-Wire Wire Line
-	6000 5050 6000 5100
-Wire Wire Line
-	6700 5050 6700 5100
-Wire Wire Line
-	5600 2300 5550 2300
-Wire Wire Line
-	5550 2250 5550 2900
+P 6000 4900
+F 0 "#PWR?" H 6000 4900 30  0001 C CNN
+F 1 "GND" H 6000 4830 30  0001 C CNN
+F 2 "" H 6000 4900 60  0000 C CNN
+F 3 "" H 6000 4900 60  0000 C CNN
+	1    6000 4900
+	1    0    0    -1
+$EndComp
+Wire Wire Line
+	6000 4850 6000 4900
+Wire Wire Line
+	6700 4850 6700 4900
+Wire Wire Line
+	5500 2300 5600 2300
 Wire Wire Line
 	5550 2500 5600 2500
@@
 6E 56 52 49 51 4E 59 71 7E 65 C5 4D 0F AF 00 BF F6 21 9D BA 45 88 9C 00 16 00 C0 66 90 E0 00 00
 AC 42 3B 38 00 00 AB 90 E0 00 00 AC 42 82 03 00 B0 EA FF 00 E3 76 B5 A7 81 B6 BC 08 00 00 00 00
-49 45 4E 44 AE 42 60 82 FC $EndBitmap
+49 45 4E 44 AE 42 60 82 30 $EndBitmap
 EndData
 $EndBitmap
@@
 EndData
 $EndBitmap
-Text HLabel 5550 2250 0    60   Input ~ 0
+Text HLabel 5500 2300 0    60   Input ~ 0
 RF_3_3V
 Wire Wire Line
@@
 Text HLabel 5550 3800 0    60   Input ~ 0
 RF_~SS
+Wire Wire Line
+	5550 2300 5550 2900
+Text HLabel 5550 3700 0    60   Input ~ 0
+GDO2
+Text HLabel 5550 3600 0    60   Input ~ 0
+GDO0_ATEST
+Wire Wire Line
+	6000 4550 6000 4650
+Wire Wire Line
+	6700 4550 6700 4650
 $EndSCHEMATC

Commit message: Added Dipole Antenna
Parts:
- added ANT?: DIPOLE, symbol DIPOLE
Connections:
- wire segments 34 -> 38
Changed lines of the file:
@@
 Sheet 7 7
 Title "Pong.0"
-Date "20 sep 2013"
+Date "24 sep 2013"
 Rev "0.3"
 Comp "Projects and Stuff LLC"
@@
 U 1 1 522A1901
 P 6350 4600
-F 0 "X?" H 6350 4750 60  0000 C CNN
+F 0 "X?" H 6350 4700 60  0000 C CNN
 F 1 "26 MHz" H 6350 4450 60  0000 C CNN
 F 2 "~" H 6350 4600 60  0000 C CNN
@@
 6E 56 52 49 51 4E 59 71 7E 65 C5 4D 0F AF 00 BF F6 21 9D BA 45 88 9C 00 16 00 C0 66 90 E0 00 00
 AC 42 3B 38 00 00 AB 90 E0 00 00 AC 42 82 03 00 B0 EA FF 00 E3 76 B5 A7 81 B6 BC 08 00 00 00 00
-49 45 4E 44 AE 42 60 82 30 $EndBitmap
+49 45 4E 44 AE 42 60 82 81 $EndBitmap
 EndData
 $EndBitmap
@@
 Wire Wire Line
 	6700 4550 6700 4650
+$Comp
+L DIPOLE ANT?
+U 1 1 5241CE1F
+P 7800 2450
+F 0 "ANT?" H 7950 2650 60  0000 C CNN
+F 1 "DIPOLE" H 7800 2900 60  0001 C CNN
+F 2 "" H 7800 2450 60  0000 C CNN
+F 3 "" H 7800 2450 60  0000 C CNN
+	1    7800 2450
+	1    0    0    -1
+$EndComp
+Wire Wire Line
+	7500 2600 7550 2600
+Wire Wire Line
+	7500 2700 8100 2700
+Wire Wire Line
+	8100 2700 8100 2600
+Wire Wire Line
+	8100 2600 8050 2600
 $EndSCHEMATC

Commit message: Minor misc changes
Connections:
- net labels added: RF_GDO0, RF_GDO2
- net labels removed: GDO0_ATEST, GDO2
Changed lines of the file:
@@
 $Descr B 17000 11000
 encoding utf-8
-Sheet 7 7
+Sheet 6 7
 Title "Pong.0"
 Date "25 sep 2013"
@@
 Connection ~ 6700 4600
 $Comp
-L GND #PWR?
+L GND #PWR059
 U 1 1 522A193B
 P 6700 4900
-F 0 "#PWR?" H 6700 4900 30  0001 C CNN
+F 0 "#PWR059" H 6700 4900 30  0001 C CNN
 F 1 "GND" H 6700 4830 30  0001 C CNN
 F 2 "" H 6700 4900 60  0000 C CNN
@@
 $EndComp
 $Comp
-L GND #PWR?
+L GND #PWR060
 U 1 1 522A1948
 P 6000 4900
-F 0 "#PWR?" H 6000 4900 30  0001 C CNN
+F 0 "#PWR060" H 6000 4900 30  0001 C CNN
 F 1 "GND" H 6000 4830 30  0001 C CNN
 F 2 "" H 6000 4900 60  0000 C CNN
@@
 L CSMALL C?
 U 1 1 522A1B69
-P 5350 3000
-F 0 "C?" H 5375 3050 30  0000 L CNN
-F 1 "0.1uF" H 5375 2950 30  0000 L CNN
-F 2 "~" H 5350 3000 60  0000 C CNN
-F 3 "~" H 5350 3000 60  0000 C CNN
-	1    5350 3000
-	0    -1   -1   0
-$EndComp
-$Comp
-L GND #PWR?
+P 5000 3150
+F 0 "C?" H 5025 3200 30  0000 L CNN
+F 1 "0.1uF" H 5025 3100 30  0000 L CNN
+F 2 "~" H 5000 3150 60  0000 C CNN
+F 3 "~" H 5000 3150 60  0000 C CNN
+	1    5000 3150
+	1    0    0    -1
+$EndComp
+$Comp
+L GND #PWR061
 U 1 1 522A1B71
-P 5200 3050
-F 0 "#PWR?" H 5200 3050 30  0001 C CNN
-F 1 "GND" H 5200 2980 30  0001 C CNN
-F 2 "" H 5200 3050 60  0000 C CNN
-F 3 "" H 5200 3050 60  0000 C CNN
-	1    5200 3050
-	1    0    0    -1
-$EndComp
-Wire Wire Line
-	5250 3000 5200 3000
-Wire Wire Line
-	5200 3000 5200 3050
-Wire Wire Line
-	5450 3000 5600 3000
+P 5000 3350
+F 0 "#PWR061" H 5000 3350 30  0001 C CNN
+F 1 "GND" H 5000 3280 30  0001 C CNN
+F 2 "" H 5000 3350 60  0000 C CNN
+F 3 "" H 5000 3350 60  0000 C CNN
+	1    5000 3350
+	1    0    0    -1
+$EndComp
+Wire Wire Line
+	5000 3250 5000 3350
 $Comp
 L R R?
@@
 	7550 3650 7550 3700
 $Comp
-L GND #PWR?
+L GND #PWR062
 U 1 1 522A1E6F
 P 7550 4250
-F 0 "#PWR?" H 7550 4250 30  0001 C CNN
+F 0 "#PWR062" H 7550 4250 30  0001 C CNN
 F 1 "GND" H 7550 4180 30  0001 C CNN
 F 2 "" H 7550 4250 60  0000 C CNN
@@
 Connection ~ 7100 4600
 $Comp
-L GND #PWR?
+L GND #PWR063
 U 1 1 522A20B2
 P 7100 4650
-F 0 "#PWR?" H 7100 4650 30  0001 C CNN
+F 0 "#PWR063" H 7100 4650 30  0001 C CNN
 F 1 "GND" H 7100 4580 30  0001 C CNN
 F 2 "" H 7100 4650 60  0000 C CNN
@@
 $EndComp
 $Comp
-L GND #PWR?
+L GND #PWR064
 U 1 1 522CB343
 P 5000 2700
-F 0 "#PWR?" H 5000 2700 30  0001 C CNN
+F 0 "#PWR064" H 5000 2700 30  0001 C CNN
 F 1 "GND" H 5000 2630 30  0001 C CNN
 F 2 "" H 5000 2700 60  0000 C CNN
@@
 $EndComp
 $Comp
-L GND #PWR?
+L GND #PWR065
 U 1 1 522CB350
 P 5300 2700
-F 0 "#PWR?" H 5300 2700 30  0001 C CNN
+F 0 "#PWR065" H 5300 2700 30  0001 C CNN
 F 1 "GND" H 5300 2630 30  0001 C CNN
 F 2 "" H 5300 2700 60  0000 C CNN
@@
 6E 56 52 49 51 4E 59 71 7E 65 C5 4D 0F AF 00 BF F6 21 9D BA 45 88 9C 00 16 00 C0 66 90 E0 00 00
 AC 42 3B 38 00 00 AB 90 E0 00 00 AC 42 82 03 00 B0 EA FF 00 E3 76 B5 A7 81 B6 BC 08 00 00 00 00
-49 45 4E 44 AE 42 60 82 D0 $EndBitmap
+49 45 4E 44 AE 42 60 82 E3 $EndBitmap
 EndData
 $EndBitmap
@@
 	5550 2300 5550 2900
 Text HLabel 5550 3700 0    60   Input ~ 0
-GDO2
+RF_GDO2
 Text HLabel 5550 3600 0    60   Input ~ 0
-GDO0_ATEST
+RF_GDO0
 Wire Wire Line
 	6000 4550 6000 4650
@@
 Wire Wire Line
 	8100 2600 8050 2600
+Wire Wire Line
+	5600 3000 5000 3000
+Wire Wire Line
+	5000 3000 5000 3050
 $EndSCHEMATC

Commit message: Annotated Schematics
Parts:
- gave numbers to parts that had none: 9
Changed lines of the file:
@@
 $EndDescr
 $Comp
-L CC2500 U?
+L CC2500 U7
 U 1 1 522A18F2
 P 6550 3200
-F 0 "U?" H 7200 2100 60  0000 C CNN
+F 0 "U7" H 7200 2100 60  0000 C CNN
 F 1 "CC2500" H 6100 4250 60  0000 C CNN
 F 2 "" H 6950 3200 60  0000 C CNN
@@
 $EndComp
 $Comp
-L CRYSTAL X?
+L CRYSTAL X1
 U 1 1 522A1901
 P 6350 4600
-F 0 "X?" H 6350 4700 60  0000 C CNN
+F 0 "X1" H 6350 4700 60  0000 C CNN
 F 1 "26 MHz" H 6350 4450 60  0000 C CNN
 F 2 "~" H 6350 4600 60  0000 C CNN
@@
 $EndComp
 $Comp
-L CSMALL C?
+L CSMALL C49
 U 1 1 522A191A
 P 6000 4750
-F 0 "C?" H 6025 4800 30  0000 L CNN
+F 0 "C49" H 6025 4800 30  0000 L CNN
 F 1 "15pF" H 6025 4700 30  0000 L CNN
 F 2 "~" H 6000 4750 60  0000 C CNN
@@
 $EndComp
 $Comp
-L CSMALL C?
+L CSMALL C50
 U 1 1 522A1927
 P 6700 4750
-F 0 "C?" H 6725 4800 30  0000 L CNN
+F 0 "C50" H 6725 4800 30  0000 L CNN
 F 1 "15pF" H 6725 4700 30  0000 L CNN
 F 2 "~" H 6700 4750 60  0000 C CNN
@@
 Connection ~ 6700 4600
 $Comp
-L GND #PWR059
+L GND #PWR66
 U 1 1 522A193B
 P 6700 4900
-F 0 "#PWR059" H 6700 4900 30  0001 C CNN
+F 0 "#PWR66" H 6700 4900 30  0001 C CNN
 F 1 "GND" H 6700 4830 30  0001 C CNN
 F 2 "" H 6700 4900 60  0000 C CNN
@@
 $EndComp
 $Comp
-L GND #PWR060
+L GND #PWR65
 U 1 1 522A1948
 P 6000 4900
-F 0 "#PWR060" H 6000 4900 30  0001 C CNN
+F 0 "#PWR65" H 6000 4900 30  0001 C CNN
 F 1 "GND" H 6000 4830 30  0001 C CNN
 F 2 "" H 6000 4900 60  0000 C CNN
@@
 Connection ~ 5550 2300
 $Comp
-L CSMALL C?
+L CSMALL C47
 U 1 1 522A1B69
 P 5000 3150
-F 0 "C?" H 5025 3200 30  0000 L CNN
+F 0 "C47" H 5025 3200 30  0000 L CNN
 F 1 "0.1uF" H 5025 3100 30  0000 L CNN
 F 2 "~" H 5000 3150 60  0000 C CNN
@@
 $EndComp
 $Comp
-L GND #PWR061
+L GND #PWR63
 U 1 1 522A1B71
 P 5000 3350
-F 0 "#PWR061" H 5000 3350 30  0001 C CNN
+F 0 "#PWR63" H 5000 3350 30  0001 C CNN
 F 1 "GND" H 5000 3280 30  0001 C CNN
 F 2 "" H 5000 3350 60  0000 C CNN
@@
 	5000 3250 5000 3350
 $Comp
-L R R?
+L R R23
 U 1 1 522A1E48
 P 7550 3950
-F 0 "R?" V 7630 3950 40  0000 C CNN
+F 0 "R23" V 7630 3950 40  0000 C CNN
 F 1 "R" V 7557 3951 40  0000 C CNN
 F 2 "~" V 7480 3950 30  0000 C CNN
@@
 	7550 3650 7550 3700
 $Comp
-L GND #PWR062
+L GND #PWR68
 U 1 1 522A1E6F
 P 7550 4250
-F 0 "#PWR062" H 7550 4250 30  0001 C CNN
+F 0 "#PWR68" H 7550 4250 30  0001 C CNN
 F 1 "GND" H 7550 4180 30  0001 C CNN
 F 2 "" H 7550 4250 60  0000 C CNN
@@
 Connection ~ 7100 4600
 $Comp
-L GND #PWR063
+L GND #PWR67
 U 1 1 522A20B2
 P 7100 4650
-F 0 "#PWR063" H 7100 4650 30  0001 C CNN
+F 0 "#PWR67" H 7100 4650 30  0001 C CNN
 F 1 "GND" H 7100 4580 30  0001 C CNN
 F 2 "" H 7100 4650 60  0000 C CNN
@@
 $EndComp
 $Comp
-L CSMALL C?
+L CSMALL C48
 U 1 1 522CB32E
 P 5300 2550
-F 0 "C?" H 5325 2600 30  0000 L CNN
+F 0 "C48" H 5325 2600 30  0000 L CNN
 F 1 "1uF" H 5325 2500 30  0000 L CNN
 F 2 "~" H 5300 2550 60  0000 C CNN
@@
 $EndComp
 $Comp
-L CSMALL C?
+L CSMALL C46
 U 1 1 522CB33B
 P 5000 2550
-F 0 "C?" H 5025 2600 30  0000 L CNN
+F 0 "C46" H 5025 2600 30  0000 L CNN
 F 1 "0.1uF" H 5025 2500 30  0000 L CNN
 F 2 "~" H 5000 2550 60  0000 C CNN
@@
 $EndComp
 $Comp
-L GND #PWR064
+L GND #PWR62
 U 1 1 522CB343
 P 5000 2700
-F 0 "#PWR064" H 5000 2700 30  0001 C CNN
+F 0 "#PWR62" H 5000 2700 30  0001 C CNN
 F 1 "GND" H 5000 2630 30  0001 C CNN
 F 2 "" H 5000 2700 60  0000 C CNN
@@
 $EndComp
 $Comp
-L GND #PWR065
+L GND #PWR64
 U 1 1 522CB350
 P 5300 2700
-F 0 "#PWR065" H 5300 2700 30  0001 C CNN
+F 0 "#PWR64" H 5300 2700 30  0001 C CNN
 F 1 "GND" H 5300 2630 30  0001 C CNN
 F 2 "" H 5300 2700 60  0000 C CNN
@@
 6E 56 52 49 51 4E 59 71 7E 65 C5 4D 0F AF 00 BF F6 21 9D BA 45 88 9C 00 16 00 C0 66 90 E0 00 00
 AC 42 3B 38 00 00 AB 90 E0 00 00 AC 42 82 03 00 B0 EA FF 00 E3 76 B5 A7 81 B6 BC 08 00 00 00 00
-49 45 4E 44 AE 42 60 82 79 $EndBitmap
+49 45 4E 44 AE 42 60 82 AF $EndBitmap
 EndData
 $EndBitmap
@@
 	6700 4550 6700 4650
 $Comp
-L DIPOLE ANT?
+L DIPOLE ANT1
 U 1 1 5241CE1F
 P 7800 2450
-F 0 "ANT?" H 7950 2650 60  0000 C CNN
+F 0 "ANT1" H 7950 2650 60  0000 C CNN
 F 1 "DIPOLE" H 7800 2900 60  0001 C CNN
 F 2 "" H 7800 2450 60  0000 C CNN
