File: Hardware/Sensors.sch (KiCad schematic (older format))
At the start: 0 parts

Commit message: Continued populating the schematics.
Parts:
- added QM? (x18): CAPSENSOR, ~, symbol CAPSENSOR
Changed lines of the file:
@@
 $Descr B 17000 11000
 encoding utf-8
-Sheet 4 7
+Sheet 4 8
 Title "Pong.0"
-Date "12 sep 2013"
-Rev "0.2"
+Date "19 sep 2013"
+Rev "0.3"
 Comp "Projects and Stuff LLC"
 Comment1 ""
@@
 6E 56 52 49 51 4E 59 71 7E 65 C5 4D 0F AF 00 BF F6 21 9D BA 45 88 9C 00 16 00 C0 66 90 E0 00 00
 AC 42 3B 38 00 00 AB 90 E0 00 00 AC 42 82 03 00 B0 EA FF 00 E3 76 B5 A7 81 B6 BC 08 00 00 00 00
-49 45 4E 44 AE 42 60 82 DC $EndBitmap
+49 45 4E 44 AE 42 60 82 20 $EndBitmap
 EndData
 $EndBitmap
@@
 EndData
 $EndBitmap
+$Comp
+L CAPSENSOR QM?
+U 1 1 52365848
+P 5200 2850
+F 0 "QM?" H 5160 2970 60  0000 C CNN
+F 1 "CAPSENSOR" V 5310 2840 40  0001 C CNN
+F 2 "~" H 5200 2850 60  0000 C CNN
+F 3 "~" H 5200 2850 60  0000 C CNN
+	1    5200 2850
+	1    0    0    -1
+$EndComp
+$Comp
+L CAPSENSOR QM?
+U 1 1 52365855
+P 5700 2850
+F 0 "QM?" H 5660 2970 60  0000 C CNN
+F 1 "CAPSENSOR" V 5810 2840 40  0001 C CNN
+F 2 "~" H 5700 2850 60  0000 C CNN
+F 3 "~" H 5700 2850 60  0000 C CNN
+	1    5700 2850
+	1    0    0    -1
+$EndComp
+$Comp
+L CAPSENSOR QM?
+U 1 1 5236585B
+P 5200 3350
+F 0 "QM?" H 5160 3470 60  0000 C CNN
+F 1 "CAPSENSOR" V 5310 3340 40  0001 C CNN
+F 2 "~" H 5200 3350 60  0000 C CNN
+F 3 "~" H 5200 3350 60  0000 C CNN
+	1    5200 3350
+	1    0    0    -1
+$EndComp
+$Comp
+L CAPSENSOR QM?
+U 1 1 52365861
+P 5700 3350
+F 0 "QM?" H 5660 3470 60  0000 C CNN
+F 1 "CAPSENSOR" V 5810 3340 40  0001 C CNN
+F 2 "~" H 5700 3350 60  0000 C CNN
+F 3 "~" H 5700 3350 60  0000 C CNN
+	1    5700 3350
+	1    0    0    -1
+$EndComp
+$Comp
+L CAPSENSOR QM?
+U 1 1 52365867
+P 6200 2850
+F 0 "QM?" H 6160 2970 60  0000 C CNN
+F 1 "CAPSENSOR" V 6310 2840 40  0001 C CNN
+F 2 "~" H 6200 2850 60  0000 C CNN
+F 3 "~" H 6200 2850 60  0000 C CNN
+	1    6200 2850
+	1    0    0    -1
+$EndComp
+$Comp
+L CAPSENSOR QM?
+U 1 1 5236586D
+P 6700 2850
+F 0 "QM?" H 6660 2970 60  0000 C CNN
+F 1 "CAPSENSOR" V 6810 2840 40  0001 C CNN
+F 2 "~" H 6700 2850 60  0000 C CNN
+F 3 "~" H 6700 2850 60  0000 C CNN
+	1    6700 2850
+	1    0    0    -1
+$EndComp
+$Comp
+L CAPSENSOR QM?
+U 1 1 52365873
+P 6200 3350
+F 0 "QM?" H 6160 3470 60  0000 C CNN
+F 1 "CAPSENSOR" V 6310 3340 40  0001 C CNN
+F 2 "~" H 6200 3350 60  0000 C CNN
+F 3 "~" H 6200 3350 60  0000 C CNN
+	1    6200 3350
+	1    0    0    -1
+$EndComp
+$Comp
+L CAPSENSOR QM?
+U 1 1 52365879
+P 6700 3350
+F 0 "QM?" H 6660 3470 60  0000 C CNN
+F 1 "CAPSENSOR" V 6810 3340 40  0001 C CNN
+F 2 "~" H 6700 3350 60  0000 C CNN
+F 3 "~" H 6700 3350 60  0000 C CNN
+	1    6700 3350
+	1    0    0    -1
+$EndComp
+$Comp
+L CAPSENSOR QM?
+U 1 1 5236587F
+P 7200 2850
+F 0 "QM?" H 7160 2970 60  0000 C CNN
+F 1 "CAPSENSOR" V 7310 2840 40  0001 C CNN
+F 2 "~" H 7200 2850 60  0000 C CNN
+F 3 "~" H 7200 2850 60  0000 C CNN
+	1    7200 2850
+	1    0    0    -1
+$EndComp
+$Comp
+L CAPSENSOR QM?
+U 1 1 52365885
+P 7700 2850
+F 0 "QM?" H 7660 2970 60  0000 C CNN
+F 1 "CAPSENSOR" V 7810 2840 40  0001 C CNN
+F 2 "~" H 7700 2850 60  0000 C CNN
+F 3 "~" H 7700 2850 60  0000 C CNN
+	1    7700 2850
+	1    0    0    -1
+$EndComp
+$Comp
+L CAPSENSOR QM?
+U 1 1 5236588B
+P 7200 3350
+F 0 "QM?" H 7160 3470 60  0000 C CNN
+F 1 "CAPSENSOR" V 7310 3340 40  0001 C CNN
+F 2 "~" H 7200 3350 60  0000 C CNN
+F 3 "~" H 7200 3350 60  0000 C CNN
+	1    7200 3350
+	1    0    0    -1
+$EndComp
+$Comp
+L CAPSENSOR QM?
+U 1 1 52365891
+P 7700 3350
+F 0 "QM?" H 7660 3470 60  0000 C CNN
+F 1 "CAPSENSOR" V 7810 3340 40  0001 C CNN
+F 2 "~" H 7700 3350 60  0000 C CNN
+F 3 "~" H 7700 3350 60  0000 C CNN
+	1    7700 3350
+	1    0    0    -1
+$EndComp
+$Comp
+L CAPSENSOR QM?
+U 1 1 52365897
+P 8200 2850
+F 0 "QM?" H 8160 2970 60  0000 C CNN
+F 1 "CAPSENSOR" V 8310 2840 40  0001 C CNN
+F 2 "~" H 8200 2850 60  0000 C CNN
+F 3 "~" H 8200 2850 60  0000 C CNN
+	1    8200 2850
+	1    0    0    -1
+$EndComp
+$Comp
+L CAPSENSOR QM?
+U 1 1 5236589D
+P 8700 2850
+F 0 "QM?" H 8660 2970 60  0000 C CNN
+F 1 "CAPSENSOR" V 8810 2840 40  0001 C CNN
+F 2 "~" H 8700 2850 60  0000 C CNN
+F 3 "~" H 8700 2850 60  0000 C CNN
+	1    8700 2850
+	1    0    0    -1
+$EndComp
+$Comp
+L CAPSENSOR QM?
+U 1 1 523658A3
+P 8200 3350
+F 0 "QM?" H 8160 3470 60  0000 C CNN
+F 1 "CAPSENSOR" V 8310 3340 40  0001 C CNN
+F 2 "~" H 8200 3350 60  0000 C CNN
+F 3 "~" H 8200 3350 60  0000 C CNN
+	1    8200 3350
+	1    0    0    -1
+$EndComp
+$Comp
+L CAPSENSOR QM?
+U 1 1 523658A9
+P 8700 3350
+F 0 "QM?" H 8660 3470 60  0000 C CNN
+F 1 "CAPSENSOR" V 8810 3340 40  0001 C CNN
+F 2 "~" H 8700 3350 60  0000 C CNN
+F 3 "~" H 8700 3350 60  0000 C CNN
+	1    8700 3350
+	1    0    0    -1
+$EndComp
+$Comp
+L CAPSENSOR QM?
+U 1 1 523658AF
+P 9200 2850
+F 0 "QM?" H 9160 2970 60  0000 C CNN
+F 1 "CAPSENSOR" V 9310 2840 40  0001 C CNN
+F 2 "~" H 9200 2850 60  0000 C CNN
+F 3 "~" H 9200 2850 60  0000 C CNN
+	1    9200 2850
+	1    0    0    -1
+$EndComp
+$Comp
+L CAPSENSOR QM?
+U 1 1 523658B5
+P 9200 3350
+F 0 "QM?" H 9160 3470 60  0000 C CNN
+F 1 "CAPSENSOR" V 9310 3340 40  0001 C CNN
+F 2 "~" H 9200 3350 60  0000 C CNN
+F 3 "~" H 9200 3350 60  0000 C CNN
+	1    9200 3350
+	1    0    0    -1
+$EndComp
 $EndSCHEMATC
