File: Hardware/Sensors.sch (KiCad schematic (older format))
At the start: 59 parts

Commit message: Non-critical changes
Parts:
- gave numbers to parts that had none: 39
Changed lines of the file:
@@
 $Descr B 17000 11000
 encoding utf-8
-Sheet 3 7
+Sheet 4 7
 Title "Pong.0"
-Date "20 sep 2013"
+Date "24 sep 2013"
 Rev "0.3"
 Comp "Projects and Stuff LLC"
@@
 6E 56 52 49 51 4E 59 71 7E 65 C5 4D 0F AF 00 BF F6 21 9D BA 45 88 9C 00 16 00 C0 66 90 E0 00 00
 AC 42 3B 38 00 00 AB 90 E0 00 00 AC 42 82 03 00 B0 EA FF 00 E3 76 B5 A7 81 B6 BC 08 00 00 00 00
-49 45 4E 44 AE 42 60 82 30 $EndBitmap
+49 45 4E 44 AE 42 60 82 81 $EndBitmap
 EndData
 $EndBitmap
@@
 $EndBitmap
 $Comp
-L CAPSENSOR QM?
+L CAPSENSOR QM1
 U 1 1 52365848
 P 5200 2850
-F 0 "QM?" H 5160 2970 60  0000 C CNN
+F 0 "QM1" H 5160 2970 60  0000 C CNN
 F 1 "CAPSENSOR" V 5310 2840 40  0001 C CNN
 F 2 "~" H 5200 2850 60  0000 C CNN
@@
 $EndComp
 $Comp
-L CAPSENSOR QM?
+L CAPSENSOR QM9
 U 1 1 52365855
 P 5950 2850
-F 0 "QM?" H 5910 2970 60  0000 C CNN
+F 0 "QM9" H 5910 2970 60  0000 C CNN
 F 1 "CAPSENSOR" V 6060 2840 40  0001 C CNN
 F 2 "~" H 5950 2850 60  0000 C CNN
@@
 $EndComp
 $Comp
-L CAPSENSOR QM?
+L CAPSENSOR QM2
 U 1 1 5236585B
 P 5200 3350
-F 0 "QM?" H 5160 3470 60  0000 C CNN
+F 0 "QM2" H 5160 3470 60  0000 C CNN
 F 1 "CAPSENSOR" V 5310 3340 40  0001 C CNN
 F 2 "~" H 5200 3350 60  0000 C CNN
@@
 $EndComp
 $Comp
-L CAPSENSOR QM?
+L CAPSENSOR QM10
 U 1 1 52365861
 P 5950 3350
-F 0 "QM?" H 5910 3470 60  0000 C CNN
+F 0 "QM10" H 5910 3470 60  0000 C CNN
 F 1 "CAPSENSOR" V 6060 3340 40  0001 C CNN
 F 2 "~" H 5950 3350 60  0000 C CNN
@@
 $EndComp
 $Comp
-L CAPSENSOR QM?
+L CAPSENSOR QM17
 U 1 1 52365867
 P 6700 2850
-F 0 "QM?" H 6660 2970 60  0000 C CNN
+F 0 "QM17" H 6660 2970 60  0000 C CNN
 F 1 "CAPSENSOR" V 6810 2840 40  0001 C CNN
 F 2 "~" H 6700 2850 60  0000 C CNN
@@
 $EndComp
 $Comp
-L CAPSENSOR QM?
+L CAPSENSOR QM18
 U 1 1 52365873
 P 6700 3350
-F 0 "QM?" H 6660 3470 60  0000 C CNN
+F 0 "QM18" H 6660 3470 60  0000 C CNN
 F 1 "CAPSENSOR" V 6810 3340 40  0001 C CNN
 F 2 "~" H 6700 3350 60  0000 C CNN
@@
 $EndComp
 $Comp
-L CAPSENSOR QM?
+L CAPSENSOR QM3
 U 1 1 523C713D
 P 5200 3850
-F 0 "QM?" H 5160 3970 60  0000 C CNN
+F 0 "QM3" H 5160 3970 60  0000 C CNN
 F 1 "CAPSENSOR" V 5310 3840 40  0001 C CNN
 F 2 "~" H 5200 3850 60  0000 C CNN
@@
 $EndComp
 $Comp
-L CAPSENSOR QM?
+L CAPSENSOR QM4
 U 1 1 523C7143
 P 5200 4350
-F 0 "QM?" H 5160 4470 60  0000 C CNN
+F 0 "QM4" H 5160 4470 60  0000 C CNN
 F 1 "CAPSENSOR" V 5310 4340 40  0001 C CNN
 F 2 "~" H 5200 4350 60  0000 C CNN
@@
 $EndComp
 $Comp
-L CAPSENSOR QM?
+L CAPSENSOR QM11
 U 1 1 523C7149
 P 5950 3850
-F 0 "QM?" H 5910 3970 60  0000 C CNN
+F 0 "QM11" H 5910 3970 60  0000 C CNN
 F 1 "CAPSENSOR" V 6060 3840 40  0001 C CNN
 F 2 "~" H 5950 3850 60  0000 C CNN
@@
 $EndComp
 $Comp
-L CAPSENSOR QM?
+L CAPSENSOR QM19
 U 1 1 523C714F
 P 6700 3850
-F 0 "QM?" H 6660 3970 60  0000 C CNN
+F 0 "QM19" H 6660 3970 60  0000 C CNN
 F 1 "CAPSENSOR" V 6810 3840 40  0001 C CNN
 F 2 "~" H 6700 3850 60  0000 C CNN
@@
 $EndComp
 $Comp
-L CAPSENSOR QM?
+L CAPSENSOR QM12
 U 1 1 523C7155
 P 5950 4350
-F 0 "QM?" H 5910 4470 60  0000 C CNN
+F 0 "QM12" H 5910 4470 60  0000 C CNN
 F 1 "CAPSENSOR" V 6060 4340 40  0001 C CNN
 F 2 "~" H 5950 4350 60  0000 C CNN
@@
 $EndComp
 $Comp
-L CAPSENSOR QM?
+L CAPSENSOR QM20
 U 1 1 523C715B
 P 6700 4350
-F 0 "QM?" H 6660 4470 60  0000 C CNN
+F 0 "QM20" H 6660 4470 60  0000 C CNN
 F 1 "CAPSENSOR" V 6810 4340 40  0001 C CNN
 F 2 "~" H 6700 4350 60  0000 C CNN
@@
 $EndComp
 $Comp
-L CAPSENSOR QM?
+L CAPSENSOR QM5
 U 1 1 523C7161
 P 5200 4850
-F 0 "QM?" H 5160 4970 60  0000 C CNN
+F 0 "QM5" H 5160 4970 60  0000 C CNN
 F 1 "CAPSENSOR" V 5310 4840 40  0001 C CNN
 F 2 "~" H 5200 4850 60  0000 C CNN
@@
 $EndComp
 $Comp
-L CAPSENSOR QM?
+L CAPSENSOR QM13
 U 1 1 523C7167
 P 5950 4850
-F 0 "QM?" H 5910 4970 60  0000 C CNN
+F 0 "QM13" H 5910 4970 60  0000 C CNN
 F 1 "CAPSENSOR" V 6060 4840 40  0001 C CNN
 F 2 "~" H 5950 4850 60  0000 C CNN
@@
 $EndComp
 $Comp
-L CAPSENSOR QM?
+L CAPSENSOR QM6
 U 1 1 523C716D
 P 5200 5350
-F 0 "QM?" H 5160 5470 60  0000 C CNN
+F 0 "QM6" H 5160 5470 60  0000 C CNN
 F 1 "CAPSENSOR" V 5310 5340 40  0001 C CNN
 F 2 "~" H 5200 5350 60  0000 C CNN
@@
 $EndComp
 $Comp
-L CAPSENSOR QM?
+L CAPSENSOR QM14
 U 1 1 523C7173
 P 5950 5350
-F 0 "QM?" H 5910 5470 60  0000 C CNN
+F 0 "QM14" H 5910 5470 60  0000 C CNN
 F 1 "CAPSENSOR" V 6060 5340 40  0001 C CNN
 F 2 "~" H 5950 5350 60  0000 C CNN
@@
 $EndComp
 $Comp
-L CAPSENSOR QM?
+L CAPSENSOR QM21
 U 1 1 523C7179
 P 6700 4850
-F 0 "QM?" H 6660 4970 60  0000 C CNN
+F 0 "QM21" H 6660 4970 60  0000 C CNN
 F 1 "CAPSENSOR" V 6810 4840 40  0001 C CNN
 F 2 "~" H 6700 4850 60  0000 C CNN
@@
 $EndComp
 $Comp
-L CAPSENSOR QM?
+L CAPSENSOR QM22
 U 1 1 523C717F
 P 6700 5350
-F 0 "QM?" H 6660 5470 60  0000 C CNN
+F 0 "QM22" H 6660 5470 60  0000 C CNN
 F 1 "CAPSENSOR" V 6810 5340 40  0001 C CNN
 F 2 "~" H 6700 5350 60  0000 C CNN
@@
 $EndComp
 $Comp
-L CAPSENSOR QM?
+L CAPSENSOR QM7
 U 1 1 523C7185
 P 5200 5850
-F 0 "QM?" H 5160 5970 60  0000 C CNN
+F 0 "QM7" H 5160 5970 60  0000 C CNN
 F 1 "CAPSENSOR" V 5310 5840 40  0001 C CNN
 F 2 "~" H 5200 5850 60  0000 C CNN
@@
 $EndComp
 $Comp
-L CAPSENSOR QM?
+L CAPSENSOR QM8
 U 1 1 523C718B
 P 5200 6350
-F 0 "QM?" H 5160 6470 60  0000 C CNN
+F 0 "QM8" H 5160 6470 60  0000 C CNN
 F 1 "CAPSENSOR" V 5310 6340 40  0001 C CNN
 F 2 "~" H 5200 6350 60  0000 C CNN
@@
 $EndComp
 $Comp
-L CAPSENSOR QM?
+L CAPSENSOR QM15
 U 1 1 523C7191
 P 5950 5850
-F 0 "QM?" H 5910 5970 60  0000 C CNN
+F 0 "QM15" H 5910 5970 60  0000 C CNN
 F 1 "CAPSENSOR" V 6060 5840 40  0001 C CNN
 F 2 "~" H 5950 5850 60  0000 C CNN
@@
 $EndComp
 $Comp
-L CAPSENSOR QM?
+L CAPSENSOR QM23
 U 1 1 523C7197
 P 6700 5850
-F 0 "QM?" H 6660 5970 60  0000 C CNN
+F 0 "QM23" H 6660 5970 60  0000 C CNN
 F 1 "CAPSENSOR" V 6810 5840 40  0001 C CNN
 F 2 "~" H 6700 5850 60  0000 C CNN
@@
 $EndComp
 $Comp
-L CAPSENSOR QM?
+L CAPSENSOR QM16
 U 1 1 523C719D
 P 5950 6350
-F 0 "QM?" H 5910 6470 60  0000 C CNN
+F 0 "QM16" H 5910 6470 60  0000 C CNN
 F 1 "CAPSENSOR" V 6060 6340 40  0001 C CNN
 F 2 "~" H 5950 6350 60  0000 C CNN
@@
 $EndComp
 $Comp
-L CAPSENSOR QM?
+L CAPSENSOR QM24
 U 1 1 523C71A3
 P 6700 6350
-F 0 "QM?" H 6660 6470 60  0000 C CNN
+F 0 "QM24" H 6660 6470 60  0000 C CNN
 F 1 "CAPSENSOR" V 6810 6340 40  0001 C CNN
 F 2 "~" H 6700 6350 60  0000 C CNN
@@
 $EndComp
 $Comp
-L CAPSENSOR QM?
+L CAPSENSOR QM30
 U 1 1 523C79D6
 P 10400 4900
-F 0 "QM?" H 10360 5020 60  0000 C CNN
+F 0 "QM30" H 10360 5020 60  0000 C CNN
 F 1 "CAPSENSOR" V 10510 4890 40  0001 C CNN
 F 2 "" H 10400 4900 60  0001 C CNN
@@
 $EndComp
 $Comp
-L R R?
+L R RS5
 U 1 1 523C79DC
 P 10200 4550
-F 0 "R?" V 10280 4550 50  0000 C CNN
+F 0 "RS5" V 10280 4550 50  0000 C CNN
 F 1 "1k" V 10200 4550 50  0000 C CNN
 F 2 "" H 10200 4550 60  0001 C CNN
@@
 $EndComp
 $Comp
-L R R?
+L R RS4
 U 1 1 523C79E2
 P 10200 3900
-F 0 "R?" V 10280 3900 50  0000 C CNN
+F 0 "RS4" V 10280 3900 50  0000 C CNN
 F 1 "1k" V 10200 3900 50  0000 C CNN
 F 2 "" H 10200 3900 60  0001 C CNN
@@
 $EndComp
 $Comp
-L R R?
+L R RS3
 U 1 1 523C79E8
 P 10200 3250
-F 0 "R?" V 10280 3250 50  0000 C CNN
+F 0 "RS3" V 10280 3250 50  0000 C CNN
 F 1 "1k" V 10200 3250 50  0000 C CNN
 F 2 "" H 10200 3250 60  0001 C CNN
@@
 $EndComp
 $Comp
-L R R?
+L R RS2
 U 1 1 523C79EE
 P 10200 2600
-F 0 "R?" V 10280 2600 50  0000 C CNN
+F 0 "RS2" V 10280 2600 50  0000 C CNN
 F 1 "1k" V 10200 2600 50  0000 C CNN
 F 2 "" H 10200 2600 60  0001 C CNN
@@
 $EndComp
 $Comp
-L R R?
+L R RS1
 U 1 1 523C79F4
 P 10200 1950
-F 0 "R?" V 10280 1950 50  0000 C CNN
+F 0 "RS1" V 10280 1950 50  0000 C CNN
 F 1 "1k" V 10200 1950 50  0000 C CNN
 F 2 "" H 10200 1950 60  0001 C CNN
@@
 $EndComp
 $Comp
-L CAPSENSOR QM?
+L CAPSENSOR QM29
 U 1 1 523C79FA
 P 10400 4250
-F 0 "QM?" H 10360 4370 60  0000 C CNN
+F 0 "QM29" H 10360 4370 60  0000 C CNN
 F 1 "CAPSENSOR" V 10510 4240 40  0001 C CNN
 F 2 "" H 10400 4250 60  0001 C CNN
@@
 $EndComp
 $Comp
-L CAPSENSOR QM?
+L CAPSENSOR QM28
 U 1 1 523C7A00
 P 10400 3600
-F 0 "QM?" H 10360 3720 60  0000 C CNN
+F 0 "QM28" H 10360 3720 60  0000 C CNN
 F 1 "CAPSENSOR" V 10510 3590 40  0001 C CNN
 F 2 "" H 10400 3600 60  0001 C CNN
@@
 $EndComp
 $Comp
-L CAPSENSOR QM?
+L CAPSENSOR QM27
 U 1 1 523C7A06
 P 10400 2950
-F 0 "QM?" H 10360 3070 60  0000 C CNN
+F 0 "QM27" H 10360 3070 60  0000 C CNN
 F 1 "CAPSENSOR" V 10510 2940 40  0001 C CNN
 F 2 "" H 10400 2950 60  0001 C CNN
@@
 $EndComp
 $Comp
-L CAPSENSOR QM?
+L CAPSENSOR QM26
 U 1 1 523C7A0C
 P 10400 2300
-F 0 "QM?" H 10360 2420 60  0000 C CNN
+F 0 "QM26" H 10360 2420 60  0000 C CNN
 F 1 "CAPSENSOR" V 10510 2290 40  0001 C CNN
 F 2 "" H 10400 2300 60  0001 C CNN
@@
 $EndComp
 $Comp
-L CAPSENSOR QM?
+L CAPSENSOR QM25
 U 1 1 523C7A12
 P 10400 1650
-F 0 "QM?" H 10360 1770 60  0000 C CNN
+F 0 "QM25" H 10360 1770 60  0000 C CNN
 F 1 "CAPSENSOR" V 10510 1640 40  0001 C CNN
 F 2 "" H 10400 1650 60  0001 C CNN
@@
 $EndComp
 $Comp
-L CAPSENSOR QM?
+L CAPSENSOR QM31
 U 1 1 523C7A23
 P 10400 5550
-F 0 "QM?" H 10360 5670 60  0000 C CNN
+F 0 "QM31" H 10360 5670 60  0000 C CNN
 F 1 "CAPSENSOR" V 10510 5540 40  0001 C CNN
 F 2 "" H 10400 5550 60  0001 C CNN
@@
 $EndComp
 $Comp
-L R R?
+L R RS6
 U 1 1 523C7A29
 P 10200 5200
-F 0 "R?" V 10280 5200 50  0000 C CNN
+F 0 "RS6" V 10280 5200 50  0000 C CNN
 F 1 "1k" V 10200 5200 50  0000 C CNN
 F 2 "" H 10200 5200 60  0001 C CNN
@@
 $EndComp
 $Comp
-L CAPSENSOR QM?
+L CAPSENSOR QM32
 U 1 1 523C7A3A
 P 10400 6200
-F 0 "QM?" H 10360 6320 60  0000 C CNN
+F 0 "QM32" H 10360 6320 60  0000 C CNN
 F 1 "CAPSENSOR" V 10510 6190 40  0001 C CNN
 F 2 "" H 10400 6200 60  0001 C CNN
@@
 $EndComp
 $Comp
-L R R?
+L R RS7
 U 1 1 523C7A40
 P 10200 5850
-F 0 "R?" V 10280 5850 50  0000 C CNN
+F 0 "RS7" V 10280 5850 50  0000 C CNN
 F 1 "1k" V 10200 5850 50  0000 C CNN
 F 2 "" H 10200 5850 60  0001 C CNN
@@
 Sensor_AIN0
 $Comp
-L GND #PWR?
+L GND #PWR1
 U 1 1 523C799A
 P 8550 8900
-F 0 "#PWR?" H 8550 8900 30  0001 C CNN
+F 0 "#PWR1" H 8550 8900 30  0001 C CNN
 F 1 "GND" H 8550 8830 30  0001 C CNN
 F 2 "" H 8550 8900 60  0001 C CNN
