File: Hardware/Sensors.sch (KiCad schematic (older format))
At the start: 59 parts

Commit message: Added slider, more capacitive sensors, and several ICs. Continuing board layout.
Parts:
- removed QM25, QM26, QM27, QM28, QM29, QM30, QM31, QM32: CAPSENSOR, symbol CAPSENSOR
- added U10: CAPSLIDER, symbol CAPSLIDER
Connections:
- wire segments 185 -> 169
Other:
- moved on the sheet: RSMP3, RY3
Changed lines of the file:
@@
 Sheet 3 7
 Title "Pong.0"
-Date "16 nov 2013"
+Date "22 feb 2014"
 Rev "0.3"
 Comp "Projects and Stuff LLC"
@@
 6E 56 52 49 51 4E 59 71 7E 65 C5 4D 0F AF 00 BF F6 21 9D BA 45 88 9C 00 16 00 C0 66 90 E0 00 00
 AC 42 3B 38 00 00 AB 90 E0 00 00 AC 42 82 03 00 B0 EA FF 00 E3 76 B5 A7 81 B6 BC 08 00 00 00 00
-49 45 4E 44 AE 42 60 82 89 $EndBitmap
+49 45 4E 44 AE 42 60 82 AD $EndBitmap
 EndData
 $EndBitmap
@@
 $EndComp
 $Comp
-L CAPSENSOR QM30
-U 1 1 523C79D6
-P 10400 4900
-F 0 "QM30" H 10360 5020 60  0000 C CNN
-F 1 "CAPSENSOR" V 10510 4890 40  0001 C CNN
-F 2 "" H 10400 4900 60  0001 C CNN
-F 3 "" H 10400 4900 60  0001 C CNN
-	1    10400 4900
-	1    0    0    -1
-$EndComp
-$Comp
 L R RS5
 U 1 1 523C79DC
@@
 $EndComp
 $Comp
-L CAPSENSOR QM29
-U 1 1 523C79FA
-P 10400 4250
-F 0 "QM29" H 10360 4370 60  0000 C CNN
-F 1 "CAPSENSOR" V 10510 4240 40  0001 C CNN
-F 2 "" H 10400 4250 60  0001 C CNN
-F 3 "" H 10400 4250 60  0001 C CNN
-	1    10400 4250
-	1    0    0    -1
-$EndComp
-$Comp
-L CAPSENSOR QM28
-U 1 1 523C7A00
-P 10400 3600
-F 0 "QM28" H 10360 3720 60  0000 C CNN
-F 1 "CAPSENSOR" V 10510 3590 40  0001 C CNN
-F 2 "" H 10400 3600 60  0001 C CNN
-F 3 "" H 10400 3600 60  0001 C CNN
-	1    10400 3600
-	1    0    0    -1
-$EndComp
-$Comp
-L CAPSENSOR QM27
-U 1 1 523C7A06
-P 10400 2950
-F 0 "QM27" H 10360 3070 60  0000 C CNN
-F 1 "CAPSENSOR" V 10510 2940 40  0001 C CNN
-F 2 "" H 10400 2950 60  0001 C CNN
-F 3 "" H 10400 2950 60  0001 C CNN
-	1    10400 2950
-	1    0    0    -1
-$EndComp
-$Comp
-L CAPSENSOR QM26
-U 1 1 523C7A0C
-P 10400 2300
-F 0 "QM26" H 10360 2420 60  0000 C CNN
-F 1 "CAPSENSOR" V 10510 2290 40  0001 C CNN
-F 2 "" H 10400 2300 60  0001 C CNN
-F 3 "" H 10400 2300 60  0001 C CNN
-	1    10400 2300
-	1    0    0    -1
-$EndComp
-$Comp
-L CAPSENSOR QM25
-U 1 1 523C7A12
-P 10400 1650
-F 0 "QM25" H 10360 1770 60  0000 C CNN
-F 1 "CAPSENSOR" V 10510 1640 40  0001 C CNN
-F 2 "" H 10400 1650 60  0001 C CNN
-F 3 "" H 10400 1650 60  0001 C CNN
-	1    10400 1650
-	1    0    0    -1
-$EndComp
-$Comp
-L CAPSENSOR QM31
-U 1 1 523C7A23
-P 10400 5550
-F 0 "QM31" H 10360 5670 60  0000 C CNN
-F 1 "CAPSENSOR" V 10510 5540 40  0001 C CNN
-F 2 "" H 10400 5550 60  0001 C CNN
-F 3 "" H 10400 5550 60  0001 C CNN
-	1    10400 5550
-	1    0    0    -1
-$EndComp
-$Comp
 L R RS6
 U 1 1 523C7A29
@@
 F 3 "" H 10200 5200 60  0001 C CNN
 	1    10200 5200
-	1    0    0    -1
-$EndComp
-$Comp
-L CAPSENSOR QM32
-U 1 1 523C7A3A
-P 10400 6200
-F 0 "QM32" H 10360 6320 60  0000 C CNN
-F 1 "CAPSENSOR" V 10510 6190 40  0001 C CNN
-F 2 "" H 10400 6200 60  0001 C CNN
-F 3 "" H 10400 6200 60  0001 C CNN
-	1    10400 6200
 	1    0    0    -1
 $EndComp
@@
 Text HLabel 4400 6350 0    60   Input ~ 0
 Sensor_X7
-Connection ~ 10600 4450
-Wire Wire Line
-	10600 4450 10400 4450
-Wire Wire Line
-	10400 4450 10400 4400
-Wire Wire Line
-	10600 3150 10400 3150
-Wire Wire Line
-	10400 3150 10400 3100
-Wire Wire Line
-	10600 1850 10400 1850
-Wire Wire Line
-	10400 1850 10400 1800
 Wire Wire Line
 	10200 4800 10200 4950
@@
 Connection ~ 10200 4900
 Wire Wire Line
-	10400 2450 10400 2500
-Wire Wire Line
-	10400 2500 10600 2500
-Wire Wire Line
-	10400 3750 10400 3800
-Wire Wire Line
-	10400 3800 10600 3800
-Wire Wire Line
-	10400 5050 10400 5100
-Wire Wire Line
-	10400 5100 10600 5100
-Connection ~ 10600 5100
-Wire Wire Line
 	10200 5450 10200 5600
 Connection ~ 10200 5550
 Wire Wire Line
-	10400 5700 10400 5750
-Wire Wire Line
-	10400 5750 10600 5750
-Wire Wire Line
 	10200 6100 10200 6200
 Connection ~ 10200 6200
 Wire Wire Line
-	10400 6350 10400 6400
-Wire Wire Line
-	10400 6400 10600 6400
-Wire Wire Line
 	10200 6200 10250 6200
 Wire Wire Line
@@
 Wire Wire Line
 	10200 2300 10250 2300
-Wire Wire Line
-	10600 1850 10600 6600
-Connection ~ 10600 2500
-Connection ~ 10600 3150
-Connection ~ 10600 3800
-Connection ~ 10600 5750
-Connection ~ 10600 6400
 Wire Wire Line
 	9500 1600 10200 1600
@@
 	6700 8050 6700 8000
 Wire Wire Line
-	5150 8050 10600 8050
+	5150 8050 10700 8050
 Connection ~ 5950 8050
 Connection ~ 5200 8050
@@
 Sensor_AIN0
 $Comp
-L GND #PWR021
+L GND #PWR21
 U 1 1 523C799A
 P 8550 8900
-F 0 "#PWR021" H 8550 8900 30  0001 C CNN
+F 0 "#PWR21" H 8550 8900 30  0001 C CNN
 F 1 "GND" H 8550 8830 30  0001 C CNN
 F 2 "" H 8550 8900 60  0001 C CNN
@@
 L R RY3
 U 1 1 523CDC23
-P 10600 6850
-F 0 "RY3" V 10680 6850 50  0000 C CNN
-F 1 "1k" V 10600 6850 50  0000 C CNN
-F 2 "" H 10600 6850 60  0001 C CNN
-F 3 "" H 10600 6850 60  0001 C CNN
-	1    10600 6850
+P 10700 6850
+F 0 "RY3" V 10780 6850 50  0000 C CNN
+F 1 "1k" V 10700 6850 50  0000 C CNN
+F 2 "" H 10700 6850 60  0001 C CNN
+F 3 "" H 10700 6850 60  0001 C CNN
+	1    10700 6850
 	1    0    0    -1
 $EndComp
@@
 L CSMALL CS3
 U 1 1 523CDC29
-P 10600 7300
-F 0 "CS3" H 10625 7350 30  0000 L CNN
-F 1 "4.7nF" H 10625 7250 30  0000 L CNN
-F 2 "~" H 10600 7300 60  0000 C CNN
-F 3 "~" H 10600 7300 60  0000 C CNN
-	1    10600 7300
+P 10700 7300
+F 0 "CS3" H 10725 7350 30  0000 L CNN
+F 1 "4.7nF" H 10725 7250 30  0000 L CNN
+F 2 "~" H 10700 7300 60  0000 C CNN
+F 3 "~" H 10700 7300 60  0000 C CNN
+	1    10700 7300
 	1    0    0    -1
 $EndComp
@@
 L R RSMP3
 U 1 1 523CDC2F
-P 10600 7750
-F 0 "RSMP3" V 10680 7750 50  0000 C CNN
-F 1 "470k" V 10600 7750 50  0000 C CNN
-F 2 "" H 10600 7750 60  0001 C CNN
-F 3 "" H 10600 7750 60  0001 C CNN
-	1    10600 7750
-	1    0    0    -1
-$EndComp
-Text HLabel 10550 7150 0    60   Input ~ 0
+P 10700 7750
+F 0 "RSMP3" V 10780 7750 50  0000 C CNN
+F 1 "470k" V 10700 7750 50  0000 C CNN
+F 2 "" H 10700 7750 60  0001 C CNN
+F 3 "" H 10700 7750 60  0001 C CNN
+	1    10700 7750
+	1    0    0    -1
+$EndComp
+Text HLabel 10650 7150 0    60   Input ~ 0
 Sensor_Y3A
-Text HLabel 10550 7450 0    60   Input ~ 0
+Text HLabel 10650 7450 0    60   Input ~ 0
 Sensor_Y3B
 Wire Wire Line
-	10600 7100 10600 7200
-Wire Wire Line
-	10600 7400 10600 7500
-Wire Wire Line
-	10600 7150 10550 7150
-Connection ~ 10600 7150
-Wire Wire Line
-	10600 7450 10550 7450
-Connection ~ 10600 7450
-Wire Wire Line
-	10600 8050 10600 8000
+	10700 7100 10700 7200
+Wire Wire Line
+	10700 7400 10700 7500
+Wire Wire Line
+	10700 7150 10650 7150
+Connection ~ 10700 7150
+Wire Wire Line
+	10700 7450 10650 7450
+Connection ~ 10700 7450
 Connection ~ 6700 8050
+$Comp
+L CAPSLIDER U10
+U 1 1 53090843
+P 10700 6200
+F 0 "U10" H 10800 6000 60  0000 C CNN
+F 1 "CAPSLIDER" H 10700 10850 60  0000 C CNN
+F 2 "" H 10700 6200 60  0000 C CNN
+F 3 "" H 10700 6200 60  0000 C CNN
+	1    10700 6200
+	1    0    0    -1
+$EndComp
+Wire Wire Line
+	10700 8050 10700 8000
+Wire Wire Line
+	10700 6500 10700 6600
 $EndSCHEMATC
