File: Hardware/Slider.sch (KiCad schematic (older format))
At the start: 0 parts

Commit message: Added Slider. Imported Sheet Pins. Made other minor adjustments to schematics.
Parts:
- added C?: 4.7nF, symbol CSMALL
- added QM? (x8): CAPSENSOR, symbol CAPSENSOR
- added R? (x16): 1k, symbol R
- added R?: 470k, symbol R
Connections:
- net labels added: AIN0, SMP, X0, X1, X2, X3, X4, X5, X6, X7, Y3A, Y3B
- net labels removed: 3_3V, 5V, D+, D-, VBUS
- wire segments 7 -> 57
Other:
- note added: "This block copied from another project. Requires\nverification and update to comply with XMega."

Commit message: Continued populating the schematics.
Connections:
- net labels added: Slider_AIN0, Slider_SMP, Slider_X0, Slider_X1, Slider_X2, Slider_X3, Slider_X4, Slider_X5, Slider_X6, Slider_X7, Slider_Y3A, Slider_Y3B
- net labels removed: AIN0, SMP, X0, X1, X2, X3, X4, X5, X6, X7, Y3A, Y3B
Changed lines of the file:
@@
 $Descr B 17000 11000
 encoding utf-8
-Sheet 7 7
+Sheet 6 8
 Title "Pong.0"
-Date "12 sep 2013"
-Rev "0.2"
+Date "19 sep 2013"
+Rev "0.3"
 Comp "Projects and Stuff LLC"
 Comment1 ""
@@
 6E 56 52 49 51 4E 59 71 7E 65 C5 4D 0F AF 00 BF F6 21 9D BA 45 88 9C 00 16 00 C0 66 90 E0 00 00
 AC 42 3B 38 00 00 AB 90 E0 00 00 AC 42 82 03 00 B0 EA FF 00 E3 76 B5 A7 81 B6 BC 08 00 00 00 00
-49 45 4E 44 AE 42 60 82 DC $EndBitmap
+49 45 4E 44 AE 42 60 82 20 $EndBitmap
 EndData
 $EndBitmap
@@
 	1    0    0    -1
 $EndComp
-Text Label 6550 8050 2    60   ~ 0
-AIN0
-Text Label 5600 4750 2    60   ~ 0
-X5
-Text Label 5600 4100 2    60   ~ 0
-X4
-Text Label 5600 3450 2    60   ~ 0
-X3
-Text Label 5600 2800 2    60   ~ 0
-X2
-Text Label 5600 2150 2    60   ~ 0
-X1
-Text Label 5600 1500 2    60   ~ 0
-X0
-Text Label 6550 7200 2    60   ~ 0
-Y3B
-Text Label 6550 6900 2    60   ~ 0
-Y3A
-Text Label 6550 7800 2    60   ~ 0
-SMP
 $Comp
 L CSMALL C?
@@
 P 6400 4800
 F 0 "QM?" H 6360 4920 60  0000 C CNN
-F 1 "CAPSENSOR" V 6510 4790 40  0000 C CNN
+F 1 "CAPSENSOR" V 6510 4790 40  0001 C CNN
 F 2 "" H 6400 4800 60  0001 C CNN
 F 3 "" H 6400 4800 60  0001 C CNN
@@
 P 6400 4150
 F 0 "QM?" H 6360 4270 60  0000 C CNN
-F 1 "CAPSENSOR" V 6510 4140 40  0000 C CNN
+F 1 "CAPSENSOR" V 6510 4140 40  0001 C CNN
 F 2 "" H 6400 4150 60  0001 C CNN
 F 3 "" H 6400 4150 60  0001 C CNN
@@
 P 6400 3500
 F 0 "QM?" H 6360 3620 60  0000 C CNN
-F 1 "CAPSENSOR" V 6510 3490 40  0000 C CNN
+F 1 "CAPSENSOR" V 6510 3490 40  0001 C CNN
 F 2 "" H 6400 3500 60  0001 C CNN
 F 3 "" H 6400 3500 60  0001 C CNN
@@
 P 6400 2850
 F 0 "QM?" H 6360 2970 60  0000 C CNN
-F 1 "CAPSENSOR" V 6510 2840 40  0000 C CNN
+F 1 "CAPSENSOR" V 6510 2840 40  0001 C CNN
 F 2 "" H 6400 2850 60  0001 C CNN
 F 3 "" H 6400 2850 60  0001 C CNN
@@
 P 6400 2200
 F 0 "QM?" H 6360 2320 60  0000 C CNN
-F 1 "CAPSENSOR" V 6510 2190 40  0000 C CNN
+F 1 "CAPSENSOR" V 6510 2190 40  0001 C CNN
 F 2 "" H 6400 2200 60  0001 C CNN
 F 3 "" H 6400 2200 60  0001 C CNN
@@
 P 6400 1550
 F 0 "QM?" H 6360 1670 60  0000 C CNN
-F 1 "CAPSENSOR" V 6510 1540 40  0000 C CNN
+F 1 "CAPSENSOR" V 6510 1540 40  0001 C CNN
 F 2 "" H 6400 1550 60  0001 C CNN
 F 3 "" H 6400 1550 60  0001 C CNN
@@
 Wire Wire Line
 	6400 5650 6600 5650
-Text Label 5600 5400 2    60   ~ 0
-X6
 $Comp
 L R R?
@@
 P 6400 5450
 F 0 "QM?" H 6360 5570 60  0000 C CNN
-F 1 "CAPSENSOR" V 6510 5440 40  0000 C CNN
+F 1 "CAPSENSOR" V 6510 5440 40  0001 C CNN
 F 2 "" H 6400 5450 60  0001 C CNN
 F 3 "" H 6400 5450 60  0001 C CNN
@@
 P 6400 6100
 F 0 "QM?" H 6360 6220 60  0000 C CNN
-F 1 "CAPSENSOR" V 6510 6090 40  0000 C CNN
+F 1 "CAPSENSOR" V 6510 6090 40  0001 C CNN
 F 2 "" H 6400 6100 60  0001 C CNN
 F 3 "" H 6400 6100 60  0001 C CNN
@@
 	1    0    0    -1
 $EndComp
-Text Label 5600 6050 2    60   ~ 0
-X7
 Wire Wire Line
 	6200 6100 6250 6100
@@
 Text Notes 6950 4350 0    60   ~ 0
 This block copied from another project. Requires\nverification and update to comply with XMega.
+Text HLabel 5600 1500 0    60   Input ~ 0
+Slider_X0
+Text HLabel 5600 2150 0    60   Input ~ 0
+Slider_X1
+Text HLabel 5600 2800 0    60   Input ~ 0
+Slider_X2
+Text HLabel 5600 3450 0    60   Input ~ 0
+Slider_X3
+Text HLabel 5600 4100 0    60   Input ~ 0
+Slider_X4
+Text HLabel 5600 4750 0    60   Input ~ 0
+Slider_X5
+Text HLabel 5600 5400 0    60   Input ~ 0
+Slider_X6
+Text HLabel 5600 6050 0    60   Input ~ 0
+Slider_X7
+Text HLabel 6550 6900 0    60   Input ~ 0
+Slider_Y3A
+Text HLabel 6550 7200 0    60   Input ~ 0
+Slider_Y3B
+Text HLabel 6550 7800 0    60   Input ~ 0
+Slider_SMP
+Text HLabel 6550 8050 0    60   Input ~ 0
+Slider_AIN0
 $EndSCHEMATC
