File: Hardware/PowerManagement.sch (KiCad schematic (older format))
At the start: 30 parts

Commit message: Corrected Label Names
Connections:
- net labels removed: PWR_GND, PWR_VBUS
- wire segments 117 -> 113
Other:
- note added: "(Should there be a series resistor?)"
- note removed: "(Are these really needed if pull-ups are available\nelsewhere? Whould there be a series resistor?)"
Changed lines of the file:
@@
 Sheet 3 7
 Title "Pong.0"
-Date "24 sep 2013"
+Date "25 sep 2013"
 Rev "0.3"
 Comp "Projects and Stuff LLC"
@@
 	4400 3200 4400 3250
 Connection ~ 4400 3250
-Text HLabel 4450 2950 2    60   Input ~ 0
-PWR_VBUS
-Wire Wire Line
-	4450 2950 4400 2950
-Wire Wire Line
-	4400 2950 4400 3000
-Connection ~ 4400 3000
 Text HLabel 4450 3400 2    60   Input ~ 0
 PWR_D+
@@
 Wire Wire Line
 	9850 5250 9900 5250
-Text Notes 10450 4800 2    30   Italic 0
-(Are these really needed if pull-ups are available\nelsewhere? Whould there be a series resistor?)
+Text Notes 9200 5400 2    30   Italic 0
+(Should there be a series resistor?)
 Wire Wire Line
 	8850 4700 8850 4650
@@
 PWR_3_3V
 NoConn ~ 7800 3350
-Text HLabel 4450 5100 2    60   Input ~ 0
-PWR_GND
-$Comp
-L GND #PWR?
-U 1 1 52168E05
-P 4400 5150
-F 0 "#PWR?" H 4400 5150 30  0001 C CNN
-F 1 "GND" H 4400 5080 30  0001 C CNN
-F 2 "" H 4400 5150 60  0000 C CNN
-F 3 "" H 4400 5150 60  0000 C CNN
-	1    4400 5150
-	1    0    0    -1
-$EndComp
-Wire Wire Line
-	4450 5100 4400 5100
-Wire Wire Line
-	4400 5100 4400 5150
 Wire Wire Line
 	2250 3900 2250 3950
@@
 6E 56 52 49 51 4E 59 71 7E 65 C5 4D 0F AF 00 BF F6 21 9D BA 45 88 9C 00 16 00 C0 66 90 E0 00 00
 AC 42 3B 38 00 00 AB 90 E0 00 00 AC 42 82 03 00 B0 EA FF 00 E3 76 B5 A7 81 B6 BC 08 00 00 00 00
-49 45 4E 44 AE 42 60 82 81 $EndBitmap
+49 45 4E 44 AE 42 60 82 D0 $EndBitmap
 EndData
 $EndBitmap

Commit message: Minor misc changes
Parts:
- removed C?: 10uF, ~, symbol CSMALL
- added C?: 10uF, symbol CPOLSMALL
Changed lines of the file:
@@
 $Descr B 17000 11000
 encoding utf-8
-Sheet 3 7
+Sheet 2 7
 Title "Pong.0"
 Date "25 sep 2013"
@@
 Connection ~ 8900 2400
 $Comp
-L GND #PWR?
+L GND #PWR01
 U 1 1 52163D8A
 P 8900 2700
-F 0 "#PWR?" H 8900 2700 30  0001 C CNN
+F 0 "#PWR01" H 8900 2700 30  0001 C CNN
 F 1 "GND" H 8900 2630 30  0001 C CNN
 F 2 "" H 8900 2700 60  0000 C CNN
@@
 	8900 2650 8900 2700
 $Comp
-L CSMALL C?
-U 1 1 52163DB6
-P 7850 3100
-F 0 "C?" H 7875 3150 30  0000 L CNN
-F 1 "10uF" H 7875 3050 30  0000 L CNN
-F 2 "~" H 7850 3100 60  0000 C CNN
-F 3 "~" H 7850 3100 60  0000 C CNN
-	1    7850 3100
-	1    0    0    -1
-$EndComp
-$Comp
-L GND #PWR?
+L GND #PWR02
 U 1 1 52163DBE
 P 7850 3250
-F 0 "#PWR?" H 7850 3250 30  0001 C CNN
+F 0 "#PWR02" H 7850 3250 30  0001 C CNN
 F 1 "GND" H 7850 3180 30  0001 C CNN
 F 2 "" H 7850 3250 60  0000 C CNN
@@
 	5750 2600 5750 2650
 $Comp
-L GND #PWR?
+L GND #PWR03
 U 1 1 52164179
 P 5750 2900
-F 0 "#PWR?" H 5750 2900 30  0001 C CNN
+F 0 "#PWR03" H 5750 2900 30  0001 C CNN
 F 1 "GND" H 5750 2830 30  0001 C CNN
 F 2 "" H 5750 2900 60  0000 C CNN
@@
 	5550 2400 5550 2450
 $Comp
-L GND #PWR?
+L GND #PWR04
 U 1 1 5216431B
 P 5550 2700
-F 0 "#PWR?" H 5550 2700 30  0001 C CNN
+F 0 "#PWR04" H 5550 2700 30  0001 C CNN
 F 1 "GND" H 5550 2630 30  0001 C CNN
 F 2 "" H 5550 2700 60  0000 C CNN
@@
 $EndComp
 $Comp
-L GND #PWR?
+L GND #PWR05
 U 1 1 521647BC
 P 5750 3500
-F 0 "#PWR?" H 5750 3500 30  0001 C CNN
+F 0 "#PWR05" H 5750 3500 30  0001 C CNN
 F 1 "GND" H 5750 3430 30  0001 C CNN
 F 2 "" H 5750 3500 60  0000 C CNN
@@
 $EndComp
 $Comp
-L GND #PWR?
+L GND #PWR06
 U 1 1 521647FC
 P 5550 3300
-F 0 "#PWR?" H 5550 3300 30  0001 C CNN
+F 0 "#PWR06" H 5550 3300 30  0001 C CNN
 F 1 "GND" H 5550 3230 30  0001 C CNN
 F 2 "" H 5550 3300 60  0000 C CNN
@@
 	5750 3600 5750 3650
 $Comp
-L GND #PWR?
+L GND #PWR07
 U 1 1 52164A60
 P 5750 3900
-F 0 "#PWR?" H 5750 3900 30  0001 C CNN
+F 0 "#PWR07" H 5750 3900 30  0001 C CNN
 F 1 "GND" H 5750 3830 30  0001 C CNN
 F 2 "" H 5750 3900 60  0000 C CNN
@@
 	5000 4600 5800 4600
 $Comp
-L GND #PWR?
+L GND #PWR08
 U 1 1 521650D5
 P 3100 3650
-F 0 "#PWR?" H 3100 3650 30  0001 C CNN
+F 0 "#PWR08" H 3100 3650 30  0001 C CNN
 F 1 "GND" H 3100 3580 30  0001 C CNN
 F 2 "" H 3100 3650 60  0000 C CNN
@@
 	5150 2400 5150 2450
 $Comp
-L GND #PWR?
+L GND #PWR09
 U 1 1 52165390
 P 5150 2900
-F 0 "#PWR?" H 5150 2900 30  0001 C CNN
+F 0 "#PWR09" H 5150 2900 30  0001 C CNN
 F 1 "GND" H 5150 2830 30  0001 C CNN
 F 2 "" H 5150 2900 60  0000 C CNN
@@
 	5150 2850 5150 2900
 $Comp
-L GND #PWR?
+L GND #PWR010
 U 1 1 52165559
 P 6950 5950
-F 0 "#PWR?" H 6950 5950 30  0001 C CNN
+F 0 "#PWR010" H 6950 5950 30  0001 C CNN
 F 1 "GND" H 6950 5880 30  0001 C CNN
 F 2 "" H 6950 5950 60  0000 C CNN
@@
 Connection ~ 7850 3550
 $Comp
-L GND #PWR?
+L GND #PWR011
 U 1 1 52165BB9
 P 8350 3850
-F 0 "#PWR?" H 8350 3850 30  0001 C CNN
+F 0 "#PWR011" H 8350 3850 30  0001 C CNN
 F 1 "GND" H 8350 3780 30  0001 C CNN
 F 2 "" H 8350 3850 60  0000 C CNN
@@
 (At least\n1uF)
 $Comp
-L GND #PWR?
+L GND #PWR012
 U 1 1 52165D09
 P 8900 4250
-F 0 "#PWR?" H 8900 4250 30  0001 C CNN
+F 0 "#PWR012" H 8900 4250 30  0001 C CNN
 F 1 "GND" H 8900 4180 30  0001 C CNN
 F 2 "" H 8900 4250 60  0000 C CNN
@@
 Connection ~ 7950 4300
 $Comp
-L GND #PWR?
+L GND #PWR013
 U 1 1 52166403
 P 7950 4950
-F 0 "#PWR?" H 7950 4950 30  0001 C CNN
+F 0 "#PWR013" H 7950 4950 30  0001 C CNN
 F 1 "GND" H 7950 4880 30  0001 C CNN
 F 2 "" H 7950 4950 60  0000 C CNN
@@
 Connection ~ 7950 4350
 $Comp
-L GND #PWR?
+L GND #PWR014
 U 1 1 5216692D
 P 8400 4950
-F 0 "#PWR?" H 8400 4950 30  0001 C CNN
+F 0 "#PWR014" H 8400 4950 30  0001 C CNN
 F 1 "GND" H 8400 4880 30  0001 C CNN
 F 2 "" H 8400 4950 60  0000 C CNN
@@
 Connection ~ 2400 4600
 $Comp
-L GND #PWR?
+L GND #PWR015
 U 1 1 5216AE04
 P 2400 4650
-F 0 "#PWR?" H 2400 4650 30  0001 C CNN
+F 0 "#PWR015" H 2400 4650 30  0001 C CNN
 F 1 "GND" H 2400 4580 30  0001 C CNN
 F 2 "" H 2400 4650 60  0000 C CNN
@@
 	4350 3450 5000 3450
 $Comp
-L GND #PWR?
+L GND #PWR016
 U 1 1 5216EA73
 P 4000 3700
-F 0 "#PWR?" H 4000 3700 30  0001 C CNN
+F 0 "#PWR016" H 4000 3700 30  0001 C CNN
 F 1 "GND" H 4000 3630 30  0001 C CNN
 F 2 "" H 4000 3700 60  0000 C CNN
@@
 	4000 3650 4000 3700
 $Comp
-L GND #PWR?
+L GND #PWR017
 U 1 1 522CBB9B
 P 6450 5900
-F 0 "#PWR?" H 6450 5900 30  0001 C CNN
+F 0 "#PWR017" H 6450 5900 30  0001 C CNN
 F 1 "GND" H 6450 5830 30  0001 C CNN
 F 2 "" H 6450 5900 60  0000 C CNN
@@
 Connection ~ 10800 2950
 $Comp
-L GND #PWR?
+L GND #PWR018
 U 1 1 522CCD85
 P 10800 3250
-F 0 "#PWR?" H 10800 3250 30  0001 C CNN
+F 0 "#PWR018" H 10800 3250 30  0001 C CNN
 F 1 "GND" H 10800 3180 30  0001 C CNN
 F 2 "" H 10800 3250 60  0000 C CNN
@@
 	12450 3250 12400 3250
 $Comp
-L GND #PWR?
+L GND #PWR019
 U 1 1 522CCEBE
 P 12450 3300
-F 0 "#PWR?" H 12450 3300 30  0001 C CNN
+F 0 "#PWR019" H 12450 3300 30  0001 C CNN
 F 1 "GND" H 12450 3230 30  0001 C CNN
 F 2 "" H 12450 3300 60  0000 C CNN
@@
 Connection ~ 12450 2750
 $Comp
-L GND #PWR?
+L GND #PWR020
 U 1 1 522CD09B
 P 12600 3050
-F 0 "#PWR?" H 12600 3050 30  0001 C CNN
+F 0 "#PWR020" H 12600 3050 30  0001 C CNN
 F 1 "GND" H 12600 2980 30  0001 C CNN
 F 2 "" H 12600 3050 60  0000 C CNN
@@
 6E 56 52 49 51 4E 59 71 7E 65 C5 4D 0F AF 00 BF F6 21 9D BA 45 88 9C 00 16 00 C0 66 90 E0 00 00
 AC 42 3B 38 00 00 AB 90 E0 00 00 AC 42 82 03 00 B0 EA FF 00 E3 76 B5 A7 81 B6 BC 08 00 00 00 00
-49 45 4E 44 AE 42 60 82 D0 $EndBitmap
+49 45 4E 44 AE 42 60 82 D7 $EndBitmap
 EndData
 $EndBitmap
@@
 EndData
 $EndBitmap
+$Comp
+L CPOLSMALL C?
+U 1 1 5243CD1A
+P 7850 3150
+F 0 "C?" H 7900 3250 28  0000 C CNN
+F 1 "10uF" H 7875 3125 28  0000 L CNN
+F 2 "" H 7850 3150 60  0000 C CNN
+F 3 "" H 7850 3150 60  0000 C CNN
+	1    7850 3150
+	1    0    0    -1
+$EndComp
 $EndSCHEMATC

Commit message: Minor cosmetic changes
Other:
- note removed: "(Should there be a series resistor?)"
Changed lines of the file:
@@
 Sheet 2 7
 Title "Pong.0"
-Date "25 sep 2013"
+Date "26 sep 2013"
 Rev "0.3"
 Comp "Projects and Stuff LLC"
@@
 Wire Wire Line
 	9850 5250 9900 5250
-Text Notes 9200 5400 2    30   Italic 0
-(Should there be a series resistor?)
 Wire Wire Line
 	8850 4700 8850 4650
@@
 6E 56 52 49 51 4E 59 71 7E 65 C5 4D 0F AF 00 BF F6 21 9D BA 45 88 9C 00 16 00 C0 66 90 E0 00 00
 AC 42 3B 38 00 00 AB 90 E0 00 00 AC 42 82 03 00 B0 EA FF 00 E3 76 B5 A7 81 B6 BC 08 00 00 00 00
-49 45 4E 44 AE 42 60 82 D7 $EndBitmap
+49 45 4E 44 AE 42 60 82 79 $EndBitmap
 EndData
 $EndBitmap

Commit message: Annotated Schematics
Parts:
- gave numbers to parts that had none: 30

Commit message: Made corrections based on ERC results
Connections:
- wire segments 113 -> 114
- no-connect marks 1 -> 2
Changed lines of the file:
@@
 Connection ~ 8900 2400
 $Comp
-L GND #PWR16
+L GND #PWR01
 U 1 1 52163D8A
 P 8900 2700
-F 0 "#PWR16" H 8900 2700 30  0001 C CNN
+F 0 "#PWR01" H 8900 2700 30  0001 C CNN
 F 1 "GND" H 8900 2630 30  0001 C CNN
 F 2 "" H 8900 2700 60  0000 C CNN
@@
 	8900 2650 8900 2700
 $Comp
-L GND #PWR12
+L GND #PWR02
 U 1 1 52163DBE
 P 7850 3250
-F 0 "#PWR12" H 7850 3250 30  0001 C CNN
+F 0 "#PWR02" H 7850 3250 30  0001 C CNN
 F 1 "GND" H 7850 3180 30  0001 C CNN
 F 2 "" H 7850 3250 60  0000 C CNN
@@
 	5750 2600 5750 2650
 $Comp
-L GND #PWR7
+L GND #PWR03
 U 1 1 52164179
 P 5750 2900
-F 0 "#PWR7" H 5750 2900 30  0001 C CNN
+F 0 "#PWR03" H 5750 2900 30  0001 C CNN
 F 1 "GND" H 5750 2830 30  0001 C CNN
 F 2 "" H 5750 2900 60  0000 C CNN
@@
 	5550 2400 5550 2450
 $Comp
-L GND #PWR5
+L GND #PWR04
 U 1 1 5216431B
 P 5550 2700
-F 0 "#PWR5" H 5550 2700 30  0001 C CNN
+F 0 "#PWR04" H 5550 2700 30  0001 C CNN
 F 1 "GND" H 5550 2630 30  0001 C CNN
 F 2 "" H 5550 2700 60  0000 C CNN
@@
 $EndComp
 $Comp
-L GND #PWR8
+L GND #PWR05
 U 1 1 521647BC
 P 5750 3500
-F 0 "#PWR8" H 5750 3500 30  0001 C CNN
+F 0 "#PWR05" H 5750 3500 30  0001 C CNN
 F 1 "GND" H 5750 3430 30  0001 C CNN
 F 2 "" H 5750 3500 60  0000 C CNN
@@
 $EndComp
 $Comp
-L GND #PWR6
+L GND #PWR06
 U 1 1 521647FC
 P 5550 3300
-F 0 "#PWR6" H 5550 3300 30  0001 C CNN
+F 0 "#PWR06" H 5550 3300 30  0001 C CNN
 F 1 "GND" H 5550 3230 30  0001 C CNN
 F 2 "" H 5550 3300 60  0000 C CNN
@@
 	5750 3600 5750 3650
 $Comp
-L GND #PWR9
+L GND #PWR07
 U 1 1 52164A60
 P 5750 3900
-F 0 "#PWR9" H 5750 3900 30  0001 C CNN
+F 0 "#PWR07" H 5750 3900 30  0001 C CNN
 F 1 "GND" H 5750 3830 30  0001 C CNN
 F 2 "" H 5750 3900 60  0000 C CNN
@@
 	5000 4600 5800 4600
 $Comp
-L GND #PWR2
+L GND #PWR08
 U 1 1 521650D5
 P 3100 3650
-F 0 "#PWR2" H 3100 3650 30  0001 C CNN
+F 0 "#PWR08" H 3100 3650 30  0001 C CNN
 F 1 "GND" H 3100 3580 30  0001 C CNN
 F 2 "" H 3100 3650 60  0000 C CNN
@@
 	5150 2400 5150 2450
 $Comp
-L GND #PWR4
+L GND #PWR09
 U 1 1 52165390
 P 5150 2900
-F 0 "#PWR4" H 5150 2900 30  0001 C CNN
+F 0 "#PWR09" H 5150 2900 30  0001 C CNN
 F 1 "GND" H 5150 2830 30  0001 C CNN
 F 2 "" H 5150 2900 60  0000 C CNN
@@
 	5150 2850 5150 2900
 $Comp
-L GND #PWR11
+L GND #PWR010
 U 1 1 52165559
 P 6950 5950
-F 0 "#PWR11" H 6950 5950 30  0001 C CNN
+F 0 "#PWR010" H 6950 5950 30  0001 C CNN
 F 1 "GND" H 6950 5880 30  0001 C CNN
 F 2 "" H 6950 5950 60  0000 C CNN
@@
 	6800 5850 6800 5900
 Wire Wire Line
-	6800 5900 7100 5900
+	6700 5900 7100 5900
 Wire Wire Line
 	7100 5900 7100 5850
@@
 Connection ~ 7850 3550
 $Comp
-L GND #PWR14
+L GND #PWR011
 U 1 1 52165BB9
 P 8350 3850
-F 0 "#PWR14" H 8350 3850 30  0001 C CNN
+F 0 "#PWR011" H 8350 3850 30  0001 C CNN
 F 1 "GND" H 8350 3780 30  0001 C CNN
 F 2 "" H 8350 3850 60  0000 C CNN
@@
 (At least\n1uF)
 $Comp
-L GND #PWR17
+L GND #PWR012
 U 1 1 52165D09
 P 8900 4250
-F 0 "#PWR17" H 8900 4250 30  0001 C CNN
+F 0 "#PWR012" H 8900 4250 30  0001 C CNN
 F 1 "GND" H 8900 4180 30  0001 C CNN
 F 2 "" H 8900 4250 60  0000 C CNN
@@
 Connection ~ 7950 4300
 $Comp
-L GND #PWR13
+L GND #PWR013
 U 1 1 52166403
 P 7950 4950
-F 0 "#PWR13" H 7950 4950 30  0001 C CNN
+F 0 "#PWR013" H 7950 4950 30  0001 C CNN
 F 1 "GND" H 7950 4880 30  0001 C CNN
 F 2 "" H 7950 4950 60  0000 C CNN
@@
 Connection ~ 7950 4350
 $Comp
-L GND #PWR15
+L GND #PWR014
 U 1 1 5216692D
 P 8400 4950
-F 0 "#PWR15" H 8400 4950 30  0001 C CNN
+F 0 "#PWR014" H 8400 4950 30  0001 C CNN
 F 1 "GND" H 8400 4880 30  0001 C CNN
 F 2 "" H 8400 4950 60  0000 C CNN
@@
 Connection ~ 2400 4600
 $Comp
-L GND #PWR1
+L GND #PWR015
 U 1 1 5216AE04
 P 2400 4650
-F 0 "#PWR1" H 2400 4650 30  0001 C CNN
+F 0 "#PWR015" H 2400 4650 30  0001 C CNN
 F 1 "GND" H 2400 4580 30  0001 C CNN
 F 2 "" H 2400 4650 60  0000 C CNN
@@
 	5050 3250 5050 4400
 Wire Wire Line
-	3100 3000 5800 3000
-Wire Wire Line
 	4350 3250 5050 3250
 Wire Wire Line
 	4350 3450 5000 3450
 $Comp
-L GND #PWR3
+L GND #PWR016
 U 1 1 5216EA73
 P 4000 3700
-F 0 "#PWR3" H 4000 3700 30  0001 C CNN
+F 0 "#PWR016" H 4000 3700 30  0001 C CNN
 F 1 "GND" H 4000 3630 30  0001 C CNN
 F 2 "" H 4000 3700 60  0000 C CNN
@@
 	4000 3650 4000 3700
 $Comp
-L GND #PWR10
+L GND #PWR017
 U 1 1 522CBB9B
 P 6450 5900
-F 0 "#PWR10" H 6450 5900 30  0001 C CNN
+F 0 "#PWR017" H 6450 5900 30  0001 C CNN
 F 1 "GND" H 6450 5830 30  0001 C CNN
 F 2 "" H 6450 5900 60  0000 C CNN
@@
 Connection ~ 10800 2950
 $Comp
-L GND #PWR18
+L GND #PWR018
 U 1 1 522CCD85
 P 10800 3250
-F 0 "#PWR18" H 10800 3250 30  0001 C CNN
+F 0 "#PWR018" H 10800 3250 30  0001 C CNN
 F 1 "GND" H 10800 3180 30  0001 C CNN
 F 2 "" H 10800 3250 60  0000 C CNN
@@
 	12450 3250 12400 3250
 $Comp
-L GND #PWR19
+L GND #PWR019
 U 1 1 522CCEBE
 P 12450 3300
-F 0 "#PWR19" H 12450 3300 30  0001 C CNN
+F 0 "#PWR019" H 12450 3300 30  0001 C CNN
 F 1 "GND" H 12450 3230 30  0001 C CNN
 F 2 "" H 12450 3300 60  0000 C CNN
@@
 Connection ~ 12450 2750
 $Comp
-L GND #PWR20
+L GND #PWR020
 U 1 1 522CD09B
 P 12600 3050
-F 0 "#PWR20" H 12600 3050 30  0001 C CNN
+F 0 "#PWR020" H 12600 3050 30  0001 C CNN
 F 1 "GND" H 12600 2980 30  0001 C CNN
 F 2 "" H 12600 3050 60  0000 C CNN
@@
 6E 56 52 49 51 4E 59 71 7E 65 C5 4D 0F AF 00 BF F6 21 9D BA 45 88 9C 00 16 00 C0 66 90 E0 00 00
 AC 42 3B 38 00 00 AB 90 E0 00 00 AC 42 82 03 00 B0 EA FF 00 E3 76 B5 A7 81 B6 BC 08 00 00 00 00
-49 45 4E 44 AE 42 60 82 AF $EndBitmap
+49 45 4E 44 AE 42 60 82 B4 $EndBitmap
 EndData
 $EndBitmap
@@
 	1    0    0    -1
 $EndComp
+Wire Wire Line
+	6700 5850 6700 5900
+Connection ~ 6800 5900
+Wire Wire Line
+	3100 3000 5800 3000
+NoConn ~ 3100 3450
 $EndSCHEMATC
