File: Hardware/Pong.0.kicad_pcb (KiCad board)
At the start: 2 copper layers, 51 parts

Commit message: Added sensors and LEDs to PCB, and began dimensioning board
Parts:
- added C1, CS0, CS1, CS2, CS3: 4.7nF, SM0603, F.Cu at (7.43, 2.01)
- added C10: CSMALL, SM0603, F.Cu at (7.43, 2.01)
- added C11, C12, C4, C5: 4.7uF, SM0603, F.Cu at (7.43, 2.01)
- added C13, C15, C17, C44, C51, C58, C8: 10uF, SM0603, F.Cu at (7.43, 2.01)
- added C14, C16, C18, C43, C45, C46, C47, C52, C53, C54, C55, C56, C57, C59, C60: 0.1uF, SM0603, F.Cu at (7.43, 2.01)
- added C19, C2, C20, C3, C48, C6, C9: 1uF, SM0603, F.Cu at (7.43, 2.01)
- added C21: 2.2uF, SM0603, F.Cu at (7.43, 2.01)
- added C22, C23, C24, C25, C26, C27, C29, C30, C31, C32, C33, C34, C36, C37, C38, C39, C40, C41: 1nF, SM0603, F.Cu at (7.43, 2.01)
- added C49, C50: 15pF, SM0603, F.Cu at (7.43, 2.01)
- added C7: 0.01uF, SM0603, F.Cu at (7.43, 2.01)
- added D1: RGB_LED_V2, PLCC-5050, F.Cu at (122.2, 444.5)
- added D10: RGB_LED_V2, PLCC-5050, F.Cu at (166.7, 400.0)
- added D11: RGB_LED_V2, PLCC-5050, F.Cu at (211.1, 400.0)
- added D12: RGB_LED_V2, PLCC-5050, F.Cu at (255.6, 400.0)
- added D13: RGB_LED_V2, PLCC-5050, F.Cu at (300.0, 400.0)
- added D14: RGB_LED_V2, PLCC-5050, F.Cu at (344.5, 400.0)
- added D15: RGB_LED_V2, PLCC-5050, F.Cu at (388.9, 400.0)
- added D16: RGB_LED_V2, PLCC-5050, F.Cu at (433.4, 400.0)
- added D17: RGB_LED_V2, PLCC-5050, F.Cu at (122.3, 355.6)
- added D18: RGB_LED_V2, PLCC-5050, F.Cu at (166.8, 355.6)
- added D19: RGB_LED_V2, PLCC-5050, F.Cu at (211.1, 355.6)
- added D2: RGB_LED_V2, PLCC-5050, F.Cu at (166.7, 444.5)
- added D20: RGB_LED_V2, PLCC-5050, F.Cu at (255.6, 355.6)
- added D21: RGB_LED_V2, PLCC-5050, F.Cu at (300.0, 355.6)
- added D22: RGB_LED_V2, PLCC-5050, F.Cu at (344.5, 355.6)
- added D23: RGB_LED_V2, PLCC-5050, F.Cu at (388.9, 355.6)
- added D24: RGB_LED_V2, PLCC-5050, F.Cu at (122.2, 311.1)
- added D25: RGB_LED_V2, PLCC-5050, F.Cu at (166.7, 311.1)
- added D26: RGB_LED_V2, PLCC-5050, F.Cu at (211.1, 311.1)
- added D27: RGB_LED_V2, PLCC-5050, F.Cu at (255.6, 311.1)
- added D28: RGB_LED_V2, PLCC-5050, F.Cu at (300.0, 311.1)
- added D29: RGB_LED_V2, PLCC-5050, F.Cu at (344.5, 311.1)
- added D3: RGB_LED_V2, PLCC-5050, F.Cu at (211.1, 444.5)
- added D30: RGB_LED_V2, PLCC-5050, F.Cu at (388.9, 311.1)
- added D31: RGB_LED_V2, PLCC-5050, F.Cu at (166.7, 266.7)
- added D32: RGB_LED_V2, PLCC-5050, F.Cu at (211.1, 266.7)
- added D33: RGB_LED_V2, PLCC-5050, F.Cu at (255.6, 266.7)
- added D34: RGB_LED_V2, PLCC-5050, F.Cu at (300.0, 266.7)
- added D35: RGB_LED_V2, PLCC-5050, F.Cu at (344.5, 266.7)
- added D36: RGB_LED_V2, PLCC-5050, F.Cu at (166.7, 222.2)
- added D37: RGB_LED_V2, PLCC-5050, F.Cu at (211.1, 222.2)
- added D38: RGB_LED_V2, PLCC-5050, F.Cu at (255.6, 222.2)
- added D39: RGB_LED_V2, PLCC-5050, F.Cu at (300.0, 222.2)
- added D4: RGB_LED_V2, PLCC-5050, F.Cu at (255.6, 444.5)
- added D40: RGB_LED_V2, PLCC-5050, F.Cu at (344.5, 222.2)
- added D41: RGB_LED_V2, PLCC-5050, F.Cu at (211.1, 177.8)
- added D42: RGB_LED_V2, PLCC-5050, F.Cu at (255.6, 177.8)
- added D43: RGB_LED_V2, PLCC-5050, F.Cu at (300.0, 177.8)
- added D44: RGB_LED_V2, PLCC-5050, F.Cu at (211.1, 133.3)
- added D45: RGB_LED_V2, PLCC-5050, F.Cu at (255.6, 133.3)
- added D46: RGB_LED_V2, PLCC-5050, F.Cu at (300.0, 133.3)
- added D47: RGB_LED_V2, PLCC-5050, F.Cu at (255.6, 88.9)
- added D48: RGB_LED_V2, PLCC-5050, F.Cu at (257.4, -43.6)
- added D49: RGB_LED_V2, PLCC-5050, F.Cu at (202.6, -65.8)
- added D5: RGB_LED_V2, PLCC-5050, F.Cu at (300.0, 444.5)
- added D50: RGB_LED_V2, PLCC-5050, F.Cu at (192.4, -15.3)
- added D51: RGB_LED_V2, PLCC-5050, F.Cu at (202.7, -55.6)
- added D52: RGB_LED_V2, PLCC-5050, F.Cu at (192.2, -25.1)
- added D53: RGB_LED_V2, PLCC-5050, F.Cu at (192.6, -34.8)
- added D54: RGB_LED_V2, PLCC-5050, F.Cu at (192.9, -45.0)
- added D55: RGB_LED_V2, PLCC-5050, F.Cu at (193.1, -55.1)
- added D56: RGB_LED_V2, PLCC-5050, F.Cu at (193.3, -65.3)
- added D57: RGB_LED_V2, PLCC-5050, F.Cu at (183.2, -15.4)
- added D58: RGB_LED_V2, PLCC-5050, F.Cu at (182.8, -25.4)
- added D59: RGB_LED_V2, PLCC-5050, F.Cu at (183.0, -34.9)
- added D6: RGB_LED_V2, PLCC-5050, F.Cu at (344.5, 444.5)
- added D60: RGB_LED_V2, PLCC-5050, F.Cu at (183.4, -45.5)
- added D61: RGB_LED_V2, PLCC-5050, F.Cu at (183.2, -55.4)
- added D62: RGB_LED_V2, PLCC-5050, F.Cu at (183.7, -65.2)
- added D63: RGB_LED_V2, PLCC-5050, F.Cu at (174.1, -15.6)
- added D64: RGB_LED_V2, PLCC-5050, F.Cu at (173.5, -25.0)
- added D65: BATT_STAT, LED-0805, F.Cu at (0.00, 0.00)
- added D66: LED, LED-0805, F.Cu at (0.00, 0.00)
- added D7: RGB_LED_V2, PLCC-5050, F.Cu at (388.9, 444.5)
- added D8: RGB_LED_V2, PLCC-5050, F.Cu at (77.8, 400.0)
- added D9: RGB_LED_V2, PLCC-5050, F.Cu at (122.2, 400.0)
- added P2: ISP, pin_array_3x2, F.Cu at (18.5, -27.0)
- added P5: JTAG, PIN_ARRAY_5x2, F.Cu at (11.9, -16.4)
- added P6: PDI, pin_array_3x2, F.Cu at (22.3, -9.32)
- added QM1: CAPSENSOR, Capsensor_35mm_x_60mm, F.Cu at (100.0, 400.0)
- added QM10: CAPSENSOR, Capsensor_35mm_x_60mm, F.Cu at (188.9, 311.1)
- added QM11: CAPSENSOR, Capsensor_35mm_x_60mm, F.Cu at (233.4, 311.1)
- added QM12: CAPSENSOR, Capsensor_35mm_x_60mm, F.Cu at (277.8, 311.1)
- added QM13: CAPSENSOR, Capsensor_35mm_x_60mm, F.Cu at (322.3, 311.1)
- added QM14: CAPSENSOR, Capsensor_35mm_x_60mm, F.Cu at (366.7, 311.1)
- added QM15: CAPSENSOR, Capsensor_35mm_x_60mm, F.Cu at (188.9, 222.2)
- added QM16: CAPSENSOR, Capsensor_35mm_x_60mm, F.Cu at (233.4, 222.2)
- added QM17: CAPSENSOR, Capsensor_35mm_x_60mm, F.Cu at (277.8, 222.2)
- added QM18: CAPSENSOR, Capsensor_35mm_x_60mm, F.Cu at (322.3, 222.2)
- added QM19: CAPSENSOR, Capsensor_35mm_x_60mm, F.Cu at (233.4, 133.4)
- added QM2: CAPSENSOR, Capsensor_35mm_x_60mm, F.Cu at (144.5, 400.0)
- added QM20: CAPSENSOR, Capsensor_35mm_x_60mm, F.Cu at (277.8, 133.3)
- added QM3: CAPSENSOR, Capsensor_35mm_x_60mm, F.Cu at (188.9, 400.0)
- added QM4: CAPSENSOR, Capsensor_35mm_x_60mm, F.Cu at (233.4, 400.0)
- added QM5: CAPSENSOR, Capsensor_35mm_x_60mm, F.Cu at (277.8, 400.0)
- added QM6: CAPSENSOR, Capsensor_35mm_x_60mm, F.Cu at (322.3, 400.0)
- added QM7: CAPSENSOR, Capsensor_35mm_x_60mm, F.Cu at (366.7, 400.0)
- added QM8: CAPSENSOR, Capsensor_35mm_x_60mm, F.Cu at (411.2, 400.0)
- added QM9: CAPSENSOR, Capsensor_35mm_x_60mm, F.Cu at (144.5, 311.1)
- added U2: BQ24163, QFN24, F.Cu at (39.0, -4.07)
- added U5: NVT2006, TSSOP16, F.Cu at (30.7, -20.2)
- added U6: AS1116, SSOP24, F.Cu at (42.6, -20.7)
- added U8: W25X20CL, SO8E, F.Cu at (37.1, -12.1)
Other:
- board outline added: 382.2 x 380 mm

Commit message: Continued layout of PCB
Parts:
- moved D49 282.8 mm to (427.8, 105.3)
- moved D50 282.8 mm to (417.6, 155.8)
- moved D51 282.8 mm to (427.9, 115.5)
- moved D52 282.8 mm to (417.4, 146.0)
- moved D53 282.8 mm to (417.8, 136.3)
- moved D54 282.8 mm to (418.1, 126.2)
- moved D55 282.8 mm to (418.2, 116.0)
- moved D56 282.8 mm to (418.5, 105.8)
- moved D57 282.8 mm to (408.4, 155.7)
- moved D58 282.8 mm to (407.9, 145.8)
- moved D59 282.8 mm to (408.2, 136.2)
- moved D60 282.8 mm to (408.6, 125.5)
- moved D61 282.8 mm to (408.4, 115.8)
- moved D62 282.8 mm to (408.9, 105.8)
- moved D63 282.8 mm to (399.3, 155.5)
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
Commit message: Added slider, more capacitive sensors, and several ICs. Continuing board layout.
Parts:
- added QM21: CAPSENSOR, CapSensor_20mm_x_24mm, F.Cu at (380.0, 199.2)
- added QM22: CAPSENSOR, CapSensor_20mm_x_24mm, F.Cu at (402.2, 199.2)
- added QM23: CAPSENSOR, CapSensor_20mm_x_24mm, F.Cu at (424.7, 199.2)
- added QM24: CAPSENSOR, CapSensor_20mm_x_24mm, F.Cu at (472.6, 442.0)
- added U1: IP4234CZ6, SOT457, F.Cu at (504.9, 226.6)
- added U10: CAPSLIDER, CapSensor_Slider_16mm_x_66mm, F.Cu at (402.2, 130.6)
- added U3: TPS61240, QFN-6, F.Cu at (498.2, 226.4)
- added U4: AS1119, WLCSP-36, F.Cu at (487.9, 246.2)
- moved P2 513.7 mm to (480.3, 197.9)
- moved P5 513.7 mm to (473.7, 208.5)
- moved P6 513.7 mm to (484.1, 215.6)
- moved U2 510.2 mm to (480.1, 252.2)
- moved U5 510.2 mm to (471.8, 236.1)
- moved U6 510.2 mm to (483.7, 235.6)
- moved U8 510.2 mm to (478.2, 244.2)
- moved D48 379.8 mm to (72.2, -8.50)
- moved C55 88.2 mm to (91.2, 29.5)
- moved C12 87.6 mm to (91.2, 27.8)
- moved C11 87.2 mm to (91.2, 26.1)
- moved C59 86.7 mm to (91.2, 24.4)
- moved C1 86.3 mm to (91.2, 22.7)
- moved C9 85.9 mm to (91.2, 21.1)
- moved C6 85.6 mm to (91.2, 19.4)
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